File: Temp_sensors/temp_sensors_array.brd (EAGLE design)
At the start: 50 x 50 mm, 7 parts, among them U1 SI7021, U2 SI7021, U3 HDC1080, U4 HDC1080, U5 BME280, U6 BME280

Commit message: temp_array: added PCA9548APWR
Signed-off-by: malo <malo@25cmsquare.io>
Parts:
- added U7: PCA9548APWR, Texas Instruments_By_element14_Batch_1:SOP65P640X120-24N
Connections:
- new net I2C0_SCL: U7.5
- new net I2C0_SDA: U7.4
- new net I2C1_SCL: U7.7
- new net I2C1_SDA: U7.6
- new net I2C2_SCL: U7.9
- new net I2C2_SDA: U7.8
- new net N$1: PWR1.12, U7.23
- new net N$10: U7.17
- new net N$11: U7.18
- new net N$12: U7.19
- new net N$13: U7.20
- new net N$2: PWR1.11, U7.22
- new net N$3: PWR1.7, U7.3
- new net N$4: U7.10
- new net N$5: U7.11
- new net N$6: U7.13
- new net N$7: U7.14
- new net N$8: U7.15
- new net N$9: U7.16
- new net VCC: PWR1.6, U7.24
- net GND: now also PWR1.3, PWR1.8, U7.12
Changed lines of the file:
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@@
 <element name="U5" library="25cmsquare" package="BME1080" value="BME280" x="15.24" y="25.4"/>
 <element name="U6" library="25cmsquare" package="BME1080" value="BME280" x="34.29" y="25.4"/>
+<element name="U7" library="Texas Instruments_By_element14_Batch_1" package="SOP65P640X120-24N" value="PCA9548APWR" x="17.78" y="10.16">
+<attribute name="OC_NEWARK" value="22M1602" x="17.78" y="10.16" size="1.778" layer="27" display="off"/>
+<attribute name="MPN" value="PCA9548APWR    False" x="17.78" y="10.16" size="1.778" layer="27" display="off"/>
+<attribute name="SUPPLIER" value="Texas Instruments" x="17.78" y="10.16" size="1.778" layer="27" display="off"/>
+<attribute name="OC_FARNELL" value="1607855" x="17.78" y="10.16" size="1.778" layer="27" display="off"/>
+<attribute name="PACKAGE" value="TSSOP-24" x="17.78" y="10.16" size="1.778" layer="27" display="off"/>
+</element>
 </elements>
 <signals>
@@
 <contactref element="U6" pad="7"/>
 <contactref element="U6" pad="1"/>
+<contactref element="PWR1" pad="3"/>
+<contactref element="U7" pad="12"/>
+<contactref element="PWR1" pad="8"/>
+<wire x1="35.3025" y1="26.375" x2="33.2775" y2="25.725" width="0" layer="19" extent="1-1"/>
+<wire x1="27.76" y1="27.94" x2="33.2775" y2="25.725" width="0" layer="19" extent="1-1"/>
 <wire x1="27.76" y1="21.59" x2="27.76" y2="27.94" width="0" layer="19" extent="1-1"/>
 <wire x1="20.14" y1="27.94" x2="27.76" y2="27.94" width="0" layer="19" extent="1-1"/>
-<wire x1="20.14" y1="21.59" x2="20.14" y2="27.94" width="0" layer="19" extent="1-1"/>
-<wire x1="16.2525" y1="26.375" x2="20.14" y2="21.59" width="0" layer="19" extent="1-1"/>
+<wire x1="16.2525" y1="26.375" x2="20.14" y2="27.94" width="0" layer="19" extent="1-1"/>
 <wire x1="14.2275" y1="25.725" x2="16.2525" y2="26.375" width="0" layer="19" extent="1-1"/>
-<wire x1="35.3025" y1="26.375" x2="14.2275" y2="25.725" width="0" layer="19" extent="1-1"/>
-<wire x1="33.2775" y1="25.725" x2="35.3025" y2="26.375" width="0" layer="19" extent="1-1"/>
+<wire x1="20.14" y1="21.59" x2="16.2525" y2="26.375" width="0" layer="19" extent="1-1"/>
+<wire x1="2.5" y1="30.08" x2="14.2275" y2="25.725" width="0" layer="19" extent="1-1"/>
+<wire x1="2.5" y1="14.84" x2="2.5" y2="30.08" width="0" layer="19" extent="1-1"/>
+<wire x1="14.859" y1="6.5786" x2="2.5" y2="14.84" width="0" layer="19" extent="1-1"/>
 </signal>
 <signal name="VDDIO">
@@
 <wire x1="14.2275" y1="25.075" x2="33.2775" y2="25.075" width="0" layer="19" extent="1-1"/>
 </signal>
+<signal name="VCC">
+<contactref element="U7" pad="24"/>
+<contactref element="PWR1" pad="6"/>
+<wire x1="2.5" y1="22.46" x2="20.701" y2="13.7414" width="0" layer="19" extent="1-1"/>
+</signal>
+<signal name="N$1">
+<contactref element="PWR1" pad="12"/>
+<contactref element="U7" pad="23"/>
+<wire x1="20.701" y1="13.081" x2="2.5" y2="40.24" width="0" layer="19" extent="1-1"/>
+</signal>
+<signal name="N$2">
+<contactref element="PWR1" pad="11"/>
+<contactref element="U7" pad="22"/>
+<wire x1="20.701" y1="12.446" x2="2.5" y2="37.7" width="0" layer="19" extent="1-1"/>
+</signal>
+<signal name="N$3">
+<contactref element="PWR1" pad="7"/>
+<contactref element="U7" pad="3"/>
+<wire x1="14.859" y1="12.446" x2="2.5" y2="27.54" width="0" layer="19" extent="1-1"/>
+</signal>
+<signal name="I2C0_SDA">
+<contactref element="U7" pad="4"/>
+</signal>
+<signal name="I2C0_SCL">
+<contactref element="U7" pad="5"/>
+</signal>
+<signal name="I2C1_SDA">
+<contactref element="U7" pad="6"/>
+</signal>
+<signal name="I2C1_SCL">
+<contactref element="U7" pad="7"/>
+</signal>
+<signal name="I2C2_SDA">
+<contactref element="U7" pad="8"/>
+</signal>
+<signal name="I2C2_SCL">
+<contactref element="U7" pad="9"/>
+</signal>
+<signal name="N$4">
+<contactref element="U7" pad="10"/>
+</signal>
+<signal name="N$5">
+<contactref element="U7" pad="11"/>
+</signal>
+<signal name="N$6">
+<contactref element="U7" pad="13"/>
+</signal>
+<signal name="N$7">
+<contactref element="U7" pad="14"/>
+</signal>
+<signal name="N$8">
+<contactref element="U7" pad="15"/>
+</signal>
+<signal name="N$9">
+<contactref element="U7" pad="16"/>
+</signal>
+<signal name="N$10">
+<contactref element="U7" pad="17"/>
+</signal>
+<signal name="N$11">
+<contactref element="U7" pad="18"/>
+</signal>
+<signal name="N$12">
+<contactref element="U7" pad="19"/>
+</signal>
+<signal name="N$13">
+<contactref element="U7" pad="20"/>
+</signal>
 </signals>
