File: xpower_1V0_2V5_3V3_POR/xpower.sch (EAGLE design)
At the start: 34 parts, among them U1 TLV70233, U2 TLV70225, U3 STM1061N29, U4 ADM1085, U5 LM3674-ADJ

Commit message: WIP: xpower - minor final tweaks.
Signed-off-by: malo <pavol.malosek@gmail.com>
Connections:
- net D_N: now also PWR1.9; no longer PWR1.10
- net D_P: now also PWR1.10; no longer PWR1.9
- net PE: no longer U$5.MTN1, U$5.MTN2, U$5.MTN4
Changed lines of the file:
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@@
 <part name="PE3" library="supply1" deviceset="PE" device=""/>
 <part name="GND26" library="supply1" deviceset="GND" device=""/>
-<part name="PE4" library="supply1" deviceset="PE" device=""/>
 <part name="PE5" library="supply1" deviceset="PE" device=""/>
 <part name="U$5" library="pma" deviceset="ZX62D-B-5PA8" device=""/>
@@
 <instance part="PE3" gate="M" x="88.9" y="104.14"/>
 <instance part="GND26" gate="1" x="109.22" y="104.14"/>
-<instance part="PE4" gate="M" x="93.98" y="166.37"/>
-<instance part="PE5" gate="M" x="93.98" y="130.81"/>
+<instance part="PE5" gate="M" x="104.14" y="133.35"/>
 <instance part="U$5" gate="G$1" x="104.14" y="152.4" rot="MR0"/>
 <instance part="C9" gate="G$1" x="96.52" y="114.3" smashed="yes" rot="MR270">
@@
 <net name="PE" class="0">
 <segment>
-<wire x1="104.14" y1="162.56" x2="104.14" y2="168.91" width="0.1524" layer="91"/>
-<wire x1="104.14" y1="168.91" x2="101.6" y2="168.91" width="0.1524" layer="91"/>
-<wire x1="101.6" y1="168.91" x2="101.6" y2="162.56" width="0.1524" layer="91"/>
-<wire x1="101.6" y1="168.91" x2="93.98" y2="168.91" width="0.1524" layer="91"/>
-<junction x="101.6" y="168.91"/>
-<pinref part="PE4" gate="M" pin="PE"/>
-<pinref part="U$5" gate="G$1" pin="MTN1"/>
-<pinref part="U$5" gate="G$1" pin="MTN2"/>
-</segment>
-<segment>
-<wire x1="104.14" y1="142.24" x2="104.14" y2="133.35" width="0.1524" layer="91"/>
-<wire x1="104.14" y1="133.35" x2="101.6" y2="133.35" width="0.1524" layer="91"/>
-<wire x1="101.6" y1="142.24" x2="101.6" y2="133.35" width="0.1524" layer="91"/>
-<wire x1="101.6" y1="133.35" x2="93.98" y2="133.35" width="0.1524" layer="91"/>
-<junction x="101.6" y="133.35"/>
+<wire x1="104.14" y1="142.24" x2="104.14" y2="135.89" width="0.1524" layer="91"/>
 <pinref part="PE5" gate="M" pin="PE"/>
 <pinref part="U$5" gate="G$1" pin="MTN3"/>
-<pinref part="U$5" gate="G$1" pin="MTN4"/>
 </segment>
 <segment>
@@
 </segment>
 <segment>
-<pinref part="PWR1" gate="G$1" pin="10"/>
-<wire x1="53.34" y1="160.02" x2="71.12" y2="160.02" width="0.1524" layer="91"/>
-<label x="71.12" y="160.02" size="1.778" layer="95" xref="yes"/>
+<pinref part="PWR1" gate="G$1" pin="9"/>
+<wire x1="53.34" y1="157.48" x2="73.66" y2="157.48" width="0.1524" layer="91"/>
+<label x="73.66" y="157.48" size="1.778" layer="95" xref="yes"/>
 </segment>
 </net>
@@
 </segment>
 <segment>
-<pinref part="PWR1" gate="G$1" pin="9"/>
-<wire x1="53.34" y1="157.48" x2="78.74" y2="157.48" width="0.1524" layer="91"/>
-<label x="78.74" y="157.48" size="1.778" layer="95" xref="yes"/>
-</segment>
-</net>
+<pinref part="PWR1" gate="G$1" pin="10"/>
+<wire x1="53.34" y1="160.02" x2="63.5" y2="160.02" width="0.1524" layer="91"/>
+<label x="63.5" y="160.02" size="1.778" layer="95" xref="yes"/>
+</segment>
+</net>

Commit message: WIP: xpower - minor final tweaks.
Signed-off-by: malo <pavol.malosek@gmail.com>
Parts:
- removed 5V: TEST-22-MULTICOMP, 25cmsquare:TEST-22-MULTICOMP
- added 5V0: TPTP14R, testpad:TPTP14R
- 1V0, 2V5, 3V3: value TEST-22-MULTICOMP -> TPTP14R; device 25cmsquare:TEST-22-MULTICOMP -> testpad:TPTP14R
Connections:
- net N$2 renamed VBUS
- net +1V0: now also 1V0.TP; no longer 1V0.1
- net +2V5: now also 2V5.TP; no longer 2V5.1
- net +3V3: now also 3V3.TP; no longer 3V3.1
- net +5V: now also 5V0.TP; no longer 5V.1
- net PE: now also U$5.MTN4; no longer U$5.MTN3
Other:
- moved on the sheet: GND
Changed lines of the file:
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@@
 <part name="GND12" library="supply1" deviceset="GND" device=""/>
 <part name="U$1" library="25cmsquare" deviceset="+1V0" device=""/>
-<part name="5V" library="25cmsquare" deviceset="TEST-22-MULTICOMP" device=""/>
-<part name="3V3" library="25cmsquare" deviceset="TEST-22-MULTICOMP" device=""/>
-<part name="2V5" library="25cmsquare" deviceset="TEST-22-MULTICOMP" device=""/>
 <part name="GND" library="25cmsquare" deviceset="TEST-22-MULTICOMP" device=""/>
-<part name="P+3" library="supply1" deviceset="+5V" device=""/>
-<part name="+3V5" library="supply1" deviceset="+3V3" device=""/>
-<part name="+2V2" library="25cmsquare" deviceset="+2V5" device=""/>
-<part name="1V0" library="25cmsquare" deviceset="TEST-22-MULTICOMP" device=""/>
-<part name="U$7" library="25cmsquare" deviceset="+1V0" device=""/>
 <part name="GND13" library="supply1" deviceset="GND" device=""/>
 <part name="+3V6" library="supply1" deviceset="+3V3" device=""/>
@@
 <part name="GND30" library="supply1" deviceset="GND" device=""/>
 <part name="P+6" library="supply1" deviceset="+5V" device=""/>
+<part name="1V0" library="testpad" deviceset="TP" device="TP14R"/>
+<part name="2V5" library="testpad" deviceset="TP" device="TP14R"/>
+<part name="3V3" library="testpad" deviceset="TP" device="TP14R"/>
+<part name="5V0" library="testpad" deviceset="TP" device="TP14R"/>
+<part name="P+3" library="supply1" deviceset="+5V" device=""/>
+<part name="+2V2" library="25cmsquare" deviceset="+2V5" device=""/>
+<part name="+3V5" library="supply1" deviceset="+3V3" device=""/>
+<part name="U$4" library="25cmsquare" deviceset="+1V0" device=""/>
 </parts>
 <sheets>
@@
 <instance part="GND12" gate="1" x="190.5" y="35.56" rot="MR0"/>
 <instance part="U$1" gate="A" x="172.72" y="86.36"/>
-<instance part="5V" gate="G$1" x="22.86" y="20.32" rot="MR270"/>
-<instance part="3V3" gate="G$1" x="30.48" y="20.32" rot="MR270"/>
-<instance part="2V5" gate="G$1" x="38.1" y="20.32" rot="MR270"/>
-<instance part="GND" gate="G$1" x="53.34" y="15.24" rot="MR90"/>
-<instance part="P+3" gate="1" x="22.86" y="22.86"/>
-<instance part="+3V5" gate="G$1" x="30.48" y="22.86"/>
-<instance part="+2V2" gate="G$1" x="38.1" y="20.32"/>
-<instance part="1V0" gate="G$1" x="45.72" y="20.32" rot="MR270"/>
-<instance part="U$7" gate="A" x="45.72" y="20.32"/>
-<instance part="GND13" gate="1" x="53.34" y="12.7" rot="MR0"/>
+<instance part="GND" gate="G$1" x="55.88" y="15.24" rot="MR90"/>
+<instance part="GND13" gate="1" x="55.88" y="12.7" rot="MR0"/>
 <instance part="+3V6" gate="G$1" x="109.22" y="81.28"/>
 <instance part="GND14" gate="1" x="109.22" y="38.1" rot="MR0"/>
@@
 <instance part="PE3" gate="M" x="88.9" y="104.14"/>
 <instance part="GND26" gate="1" x="109.22" y="104.14"/>
-<instance part="PE5" gate="M" x="104.14" y="133.35"/>
+<instance part="PE5" gate="M" x="101.6" y="132.08"/>
 <instance part="U$5" gate="G$1" x="104.14" y="152.4" rot="MR0"/>
 <instance part="C9" gate="G$1" x="96.52" y="114.3" smashed="yes" rot="MR270">
@@
 <instance part="P+6" gate="1" x="172.72" y="165.1" smashed="yes">
 <attribute name="VALUE" x="172.72" y="165.1" size="1.778" layer="96" rot="R90"/>
+</instance>
+<instance part="1V0" gate="G$1" x="25.4" y="17.78" rot="R180"/>
+<instance part="2V5" gate="G$1" x="33.02" y="17.78" rot="R180"/>
+<instance part="3V3" gate="G$1" x="40.64" y="17.78" rot="R180"/>
+<instance part="5V0" gate="G$1" x="48.26" y="17.78" rot="R180"/>
+<instance part="P+3" gate="1" x="48.26" y="22.86"/>
+<instance part="+2V2" gate="G$1" x="33.02" y="20.32" smashed="yes">
+<attribute name="VALUE" x="30.48" y="17.78" size="1.778" layer="96" rot="R90"/>
+</instance>
+<instance part="+3V5" gate="G$1" x="40.64" y="22.86"/>
+<instance part="U$4" gate="A" x="25.4" y="20.32" smashed="yes" rot="MR0">
+<attribute name="VALUE" x="20.32" y="17.78" size="1.778" layer="96" rot="MR90"/>
 </instance>
 </instances>
@@
 </segment>
 <segment>
-<pinref part="5V" gate="G$1" pin="1"/>
-<pinref part="P+3" gate="1" pin="+5V"/>
-</segment>
-<segment>
 <pinref part="U5" gate="G$1" pin="VIN"/>
 <wire x1="147.32" y1="124.46" x2="132.08" y2="124.46" width="0.1524" layer="91"/>
@@
 <wire x1="172.72" y1="157.48" x2="172.72" y2="162.56" width="0.1524" layer="91"/>
 <junction x="172.72" y="157.48"/>
+</segment>
+<segment>
+<pinref part="5V0" gate="G$1" pin="TP"/>
+<pinref part="P+3" gate="1" pin="+5V"/>
 </segment>
 </net>
@@
 </segment>
 <segment>
-<pinref part="3V3" gate="G$1" pin="1"/>
-<pinref part="+3V5" gate="G$1" pin="+3V3"/>
-</segment>
-<segment>
 <wire x1="109.22" y1="63.5" x2="109.22" y2="78.74" width="0.1524" layer="91"/>
 <pinref part="+3V6" gate="G$1" pin="+3V3"/>
@@
 <pinref part="+3V7" gate="G$1" pin="+3V3"/>
 <wire x1="53.34" y1="144.78" x2="71.12" y2="144.78" width="0.1524" layer="91"/>
+</segment>
+<segment>
+<pinref part="3V3" gate="G$1" pin="TP"/>
+<pinref part="+3V5" gate="G$1" pin="+3V3"/>
 </segment>
 </net>
@@
 </segment>
 <segment>
-<pinref part="2V5" gate="G$1" pin="1"/>
-<pinref part="+2V2" gate="G$1" pin="+2V5"/>
-</segment>
-<segment>
 <pinref part="PWR1" gate="G$1" pin="1"/>
 <wire x1="53.34" y1="137.16" x2="58.42" y2="137.16" width="0.1524" layer="91"/>
 <pinref part="+2V3" gate="G$1" pin="+2V5"/>
+</segment>
+<segment>
+<pinref part="2V5" gate="G$1" pin="TP"/>
+<pinref part="+2V2" gate="G$1" pin="+2V5"/>
 </segment>
 </net>
@@
 <pinref part="U$1" gate="A" pin="+1V0"/>
 <pinref part="R5" gate="G$1" pin="2"/>
-</segment>
-<segment>
-<pinref part="1V0" gate="G$1" pin="1"/>
-<pinref part="U$7" gate="A" pin="+1V0"/>
 </segment>
 <segment>
@@
 <wire x1="53.34" y1="139.7" x2="71.12" y2="139.7" width="0.1524" layer="91"/>
 </segment>
+<segment>
+<pinref part="1V0" gate="G$1" pin="TP"/>
+<pinref part="U$4" gate="A" pin="+1V0"/>
+</segment>
 </net>
 <net name="FB" class="0">
@@
 <net name="PE" class="0">
 <segment>
-<wire x1="104.14" y1="142.24" x2="104.14" y2="135.89" width="0.1524" layer="91"/>
-<pinref part="PE5" gate="M" pin="PE"/>
-<pinref part="U$5" gate="G$1" pin="MTN3"/>
-</segment>
-<segment>
 <pinref part="R8" gate="G$1" pin="2"/>
 <pinref part="C9" gate="G$1" pin="1"/>
@@
 <wire x1="88.9" y1="109.22" x2="88.9" y2="106.68" width="0.1524" layer="91"/>
 </segment>
-</net>
-<net name="N$2" class="0">
+<segment>
+<pinref part="PE5" gate="M" pin="PE"/>
+<pinref part="U$5" gate="G$1" pin="MTN4"/>
+<wire x1="101.6" y1="134.62" x2="101.6" y2="142.24" width="0.1524" layer="91"/>
+</segment>
+</net>
+<net name="VBUS" class="0">
 <segment>
 <pinref part="U$5" gate="G$1" pin="VBUS"/>
