File: spdif/spdif_A.brd (EAGLE design)
At the start: 70 x 70 mm, 66 parts, among them T1 DA101MC, T2 DA101MC, U1 NC7SZ175, U2 FIN1001, U3 FIN1002, U4 NC7SZ175, U5 NC7SZ175, U6 FIN1002

Commit message: spdif: fixed JP2 position - regenerated gerbers.
Signed-off-by: malo <pavol.malosek@gmail.com>
Parts:
- moved JP2 0.10 mm to (71.4, 45.0)
Other:
- board text added: "TX0"
- board text added: "TX1"
- board text added: "TX2"
- board text removed: "OUT0"
- board text removed: "OUT1"
- board text removed: "OUT2"
Changed lines of the file:
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@@
 <setting verticaltext="up"/>
 </settings>
-<grid distance="5" unitdist="mil" unit="mil" style="lines" multiple="1" display="yes" altdistance="0.025" altunitdist="inch" altunit="inch"/>
+<grid distance="5" unitdist="mil" unit="mil" style="lines" multiple="1" display="no" altdistance="0.025" altunitdist="inch" altunit="inch"/>
 <layers>
 <layer number="1" name="Top" color="4" fill="1" visible="yes" active="yes"/>
@@
 <text x="60.325" y="43.307" size="1.016" layer="25" font="vector" ratio="15">CLK1</text>
 <text x="60.325" y="48.387" size="1.016" layer="25" font="vector" ratio="15">CLK0</text>
-<text x="60.325" y="50.9778" size="1.016" layer="25" font="vector" ratio="15">OUT0</text>
-<text x="60.325" y="45.847" size="1.016" layer="25" font="vector" ratio="15">OUT1</text>
-<text x="60.325" y="40.767" size="1.016" layer="25" font="vector" ratio="15">OUT2</text>
+<text x="61.468" y="50.8508" size="1.016" layer="25" font="vector" ratio="15">TX0</text>
+<text x="61.468" y="45.847" size="1.016" layer="25" font="vector" ratio="15">TX1</text>
+<text x="61.468" y="40.767" size="1.016" layer="25" font="vector" ratio="15">TX2</text>
 <text x="5.842" y="38.481" size="1.905" layer="25" font="vector" ratio="15">16.11.22.A</text>
 <text x="62.357" y="60.452" size="1.016" layer="25" font="vector" ratio="15">GND</text>
@@
 <attribute name="VALUE" x="67.6148" y="15.621" size="1.27" layer="27"/>
 </element>
-<element name="JP2" library="25pinhead" package="2X06/90" value="" x="71.3232" y="45" smashed="yes" rot="R270">
-<attribute name="NAME" x="64.9732" y="52.62" size="1.016" layer="25" font="vector" ratio="15"/>
-<attribute name="VALUE" x="67.5132" y="35.475" size="1.27" layer="27"/>
+<element name="JP2" library="25pinhead" package="2X06/90" value="" x="71.4248" y="45" smashed="yes" rot="R270">
+<attribute name="NAME" x="65.0748" y="52.62" size="1.016" layer="25" font="vector" ratio="15"/>
+<attribute name="VALUE" x="67.6148" y="35.475" size="1.27" layer="27"/>
 </element>
 <element name="PWR" library="25cmsquare" package="LIWE_12_PIN_7X7_COMPAT" value="" x="70" y="70" rot="R180"/>
@@
 <contactref element="U5" pad="1"/>
 <contactref element="JP2" pad="7"/>
-<wire x1="48.345" y1="43.73" x2="64.9732" y2="43.73" width="0.3048" layer="1"/>
+<wire x1="48.345" y1="43.73" x2="65.0748" y2="43.73" width="0.3048" layer="1"/>
 <wire x1="48.345" y1="43.73" x2="47.0154" y2="45.0596" width="0.3048" layer="1"/>
 <wire x1="47.0154" y1="45.0596" x2="44.8564" y2="45.0596" width="0.3048" layer="1"/>
@@
 <contactref element="JP2" pad="1"/>
 <wire x1="59.5884" y1="51.3334" x2="64.9566" y2="51.3334" width="0.3048" layer="1"/>
-<wire x1="64.9566" y1="51.3334" x2="64.9732" y2="51.35" width="0.3048" layer="1"/>
+<wire x1="64.9566" y1="51.3334" x2="65.0748" y2="51.35" width="0.3048" layer="1"/>
 </signal>
 <signal name="SPDIF_OUT_1">
@@
 <contactref element="JP2" pad="5"/>
 <wire x1="44.8564" y1="46.3804" x2="64.9478" y2="46.3804" width="0.3048" layer="1"/>
-<wire x1="64.9478" y1="46.3804" x2="64.9732" y2="46.27" width="0.3048" layer="1"/>
+<wire x1="64.9478" y1="46.3804" x2="65.0748" y2="46.27" width="0.3048" layer="1"/>
 </signal>
 <signal name="N$8">
@@
 <contactref element="U4" pad="1"/>
 <contactref element="JP2" pad="3"/>
-<wire x1="63.077" y1="48.81" x2="64.9732" y2="48.81" width="0.3048" layer="1"/>
+<wire x1="63.077" y1="48.81" x2="65.0748" y2="48.81" width="0.3048" layer="1"/>
 <wire x1="63.077" y1="48.81" x2="61.8744" y2="50.0126" width="0.3048" layer="1"/>
 <wire x1="61.8744" y1="50.0126" x2="59.5884" y2="50.0126" width="0.3048" layer="1"/>
@@
 <contactref element="JP2" pad="9"/>
 <wire x1="29.591" y1="41.2496" x2="64.9478" y2="41.2496" width="0.3048" layer="1"/>
-<wire x1="64.9478" y1="41.2496" x2="64.9732" y2="41.19" width="0.3048" layer="1"/>
+<wire x1="64.9478" y1="41.2496" x2="65.0748" y2="41.19" width="0.3048" layer="1"/>
 </signal>
 <signal name="CLK_2">
@@
 <wire x1="32.3342" y1="39.9288" x2="29.591" y2="39.9288" width="0.3048" layer="1"/>
 <wire x1="33.613" y1="38.65" x2="32.3342" y2="39.9288" width="0.3048" layer="1"/>
-<wire x1="33.613" y1="38.65" x2="64.9732" y2="38.65" width="0.3048" layer="1"/>
+<wire x1="33.613" y1="38.65" x2="65.0748" y2="38.65" width="0.3048" layer="1"/>
 </signal>
 <signal name="TX2_P">
