File: spdif/spdif_B.sch (EAGLE design)
At the start: 85 parts, among them J1 PINHD-3X7/90, J2 PINHD-3X7/90, T1 DA101MC, T2 DA101MC, U1 NC7SZ175, U2 FIN1001, U3 FIN1002, U4 NC7SZ175, U5 NC7SZ175, U6 FIN1002, U7 FIN1002, U8 FIN1001, U9 FIN1002

Commit message: spdif: final tweaks
Signed-off-by: malo <pavol.malosek@gmail.com>
Parts:
- added C17: 10u, rcl:C-EUC0805
- added FB3: (no value), 25cmsquare:L0603(1608)
- added TP16, TP17, TP18, TP19, TP20: TPB1,27, testpad:TPB1,27
Connections:
- removed net +1V0: U$2_PWR.VCC6
- removed net +2V5: U$2_PWR.VCC7
- removed net +5V: U$2_PWR.VCC9
- new net N$14: J1.10, TP17.TP
- new net N$18: J1.13, TP18.TP
- new net N$19: J1.16, TP19.TP
- new net N$22: J1.19, TP20.TP
- new net N$23: FB3.1, U$2_PWR.VCC8
- net +3V3: now also C17.2, FB3.2; no longer U$2_PWR.VCC8
- net GND: now also C17.1
- net N$10: now also TP16.TP
Other:
- note removed: "digikey: 1080-1433-ND PLR135/T10 Fiber Optic Receiver General Data Transfer 16Mbps 1.45 1080-1430-ND PLT133/T10W Fiber Optic Transmitter with Driver 660nm 16Mbps 1.03 CP-1401-ND RCJ-012 3.20mm ID, 9.00mm OD (RCA) Phono (RCA) Jack 0.75 CP-1403-ND RCJ-014 3.20mm ID, 9.00mm OD (RCA) Phono (RCA) Jack 0.75 FIN1002M5XCT-ND FIN1002M5X 0/1 Receiver LVDS SOT-23-5 0.45 FIN1001M5XCT-ND FIN1001M5X 1/0 Driver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"
- moved on the sheet: U$2_PWR
Changed lines of the file:
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@@
 <part name="GND17" library="supply1" deviceset="GND" device=""/>
 <part name="D1" library="25cmsquare" deviceset="ZD" device="PESD0603-240" value="PESD0603-240"/>
-<part name="+2V1" library="25cmsquare" deviceset="+2V5" device=""/>
-<part name="U$1" library="25cmsquare" deviceset="+1V0" device=""/>
 <part name="+3V10" library="supply1" deviceset="+3V3" device=""/>
-<part name="P+1" library="supply1" deviceset="+5V" device=""/>
 <part name="GND19" library="supply1" deviceset="GND" device=""/>
 <part name="U6" library="25cmsquare" deviceset="FIN1002" device=""/>
@@
 <part name="C16" library="rcl" deviceset="C-EU" device="C0603" value="100n, 0603"/>
 <part name="GND39" library="supply1" deviceset="GND" device=""/>
+<part name="TP16" library="testpad" deviceset="TP" device="B1,27"/>
+<part name="TP17" library="testpad" deviceset="TP" device="B1,27"/>
+<part name="TP18" library="testpad" deviceset="TP" device="B1,27"/>
+<part name="TP19" library="testpad" deviceset="TP" device="B1,27"/>
+<part name="TP20" library="testpad" deviceset="TP" device="B1,27"/>
+<part name="C17" library="rcl" deviceset="C-EU" device="C0805" value="10u"/>
+<part name="FB3" library="25cmsquare" deviceset="L" device="0603(1608)"/>
+<part name="GND40" library="supply1" deviceset="GND" device=""/>
 </parts>
 <sheets>
@@
 <plain>
 <text x="170.18" y="10.16" size="5.08" layer="94">16.11.22.B</text>
-<text x="266.7" y="134.62" size="1.778" layer="94">digikey:
-1080-1433-ND             PLR135/T10          Fiber Optic Receiver General Data Transfer 16Mbps   1.45
-1080-1430-ND             PLT133/T10W       Fiber Optic Transmitter with Driver 660nm 16Mbps 1.03
-CP-1401-ND                RCJ-012               3.20mm ID, 9.00mm OD (RCA) Phono (RCA) Jack                 0.75
-CP-1403-ND                RCJ-014               3.20mm ID, 9.00mm OD (RCA) Phono (RCA) Jack                 0.75
-FIN1002M5XCT-ND      FIN1002M5X        0/1 Receiver LVDS SOT-23-5  0.45
-FIN1001M5XCT-ND      FIN1001M5X        1/0 Driver LVDS SOT-23-5   0.66
-NC7SZ175P6XCT-ND    NC7SZ175P6X       IC D-TYPE POS TRG SNGL SC70-6  0.32
-811-3122-1-ND           DA101MC- R         DIGITAL AUDIO TX   0.96</text>
 </plain>
 <instances>
@@
 <attribute name="VALUE" x="36.449" y="26.162" size="1.778" layer="96" rot="R90"/>
 </instance>
-<instance part="+2V1" gate="G$1" x="58.42" y="157.48" smashed="yes" rot="R270">
-<attribute name="VALUE" x="60.96" y="157.48" size="1.778" layer="96"/>
-</instance>
-<instance part="U$1" gate="A" x="50.8" y="154.94" smashed="yes" rot="R270">
-<attribute name="VALUE" x="53.34" y="154.94" size="1.778" layer="96"/>
-</instance>
-<instance part="+3V10" gate="G$1" x="53.34" y="160.02" smashed="yes" rot="R270">
-<attribute name="VALUE" x="53.34" y="160.02" size="1.778" layer="96"/>
-</instance>
-<instance part="P+1" gate="1" x="53.34" y="162.56" smashed="yes" rot="R270">
-<attribute name="VALUE" x="53.34" y="162.56" size="1.778" layer="96"/>
+<instance part="+3V10" gate="G$1" x="63.5" y="160.02" smashed="yes" rot="R270">
+<attribute name="VALUE" x="63.5" y="160.02" size="1.778" layer="96"/>
 </instance>
 <instance part="GND19" gate="1" x="7.62" y="154.94"/>
@@
 <instance part="GND18" gate="1" x="170.18" y="127"/>
 <instance part="J1" gate="G$1" x="182.88" y="149.86"/>
-<instance part="U$2" gate="_PWR" x="25.4" y="154.94" rot="R180"/>
+<instance part="U$2" gate="_PWR" x="20.32" y="154.94" rot="R180"/>
 <instance part="U$2" gate="_IO" x="99.06" y="152.4" rot="R180"/>
 <instance part="U8" gate="G$1" x="203.2" y="86.36" smashed="yes">
@@
 <instance part="TP14" gate="G$1" x="228.6" y="91.44"/>
 <instance part="TP15" gate="G$1" x="228.6" y="81.28" rot="R180"/>
+<instance part="TP17" gate="G$1" x="149.86" y="149.86" rot="R90"/>
+<instance part="TP18" gate="G$1" x="160.02" y="144.78" rot="R90"/>
+<instance part="TP19" gate="G$1" x="152.4" y="139.7" rot="R90"/>
+<instance part="TP20" gate="G$1" x="157.48" y="134.62" rot="R90"/>
+<instance part="C17" gate="G$1" x="58.42" y="152.4" rot="R180"/>
+<instance part="FB3" gate="G$1" x="48.26" y="160.02" smashed="yes" rot="R90">
+<attribute name="NAME" x="45.72" y="163.83" size="1.778" layer="95"/>
+<attribute name="VALUE" x="53.34" y="163.83" size="1.778" layer="96" rot="R180"/>
+</instance>
+<instance part="GND40" gate="1" x="58.42" y="142.24"/>
 </instances>
 <busses>
@@
 </segment>
 <segment>
-<wire x1="15.24" y1="160.02" x2="7.62" y2="160.02" width="0.1524" layer="91"/>
+<wire x1="10.16" y1="160.02" x2="7.62" y2="160.02" width="0.1524" layer="91"/>
 <pinref part="GND19" gate="1" pin="GND"/>
 <wire x1="7.62" y1="160.02" x2="7.62" y2="157.48" width="0.1524" layer="91"/>
@@
 <pinref part="GND37" gate="1" pin="GND"/>
 </segment>
+<segment>
+<pinref part="C17" gate="G$1" pin="1"/>
+<pinref part="GND40" gate="1" pin="GND"/>
+<wire x1="58.42" y1="144.78" x2="58.42" y2="149.86" width="0.1524" layer="91"/>
+</segment>
 </net>
 <net name="+3V3" class="0">
@@
 </segment>
 <segment>
-<wire x1="43.18" y1="160.02" x2="50.8" y2="160.02" width="0.1524" layer="91"/>
-<pinref part="+3V10" gate="G$1" pin="+3V3"/>
-<pinref part="U$2" gate="_PWR" pin="VCC8"/>
-</segment>
-<segment>
 <pinref part="+3V11" gate="G$1" pin="+3V3"/>
 <wire x1="162.56" y1="93.98" x2="162.56" y2="99.06" width="0.1524" layer="91"/>
@@
 <wire x1="205.74" y1="99.06" x2="200.66" y2="99.06" width="0.1524" layer="91"/>
 <junction x="200.66" y="99.06"/>
+</segment>
+<segment>
+<pinref part="C17" gate="G$1" pin="2"/>
+<wire x1="58.42" y1="157.48" x2="58.42" y2="160.02" width="0.1524" layer="91"/>
+<wire x1="58.42" y1="160.02" x2="60.96" y2="160.02" width="0.1524" layer="91"/>
+<pinref part="FB3" gate="G$1" pin="2"/>
+<wire x1="55.88" y1="160.02" x2="58.42" y2="160.02" width="0.1524" layer="91"/>
+<junction x="58.42" y="160.02"/>
+<pinref part="+3V10" gate="G$1" pin="+3V3"/>
 </segment>
 </net>
@@
 </segment>
 </net>
-<net name="+2V5" class="0">
-<segment>
-<pinref part="+2V1" gate="G$1" pin="+2V5"/>
-<wire x1="43.18" y1="157.48" x2="58.42" y2="157.48" width="0.1524" layer="91"/>
-<pinref part="U$2" gate="_PWR" pin="VCC7"/>
-</segment>
-</net>
-<net name="+1V0" class="0">
-<segment>
-<wire x1="43.18" y1="154.94" x2="50.8" y2="154.94" width="0.1524" layer="91"/>
-<pinref part="U$1" gate="A" pin="+1V0"/>
-<pinref part="U$2" gate="_PWR" pin="VCC6"/>
-</segment>
-</net>
-<net name="+5V" class="0">
-<segment>
-<wire x1="43.18" y1="162.56" x2="50.8" y2="162.56" width="0.1524" layer="91"/>
-<pinref part="P+1" gate="1" pin="+5V"/>
-<pinref part="U$2" gate="_PWR" pin="VCC9"/>
-</segment>
-</net>
 <net name="U6_OUT" class="0">
 <segment>
@@
 <label x="195.58" y="165.1" size="1.778" layer="95" xref="yes"/>
 <pinref part="J1" gate="G$1" pin="3"/>
+</segment>
+</net>
+<net name="N$14" class="0">
+<segment>
+<pinref part="TP17" gate="G$1" pin="TP"/>
+<pinref part="J1" gate="G$1" pin="10"/>
+<wire x1="152.4" y1="149.86" x2="175.26" y2="149.86" width="0.1524" layer="91"/>
+</segment>
+</net>
+<net name="N$18" class="0">
+<segment>
+<pinref part="TP18" gate="G$1" pin="TP"/>
+<pinref part="J1" gate="G$1" pin="13"/>
+<wire x1="162.56" y1="144.78" x2="175.26" y2="144.78" width="0.1524" layer="91"/>
+</segment>
+</net>
+<net name="N$19" class="0">
+<segment>
+<pinref part="TP19" gate="G$1" pin="TP"/>
+<pinref part="J1" gate="G$1" pin="16"/>
+<wire x1="154.94" y1="139.7" x2="175.26" y2="139.7" width="0.1524" layer="91"/>
+</segment>
+</net>
+<net name="N$22" class="0">
+<segment>
+<pinref part="TP20" gate="G$1" pin="TP"/>
+<pinref part="J1" gate="G$1" pin="19"/>
+<wire x1="160.02" y1="134.62" x2="175.26" y2="134.62" width="0.1524" layer="91"/>
+</segment>
+</net>
+<net name="N$23" class="0">
+<segment>
+<pinref part="FB3" gate="G$1" pin="1"/>
+<wire x1="40.64" y1="160.02" x2="38.1" y2="160.02" width="0.1524" layer="91"/>
+<pinref part="U$2" gate="_PWR" pin="VCC8"/>
 </segment>
 </net>
@@
 </instance>
 <instance part="GND39" gate="1" x="10.16" y="129.54" rot="R180"/>
+<instance part="TP16" gate="G$1" x="22.86" y="142.24"/>
 </instances>
 <busses>
@@
 <pinref part="U1" gate="&gt;NAME" pin="D"/>
 <wire x1="20.32" y1="129.54" x2="20.32" y2="139.7" width="0.1524" layer="91"/>
-<wire x1="20.32" y1="139.7" x2="35.56" y2="139.7" width="0.1524" layer="91"/>
+<wire x1="20.32" y1="139.7" x2="22.86" y2="139.7" width="0.1524" layer="91"/>
+<pinref part="TP16" gate="G$1" pin="TP"/>
+<wire x1="22.86" y1="139.7" x2="35.56" y2="139.7" width="0.1524" layer="91"/>
+<junction x="22.86" y="139.7"/>
 </segment>
 </net>
@@
 </schematic>
 </drawing>
-<compatibility>
-<note version="6.3" minversion="6.2.2" severity="warning">
-Since Version 6.2.2 text objects can contain more than one line,
-which will not be processed correctly with this version.
-</note>
-</compatibility>
 </eagle>
