File: xpower/xpower_A.brd (EAGLE design)
At the start: 50 x 50 mm, 34 parts, among them U1 TLV70233, U2 TLV70225, U3 STM1061N29, U4 ADM1085, U5 LM3674-ADJ

Commit message: xpower: finished PCB.
Signed-off-by: malo <pavol.malosek@gmail.com>
Parts:
- added JP1: (no value), pinhead:1X02
- added POR: TPTP14R, testpad:TP14R
- moved 5V0 86.0 mm to (38.1, 40.8)
- moved 2V5 60.5 mm to (39.1, 9.27)
- moved 3V3 51.8 mm to (10.9, 21.6)
- moved 1V0 34.7 mm to (14.0, 4.57)
- moved GND 3.68 mm to (38.1, 37.3)
- renumbered TP1 to PG_3V3
Connections:
- net +5V: now also JP1.2
- net GND: now also JP1.1
- net POR: now also POR.TP
Routing:
- net +5V: track 135.0 -> 152.3 mm
- net +1V0: track 63.2 -> 65.6 mm
- net +3V3: track 46.2 -> 48.2 mm
- net +2V5: track 51.6 -> 53.4 mm
- net GND: vias 35 -> 38
Other:
- board text added: "16.10.22.A"
- board text added: "1V0"
- board text added: "25"
- board text added: "25cm"
- board text added: "2V5"
- board text added: "3V3"
- board text added: "5V0"
- board text added: "D_N"
- board text added: "D_P"
- board text added: "POR"
- board text added: "square.io"

Commit message: xpower: minor beautifications
Signed-off-by: malo <pavol.malosek@gmail.com>
Parts:
- C11: value 0.1u, 0805 -> 100n, 0805
Changed lines of the file:
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@@
 <attribute name="NAME" x="16.383" y="17.526" size="1.016" layer="25" font="vector" ratio="15"/>
 </element>
-<element name="C11" library="rcl" package="C0805" value="0.1u, 0805" x="22.733" y="31.877" smashed="yes" rot="R90">
+<element name="C11" library="rcl" package="C0805" value="100n, 0805" x="22.733" y="31.877" smashed="yes" rot="R90">
 <attribute name="NAME" x="21.59" y="28.956" size="1.016" layer="25" font="vector" ratio="15"/>
 </element>
