File: xpower/xpower_B.sch (EAGLE design)
At the start: 41 parts, among them U1 TLV70233, U2 TLV70225, U3 STM1061N29, U4 ADM1085, U5 LM3674-ADJ

Commit message: xpower: B variant PCB finished
Signed-off-by: malo <pavol.malosek@gmail.com>
Parts:
- removed PWR1: (no value), 25cmsquare:LIWE_12_PIN_PWR8X8_COMPAT
- added JP_1V0_IN, JP_2V5_IN, JP_3V3_IN: (no value), pinhead:PINHD-1X2
- added U$1: LIWE_40_PIN, 25cmsquare:LIWE_40_PIN
- C1, C7: value 1u, 0805 -> 1u, 0603; device rcl:C-EUC0805 -> rcl:C-EUC0603
- C10, C2: value 2u2, 0805 -> 2u2, 0603; device rcl:C-EUC0805 -> rcl:C-EUC0603
- C11, C15, C4, C6: value 100n, 0805 -> 100n, 0603; device rcl:C-EUC0805 -> rcl:C-EUC0603
- C12: value 2n2, 0805 -> 2n2, 0603; device rcl:C-EUC0805 -> rcl:C-EUC0603
- C13: value 4.7u, 0805 -> 4.7u, 0603; device rcl:C-EUC0805 -> rcl:C-EUC0603
- C14: value 10u, 0805 -> 10u, 0603; device rcl:C-EUC0805 -> rcl:C-EUC0603
- C3: value 18p, 0805 -> 18p, 0603; device rcl:C-EUC0805 -> rcl:C-EUC0603
- C9: value 4.7n, 0805 -> 4.7n, 0603; device rcl:C-EUC0805 -> rcl:C-EUC0603
- R1, R2: value 200k, 0805 -> 200k, 0603; device rcl:R-EU_R0805 -> rcl:R-EU_R0603
- R3: value 330, 0805 -> 330, 0603; device rcl:R-EU_R0805 -> rcl:R-EU_R0603
- R4, R6, R7: value 10k, 0805 -> 10k, 0603; device rcl:R-EU_R0805 -> rcl:R-EU_R0603
- R5: value 3k9, 0805 -> 3k9, 0603; device rcl:R-EU_R0805 -> rcl:R-EU_R0603
- R8: value 1M, 0805 -> 1M, 0603; device rcl:R-EU_R0805 -> rcl:R-EU_R0603
- renumbered J1V0 to JP_1V0_OUT, J3V3 to JP_3V3_OUT
Connections:
- new net N$1: C1.1, JP_2V5_IN.1, U2.EN, U2.VIN
- new net N$2: C7.1, JP_3V3_IN.1, U1.EN, U1.VIN
- new net N$3: C13.1, JP_1V0_IN.1, U5.VIN
- net +1V0: now also U$1_PWR.VCC6; no longer PWR1.2
- net +2V5: now also U$1_PWR.VCC7; no longer PWR1.1
- net +3V3: now also U$1_PWR.VCC8; no longer PWR1.4
- net +5V: now also JP_1V0_IN.2, JP_2V5_IN.2, JP_3V3_IN.2, U$1_PWR.VCC9; no longer C1.1, C13.1, C7.1, PWR1.6, U1.EN, U1.VIN, U2.EN, U2.VIN, U5.VIN
- net D_N: now also U$1_IO.USB_DN; no longer PWR1.9
- net D_P: now also U$1_IO.USB_DP; no longer PWR1.10
- net GND: now also U$1_PWR.GND6, U$1_PWR.GND7, U$1_PWR.GND8, U$1_PWR.GND9; no longer PWR1.3, PWR1.8
- net POR: now also U$1_IO.IO0; no longer PWR1.7
Other:
- moved on the sheet: C1, C10, C13, C14, C2, C3, C7, C9, L1, R1, R2, R3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
