File: xpower/xpower_B.sch (EAGLE design)
At the start: 44 parts, among them U1 TLV70233, U2 TLV70225, U3 STM1061N29, U4 ADM1085, U5 LM3674-ADJ

Commit message: xpower: final tweaks
Signed-off-by: malo <pavol.malosek@gmail.com>
Parts:
- renumbered 1V0 to +1V0, 2V5 to +2V5, 3V3 to +3V3, 5V0 to +5V0
Other:
- note removed: "10x 1828827 GRM21BR71A105KA01L SMD Multilayer Ceramic Capacitor, 0805 1 µF, 10 V £0.0422 10x 1828923 GRM21BR71A225KA01L SMD Multilayer Ceramic Capacitor, 0805 2.2 µF, 10 V £0.0772 10x 1856422 MCSH21B104K100CT SMD Multilayer Ceramic Capacitor, 0805 0.1 µF, 10 V £0.0466 10x 1759420 MC0805X475K100CT SMD Multilayer Ceramic Capacitor, 0805 4.7 µF, 10 V £0.0547 10x 1828828 GRM21BR71A106KE51L SMD Multil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"
- note removed: "2323652 TLV70233DBVT 3.3V 300mA LDO Voltage Regulators 0.385 2455665 TLV70225DBVT LDO VOLTAGE REGULATOR, FIXED, 2.5V, 300mA 0.422 1312587 LM3674MF-ADJ DC-DC Switching Buck (Step Down) Regulator, Adjustable 1.09 1224452 STM1061N29WX6F Voltage Detector, Active-Low Reset 0.604 1838906 ADM1085AKSZ-REEL7 Sequencer, 2.25V-3.6Vin 0.363 2408020 LPS3015-222MRB Surface Mount Power Inductor 1.66"
- note removed: "This work is licensed under a Creative Commons Attribution-ShareAlike 4.0 International License. http://creativecommons.org/licenses/by-sa/4.0/"
- note removed: "http://25cmsquare.io"
- moved on the sheet: C11, C12, C4, JPG_3V3, JP_1V0_OUT, JP_3V3_OUT, PG_3V3, POR, R4, R5, R6, R7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
