File: xcore/xcore_A.sch (EAGLE design)
At the start: 11 parts, among them J1 PINHD-3X13/90, J2 PINHD-3X13/90, U1 NC7WZ07, X1 XEF216-512-TQ128

Commit message: xcore: WIP schema
Signed-off-by: malo <pavol.malosek@gmail.com>
Parts:
- removed J2: PINHD-3X13/90, 25pinhead:PINHD-3X13/90
- added J0: PINHD-3X13/90, 25pinhead:PINHD-3X13/90
- added R6: 0, 0603, rcl:R-EU_R0603
- added R7: 43R2, 0603, rcl:R-EU_R0603
- added TPID: TPB1,27, testpad:TPB1,27
- R4, R5: value 33, 0603 -> 33R, 0603
- XTAG: value (none) -> 2-1761605-7
Connections:
- net N$2 renamed TRST_N
- removed net D_N: PWR1.9
- removed net D_P: PWR1.10
- new net N$15: J1.28
- new net N$16: J1.31
- new net N$17: J1.34
- new net N$18: J1.37
- new net N$7: R7.1, X1_USB.USB_RTUNE
- new net USB_DN: PWR1.9, X1_USB.USB_DN
- new net USB_DP: PWR1.10, X1_USB.USB_DP
- new net USB_ID: TPID.TP, X1_USB.USB_ID
- new net USB_VBUS: R6.1, X1_USB.USB_VBUS
- new net X0D00: J0.1, X1_TILE_0_IO.X0D00
- new net X0D01: J0.4, X1_TILE_0_IO.X0D01
- new net X0D02: J0.24, X1_TILE_0_IO.X0D02
- new net X0D03: J0.27, X1_TILE_0_IO.X0D03
- new net X0D04: J0.12, X1_TILE_0_IO.X0D04
- new net X0D05: J0.15, X1_TILE_0_IO.X0D05
- new net X0D06: J0.18, X1_TILE_0_IO.X0D06
- new net X0D07: J0.21, X1_TILE_0_IO.X0D07
- new net X0D08: J0.30, X1_TILE_0_IO.X0D08
- new net X0D09: J0.33, X1_TILE_0_IO.X0D09
- new net X0D10: J0.7, X1_TILE_0_IO.X0D10
- new net X0D11: J0.10, X1_TILE_0_IO.X0D11
- new net X0D12: J0.13, X1_TILE_0_IO.X0D12
- new net X0D13: J0.16, X1_TILE_0_IO.X0D13
- new net X0D22: J0.19, X1_TILE_0_IO.X0D22
- new net X0D23: J0.22, X1_TILE_0_IO.X0D23
- new net X0D24: J0.25, X1_TILE_0_IO.X0D24
- new net X0D25: J0.28, X1_TILE_0_IO.X0D25
- new net X0D34: J0.31, X1_TILE_0_IO.X0D34
- new net X0D35: J0.34, X1_TILE_0_IO.X0D35
- new net X0D36: J0.37, X1_TILE_0_IO.X0D36
- new net X0D37: J0.3, X1_TILE_0_IO.X0D37
- new net X0D38: J0.6, X1_TILE_0_IO.X0D38
- new net X0D39: J0.9, X1_TILE_0_IO.X0D39
- new net X1D00: J1.1, X1_TILE_1_IO.X1D00
- new net X1D01: J1.4, X1_TILE_1_IO.X1D01
- new net X1D10: J1.7, X1_TILE_1_IO.X1D10
- new net X1D11: J1.10, X1_TILE_1_IO.X1D11
- new net X1D35: J1.13, X1_TILE_1_IO.X1D35
- new net X1D36: J1.16, X1_TILE_1_IO.X1D36
- new net X1D37: J1.19, X1_TILE_1_IO.X1D37
- new net X1D38: J1.22, J1.25, X1_TILE_1_IO.X1D38
- new net X1D39: X1_TILE_1_IO.X1D39
- net +5V: now also R6.2
- net GND: now also J0.11, J0.14, J0.17, J0.2, J0.20, J0.23, J0.26, J0.29, J0.32, J0.35, J0.38, J0.5, J0.8, J1.11, J1.14, J1.17, J1.2, J1.20, J1.23, J1.26, J1.29, J1.32, J1.35, J1.38, J1.5, J1.8, R7.2
Other:
- moved on the sheet: J1, R4, R5, X1_POWER, X1_TILE_0_IO, X1_TILE_1_IO, X1_USB, XTAG

Commit message: xcore: WIP jtag chaining.
Signed-off-by: malo <pavol.malosek@gmail.com>
Parts:
- added CLK: (no value), 25pinhead:PINHD-1X2/90
- added TDO: (no value), 25pinhead:PINHD-1X3
- renumbered J0 to J_TO_MASTER, J1 to J_TO_SLAVE
Connections:
- removed net X0D02: J_TO_MASTER.24, X1_TILE_0_IO.X0D02
- removed net X0D03: J_TO_MASTER.27, X1_TILE_0_IO.X0D03
- removed net X0D08: J_TO_MASTER.30, X1_TILE_0_IO.X0D08
- removed net X0D09: J_TO_MASTER.33, X1_TILE_0_IO.X0D09
- new net N$10: J_TO_MASTER.24
- new net N$2: CLK.1, PWR1.5
- new net TDO_IN: J_TO_SLAVE.30, TDO.1
- new net TDO_OUT: J_TO_MASTER.30, TDO.2
- net CLK: now also CLK.2; no longer PWR1.5
- net TCK: now also J_TO_MASTER.36, J_TO_SLAVE.36
- net TDI: now also J_TO_MASTER.27, J_TO_SLAVE.27
- net TDO: now also TDO.3
- net TMS: now also J_TO_MASTER.33, J_TO_SLAVE.33
- net XSYS_RST_N: now also J_TO_MASTER.39, J_TO_SLAVE.39
Other:
- note added: "Place R4 and R5 close to the device."

Commit message: xcore: WIP power & decoupling
Signed-off-by: malo <pavol.malosek@gmail.com>
Parts:
- added C1, C10, C11, C12, C13, C14, C15, C16, C17, C18, C19, C20, C21, C22, C23, C24, C25, C3, C5, C6: 100n, 0603, rcl:C-EUC0603
- added R8: 4R7, 0603, rcl:R-EU_R0603
Connections:
- removed net N$10: J_TO_MASTER.24
- new net N$11: C1.2, R8.2, X1_POWER.PLL_AVDD
- net +1V0: now also C10.2, C11.2, C12.2, C13.2, C14.2, C15.2, C16.2, C17.2, C18.2, C19.2, C20.2, C21.2, R8.1, X1_POWER.USB_VDD, X1_POWER.VDD
- net +2V5: now also C3.2, X1_POWER.VDDIOT
- net +3V3: now also C22.2, C23.2, C24.2, C25.2, C5.2, C6.2, X1_POWER.OTP_VCC, X1_POWER.USB_VDD33, X1_POWER.VDDIOL, X1_POWER.VDDIOR
- net GND: now also C1.1, C10.1, C11.1, C12.1, C13.1, C14.1, C15.1, C16.1, C17.1, C18.1, C19.1, C20.1, C21.1, C22.1, C23.1, C24.1, C25.1, C3.1, C5.1, C6.1, X1_POWER.GND, X1_POWER.PLL_AGND
Other:
- moved on the sheet: R6, R7, TPID, X1_POWER, X1_USB

Commit message: xcore: updated with LIWE 7x7 and 3x21 pin header
Signed-off-by: malo <pavol.malosek@gmail.com>
Parts:
- removed PWR1: (no value), 25cmsquare:LIWE_12_PIN_PWR
- added PWR: (no value), 25cmsquare:LIWE_12_PIN_PWR7X7_COMPAT
- J_TO_MASTER, J_TO_SLAVE: value PINHD-3X13/90 -> PINHD-3X21/90; device 25pinhead:PINHD-3X13/90 -> 25pinhead:PINHD-3X21/90
Connections:
- removed net N$15: J_TO_SLAVE.28
- removed net N$16: J_TO_SLAVE.31
- removed net N$17: J_TO_SLAVE.34
- removed net N$18: J_TO_SLAVE.37
- net +1V0: now also PWR.2; no longer PWR1.2
- net +2V5: now also PWR.1; no longer PWR1.1
- net +3V3: now also PWR.4; no longer PWR1.4
- net +5V: now also PWR.6; no longer PWR1.6
- net GND: now also J_TO_MASTER.41, J_TO_MASTER.44, J_TO_MASTER.47, J_TO_MASTER.50, J_TO_MASTER.53, J_TO_MASTER.56, J_TO_MASTER.59, J_TO_MASTER.62, J_TO_SLAVE.41, J_TO_SLAVE.44, J_TO_SLAVE.47, J_TO_SLAVE.50, J_TO_SLAVE.53, J_TO_SLAVE.56, J_TO_SLAVE.59, J_TO_SLAVE.62, PWR.3, PWR.8; no longer PWR1.3, PWR1.8
- net N$2: now also PWR.5; no longer PWR1.5
- net POR: now also PWR.7; no longer PWR1.7
- net SCL: now also PWR.11; no longer PWR1.11
- net SDA: now also PWR.12; no longer PWR1.12
- net TCK: now also J_TO_MASTER.60, J_TO_SLAVE.60; no longer J_TO_MASTER.36, J_TO_SLAVE.36
- net TDI: now also J_TO_MASTER.51, J_TO_SLAVE.51; no longer J_TO_MASTER.27, J_TO_SLAVE.27
- net TDO_IN: now also J_TO_SLAVE.54; no longer J_TO_SLAVE.30
- net TDO_OUT: now also J_TO_MASTER.54; no longer J_TO_MASTER.30
- net TMS: now also J_TO_MASTER.57, J_TO_SLAVE.57; no longer J_TO_MASTER.33, J_TO_SLAVE.33
- net USB_DN: now also PWR.9; no longer PWR1.9
- net USB_DP: now also PWR.10; no longer PWR1.10
- net XSYS_RST_N: now also J_TO_MASTER.63, J_TO_SLAVE.63; no longer J_TO_MASTER.39, J_TO_SLAVE.39
Other:
- moved on the sheet: R4, R5, TDO, X1_TILE_0_IO

Commit message: xcore: part number for pinhead 3x21
Signed-off-by: malo <pavol.malosek@gmail.com>
Parts:
- J_TO_MASTER, J_TO_SLAVE: value PINHD-3X21/90 -> TSW-121-08-G-T-RA
Changed lines of the file:
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@@
 <part name="GND12" library="supply1" deviceset="GND" device=""/>
 <part name="+2V3" library="25cmsquare" deviceset="+2V5" device=""/>
-<part name="J_TO_MASTER" library="25pinhead" deviceset="PINHD-3X21" device="/90"/>
-<part name="J_TO_SLAVE" library="25pinhead" deviceset="PINHD-3X21" device="/90"/>
+<part name="J_TO_MASTER" library="25pinhead" deviceset="PINHD-3X21" device="/90" value="TSW-121-08-G-T-RA"/>
+<part name="J_TO_SLAVE" library="25pinhead" deviceset="PINHD-3X21" device="/90" value="TSW-121-08-G-T-RA"/>
 </parts>
 <sheets>

Commit message: xcore: updated PWR to LIWE_12_PIN_8X8_COMPAT
Signed-off-by: malo <pavol.malosek@gmail.com>
Parts:
- PWR: device 25cmsquare:LIWE_12_PIN_PWR7X7_COMPAT -> 25cmsquare:LIWE_12_PIN_PWR8X8_COMPAT
Changed lines of the file:
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@@
 <grid distance="0.1" unitdist="inch" unit="inch" style="lines" multiple="1" display="no" altdistance="0.01" altunitdist="inch" altunit="inch"/>
 <layers>
-<layer number="1" name="Top" color="4" fill="1" visible="no" active="no"/>
-<layer number="16" name="Bottom" color="1" fill="1" visible="no" active="no"/>
-<layer number="17" name="Pads" color="2" fill="1" visible="no" active="no"/>
-<layer number="18" name="Vias" color="2" fill="1" visible="no" active="no"/>
-<layer number="19" name="Unrouted" color="6" fill="1" visible="no" active="no"/>
-<layer number="20" name="Dimension" color="15" fill="1" visible="no" active="no"/>
-<layer number="21" name="tPlace" color="7" fill="1" visible="no" active="no"/>
-<layer number="22" name="bPlace" color="7" fill="1" visible="no" active="no"/>
-<layer number="23" name="tOrigins" color="15" fill="1" visible="no" active="no"/>
-<layer number="24" name="bOrigins" color="15" fill="1" visible="no" active="no"/>
-<layer number="25" name="tNames" color="7" fill="1" visible="no" active="no"/>
-<layer number="26" name="bNames" color="7" fill="1" visible="no" active="no"/>
-<layer number="27" name="tValues" color="7" fill="1" visible="no" active="no"/>
-<layer number="28" name="bValues" color="7" fill="1" visible="no" active="no"/>
+<layer number="1" name="Top" color="4" fill="1" visible="yes" active="no"/>
+<layer number="16" name="Bottom" color="1" fill="1" visible="yes" active="no"/>
+<layer number="17" name="Pads" color="2" fill="1" visible="yes" active="no"/>
+<layer number="18" name="Vias" color="2" fill="1" visible="yes" active="no"/>
+<layer number="19" name="Unrouted" color="6" fill="1" visible="yes" active="no"/>
+<layer number="20" name="Dimension" color="15" fill="1" visible="yes" active="no"/>
+<layer number="21" name="tPlace" color="7" fill="1" visible="yes" active="no"/>
+<layer number="22" name="bPlace" color="7" fill="1" visible="yes" active="no"/>
+<layer number="23" name="tOrigins" color="15" fill="1" visible="yes" active="no"/>
+<layer number="24" name="bOrigins" color="15" fill="1" visible="yes" active="no"/>
+<layer number="25" name="tNames" color="7" fill="1" visible="yes" active="no"/>
+<layer number="26" name="bNames" color="7" fill="1" visible="yes" active="no"/>
+<layer number="27" name="tValues" color="7" fill="1" visible="yes" active="no"/>
+<layer number="28" name="bValues" color="7" fill="1" visible="yes" active="no"/>
 <layer number="29" name="tStop" color="7" fill="3" visible="no" active="no"/>
 <layer number="30" name="bStop" color="7" fill="6" visible="no" active="no"/>
@@
 <layer number="35" name="tGlue" color="7" fill="4" visible="no" active="no"/>
 <layer number="36" name="bGlue" color="7" fill="5" visible="no" active="no"/>
-<layer number="37" name="tTest" color="7" fill="1" visible="no" active="no"/>
-<layer number="38" name="bTest" color="7" fill="1" visible="no" active="no"/>
+<layer number="37" name="tTest" color="7" fill="1" visible="yes" active="no"/>
+<layer number="38" name="bTest" color="7" fill="1" visible="yes" active="no"/>
 <layer number="39" name="tKeepout" color="4" fill="11" visible="no" active="no"/>
 <layer number="40" name="bKeepout" color="1" fill="11" visible="no" active="no"/>
@@
 <layer number="44" name="Drills" color="7" fill="1" visible="no" active="no"/>
 <layer number="45" name="Holes" color="7" fill="1" visible="no" active="no"/>
-<layer number="46" name="Milling" color="3" fill="1" visible="no" active="no"/>
-<layer number="47" name="Measures" color="7" fill="1" visible="no" active="no"/>
-<layer number="48" name="Document" color="7" fill="1" visible="no" active="no"/>
-<layer number="49" name="Reference" color="7" fill="1" visible="no" active="no"/>
-<layer number="50" name="dxf" color="7" fill="1" visible="no" active="no"/>
-<layer number="51" name="tDocu" color="7" fill="1" visible="no" active="no"/>
-<layer number="52" name="bDocu" color="7" fill="1" visible="no" active="no"/>
-<layer number="53" name="tGND_GNDA" color="7" fill="9" visible="no" active="no"/>
-<layer number="54" name="bGND_GNDA" color="1" fill="9" visible="no" active="no"/>
-<layer number="56" name="wert" color="7" fill="1" visible="no" active="no"/>
-<layer number="57" name="tCAD" color="7" fill="1" visible="no" active="no"/>
-<layer number="59" name="Invisible" color="7" fill="1" visible="no" active="no"/>
-<layer number="61" name="stand" color="7" fill="1" visible="no" active="no"/>
+<layer number="46" name="Milling" color="3" fill="1" visible="yes" active="no"/>
+<layer number="47" name="Measures" color="7" fill="1" visible="yes" active="no"/>
+<layer number="48" name="Document" color="7" fill="1" visible="yes" active="no"/>
+<layer number="49" name="Reference" color="7" fill="1" visible="yes" active="no"/>
+<layer number="50" name="dxf" color="7" fill="1" visible="yes" active="no"/>
+<layer number="51" name="tDocu" color="7" fill="1" visible="yes" active="no"/>
+<layer number="52" name="bDocu" color="7" fill="1" visible="yes" active="no"/>
+<layer number="53" name="tGND_GNDA" color="7" fill="9" visible="yes" active="no"/>
+<layer number="54" name="bGND_GNDA" color="1" fill="9" visible="yes" active="no"/>
+<layer number="56" name="wert" color="7" fill="1" visible="yes" active="no"/>
+<layer number="57" name="tCAD" color="7" fill="1" visible="yes" active="no"/>
+<layer number="59" name="Invisible" color="7" fill="1" visible="yes" active="no"/>
+<layer number="61" name="stand" color="7" fill="1" visible="yes" active="no"/>
 <layer number="90" name="Modules" color="5" fill="1" visible="yes" active="yes"/>
 <layer number="91" name="Nets" color="2" fill="1" visible="yes" active="yes"/>
@@
 <parts>
 <part name="X1" library="25cmsquare" deviceset="XEF216-512-TQ128" device="" value="XEF216-512-TQ128"/>
-<part name="PWR" library="25cmsquare" deviceset="LIWE_12_PIN_PWR" device="7X7_COMPAT"/>
+<part name="PWR" library="25cmsquare" deviceset="LIWE_12_PIN_PWR" device="8X8_COMPAT"/>
 <part name="FRAME1" library="frames" deviceset="A3L-LOC" device=""/>
 <part name="XTAG" library="25pinhead" deviceset="PINHD-2X10" device="/90" value="2-1761605-7"/>

Commit message: xcore: WIP PCB
Signed-off-by: malo <pavol.malosek@gmail.com>
Parts:
- removed C5, C6: 100n, 0603, rcl:C-EUC0603
- added C26, C27, C28: 100n, 0603, rcl:C-EUC0603K
- C10, C11, C12, C13, C14, C16, C17, C18, C22, C23, C24, C25: device rcl:C-EUC0603 -> rcl:C-EUC0603K
- CLK: device 25pinhead:PINHD-1X2/90 -> 25pinhead:PINHD-1X2
- J_TO_MASTER, J_TO_SLAVE: value TSW-121-08-G-T-RA -> TSW-125-08-G-T-RA; device 25pinhead:PINHD-3X21/90 -> 25pinhead:PINHD-3X25/90
Connections:
- net N$1 renamed X0D43
- net N$11 renamed PLL_AVDD
- net N$2 renamed IO1
- net N$3 renamed X0D42
- net N$7 renamed USB_RTUNE
- new net X0D02: J_TO_SLAVE.70, X1_TILE_0_IO.X0D02
- new net X0D03: J_TO_SLAVE.72, X1_TILE_0_IO.X0D03
- new net X0D08: J_TO_SLAVE.73, X1_TILE_0_IO.X0D08
- new net X0D09: J_TO_SLAVE.75, X1_TILE_0_IO.X0D09
- new net X0D14: J_TO_MASTER.69, X1_TILE_0_IO.X0D14
- new net X0D15: X1_TILE_0_IO.X0D15
- new net X0D16: J_TO_MASTER.58, X1_TILE_0_IO.X0D16
- new net X0D17: J_TO_MASTER.57, X1_TILE_0_IO.X0D17
- new net X0D18: J_TO_MASTER.55, X1_TILE_0_IO.X0D18
- new net X0D19: J_TO_MASTER.54, X1_TILE_0_IO.X0D19
- new net X0D20: J_TO_MASTER.67, X1_TILE_0_IO.X0D20
- new net X0D21: J_TO_MASTER.66, X1_TILE_0_IO.X0D21
- new net X0D26: J_TO_MASTER.31, X1_TILE_0_IO.X0D26
- new net X0D27: J_TO_MASTER.30, X1_TILE_0_IO.X0D27
- new net X0D28: J_TO_MASTER.27, X1_TILE_0_IO.X0D28
- new net X0D29: J_TO_MASTER.24, X1_TILE_0_IO.X0D29
- new net X0D30: J_TO_MASTER.22, X1_TILE_0_IO.X0D30
- new net X0D31: J_TO_MASTER.21, X1_TILE_0_IO.X0D31
- new net X0D32: J_TO_MASTER.28, X1_TILE_0_IO.X0D32
- new net X0D33: J_TO_MASTER.25, X1_TILE_0_IO.X0D33
- new net X1D02: J_TO_MASTER.52, X1_TILE_1_IO.X1D02
- new net X1D03: J_TO_MASTER.51, X1_TILE_1_IO.X1D03
- new net X1D04: J_TO_MASTER.49, X1_TILE_1_IO.X1D04
- new net X1D05: J_TO_MASTER.48, X1_TILE_1_IO.X1D05
- new net X1D06: J_TO_MASTER.46, X1_TILE_1_IO.X1D06
- new net X1D07: J_TO_MASTER.45, X1_TILE_1_IO.X1D07
- new net X1D08: J_TO_MASTER.43, X1_TILE_1_IO.X1D08
- new net X1D09: J_TO_MASTER.42, X1_TILE_1_IO.X1D09
- new net X1D14: J_TO_MASTER.75, X1_TILE_1_IO.X1D14
- new net X1D15: J_TO_MASTER.73, X1_TILE_1_IO.X1D15
- new net X1D16: J_TO_SLAVE.52, X1_TILE_1_IO.X1D16
- new net X1D17: J_TO_SLAVE.54, X1_TILE_1_IO.X1D17
- new net X1D18: J_TO_SLAVE.55, X1_TILE_1_IO.X1D18
- new net X1D19: J_TO_SLAVE.57, X1_TILE_1_IO.X1D19
- new net X1D20: J_TO_MASTER.72, X1_TILE_1_IO.X1D20
- new net X1D21: J_TO_MASTER.70, X1_TILE_1_IO.X1D21
- new net X1D26: J_TO_MASTER.13, X1_TILE_1_IO.X1D26
- new net X1D27: J_TO_MASTER.12, X1_TILE_1_IO.X1D27
- new net X1D28: J_TO_MASTER.10, X1_TILE_1_IO.X1D28
- new net X1D29: J_TO_MASTER.9, X1_TILE_1_IO.X1D29
- new net X1D30: J_TO_SLAVE.30, X1_TILE_1_IO.X1D30
- new net X1D31: J_TO_SLAVE.31, X1_TILE_1_IO.X1D31
- new net X1D32: J_TO_SLAVE.33, X1_TILE_1_IO.X1D32
- new net X1D33: J_TO_SLAVE.34, X1_TILE_1_IO.X1D33
- new net X1D40: J_TO_MASTER.19, X1_TILE_1_IO.X1D40
- new net X1D41: J_TO_MASTER.18, X1_TILE_1_IO.X1D41
- new net X1D42: J_TO_MASTER.16, X1_TILE_1_IO.X1D42
- new net X1D43: J_TO_MASTER.15, X1_TILE_1_IO.X1D43
- net +3V3: now also C26.2, C27.2, C28.2; no longer C5.2, C6.2
- net GND: now also C26.1, C27.1, C28.1, J_TO_MASTER.65, J_TO_MASTER.68, J_TO_MASTER.71, J_TO_MASTER.74, J_TO_SLAVE.65, J_TO_SLAVE.68, J_TO_SLAVE.71, J_TO_SLAVE.74; no longer C5.1, C6.1
- net TCK: now also J_TO_MASTER.6, J_TO_SLAVE.6; no longer J_TO_MASTER.60, J_TO_SLAVE.60
- net TDI: now also J_TO_MASTER.1, J_TO_SLAVE.1; no longer J_TO_MASTER.51, J_TO_SLAVE.51
- net TDO_IN: now also J_TO_SLAVE.3; no longer J_TO_SLAVE.54
- net TDO_OUT: now also J_TO_MASTER.3; no longer J_TO_MASTER.54
- net TMS: now also J_TO_MASTER.4, J_TO_SLAVE.4; no longer J_TO_MASTER.57, J_TO_SLAVE.57
- net X0D00: now also J_TO_SLAVE.61; no longer J_TO_MASTER.1
- net X0D01: now also J_TO_SLAVE.58; no longer J_TO_MASTER.4
- net X0D04: now also J_TO_SLAVE.63; no longer J_TO_MASTER.12
- net X0D05: now also J_TO_SLAVE.66; no longer J_TO_MASTER.15
- net X0D06: now also J_TO_SLAVE.67; no longer J_TO_MASTER.18
- net X0D07: now also J_TO_SLAVE.69; no longer J_TO_MASTER.21
- net X0D10: now also J_TO_SLAVE.60; no longer J_TO_MASTER.7
- net X0D11: now also J_TO_SLAVE.64; no longer J_TO_MASTER.10
- net X0D12: now also J_TO_MASTER.64; no longer J_TO_MASTER.13
- net X0D13: now also J_TO_MASTER.63; no longer J_TO_MASTER.16
- net X0D22: now also J_TO_MASTER.61; no longer J_TO_MASTER.19
- net X0D23: now also J_TO_MASTER.60; no longer J_TO_MASTER.22
- net X0D24: now also J_TO_MASTER.37; no longer J_TO_MASTER.25
- net X0D25: now also J_TO_MASTER.36; no longer J_TO_MASTER.28
- net X0D34: now also J_TO_MASTER.34; no longer J_TO_MASTER.31
- net X0D35: now also J_TO_MASTER.33; no longer J_TO_MASTER.34
- net X0D36: now also J_TO_SLAVE.39; no longer J_TO_MASTER.37
- net X0D37: now also J_TO_SLAVE.40; no longer J_TO_MASTER.3
- net X0D38: now also J_TO_SLAVE.42; no longer J_TO_MASTER.6
- net X0D39: now also J_TO_SLAVE.43; no longer J_TO_MASTER.9
- net X1D00: now also J_TO_MASTER.40; no longer J_TO_SLAVE.1
- net X1D01: now also J_TO_MASTER.39; no longer J_TO_SLAVE.4
- net X1D10: now also J_TO_SLAVE.36; no longer J_TO_SLAVE.7
- net X1D11: now also J_TO_SLAVE.37; no longer J_TO_SLAVE.10
- net X1D35: now also J_TO_SLAVE.45; no longer J_TO_SLAVE.13
- net X1D36: now also J_TO_SLAVE.46; no longer J_TO_SLAVE.16
- net X1D37: now also J_TO_SLAVE.48; no longer J_TO_SLAVE.19
- net X1D38: now also J_TO_SLAVE.49; no longer J_TO_SLAVE.22, J_TO_SLAVE.25
- net X1D39: now also J_TO_SLAVE.51
- net XSYS_RST_N: now also J_TO_MASTER.7, J_TO_SLAVE.7; no longer J_TO_MASTER.63, J_TO_SLAVE.63
Other:
- moved on the sheet: C1, R8, X1_POWER

Commit message: xcore: WIP PCB
Signed-off-by: malo <pavol.malosek@gmail.com>
Parts:
- added JP1, JP2: (no value), 25pinhead:PINHD-1X3
- C10, C11, C12, C13, C14, C16, C17, C18, C22, C23, C24, C25, C26, C27, C28: device rcl:C-EUC0603K -> rcl:C-EUC0402K
- C15, C19, C20, C21, C3: device rcl:C-EUC0603 -> rcl:C-EUC0402K
Connections:
- net X0D12: now also J_TO_MASTER.63; no longer J_TO_MASTER.64
- net X0D13: now also J_TO_MASTER.61; no longer J_TO_MASTER.63
- net X0D15: now also J_TO_MASTER.67
- net X0D16: now also J_TO_MASTER.57; no longer J_TO_MASTER.58
- net X0D17: now also J_TO_MASTER.55; no longer J_TO_MASTER.57
- net X0D18: now also J_TO_MASTER.54; no longer J_TO_MASTER.55
- net X0D19: now also J_TO_MASTER.52; no longer J_TO_MASTER.54
- net X0D20: now also J_TO_MASTER.66; no longer J_TO_MASTER.67
- net X0D21: now also J_TO_MASTER.64; no longer J_TO_MASTER.66
- net X0D22: now also J_TO_MASTER.60; no longer J_TO_MASTER.61
- net X0D23: now also J_TO_MASTER.58; no longer J_TO_MASTER.60
- net X0D24: now also J_TO_MASTER.36; no longer J_TO_MASTER.37
- net X0D25: now also J_TO_MASTER.34; no longer J_TO_MASTER.36
- net X0D26: now also J_TO_MASTER.30; no longer J_TO_MASTER.31
- net X0D27: now also J_TO_MASTER.28; no longer J_TO_MASTER.30
- net X0D28: now also J_TO_MASTER.25; no longer J_TO_MASTER.27
- net X0D29: now also J_TO_MASTER.22; no longer J_TO_MASTER.24
- net X0D30: now also J_TO_MASTER.21; no longer J_TO_MASTER.22
- net X0D31: now also J_TO_MASTER.19; no longer J_TO_MASTER.21
- net X0D32: now also J_TO_MASTER.27; no longer J_TO_MASTER.28
- net X0D33: now also J_TO_MASTER.24; no longer J_TO_MASTER.25
- net X0D34: now also J_TO_MASTER.33; no longer J_TO_MASTER.34
- net X0D35: now also J_TO_MASTER.31; no longer J_TO_MASTER.33
- net X1D00: now also J_TO_MASTER.39; no longer J_TO_MASTER.40
- net X1D01: now also J_TO_MASTER.37; no longer J_TO_MASTER.39
- net X1D02: now also J_TO_MASTER.51; no longer J_TO_MASTER.52
- net X1D03: now also J_TO_MASTER.49; no longer J_TO_MASTER.51
- net X1D04: now also J_TO_MASTER.48; no longer J_TO_MASTER.49
- net X1D05: now also J_TO_MASTER.46; no longer J_TO_MASTER.48
- net X1D06: now also J_TO_MASTER.45; no longer J_TO_MASTER.46
- net X1D07: now also J_TO_MASTER.43; no longer J_TO_MASTER.45
- net X1D08: now also J_TO_MASTER.42; no longer J_TO_MASTER.43
- net X1D09: now also J_TO_MASTER.40; no longer J_TO_MASTER.42
- net X1D26: now also J_TO_SLAVE.24; no longer J_TO_MASTER.13
- net X1D27: now also J_TO_SLAVE.25; no longer J_TO_MASTER.12
- net X1D28: now also J_TO_SLAVE.27; no longer J_TO_MASTER.10
- net X1D29: now also J_TO_SLAVE.28; no longer J_TO_MASTER.9
- net X1D40: now also J_TO_SLAVE.18; no longer J_TO_MASTER.19
- net X1D41: now also J_TO_SLAVE.19; no longer J_TO_MASTER.18
- net X1D42: now also J_TO_SLAVE.21; no longer J_TO_MASTER.16
- net X1D43: now also J_TO_SLAVE.22; no longer J_TO_MASTER.15
