File: xcore/xcore_A.sch (EAGLE design)
At the start: 40 parts, among them U1 NC7WZ07, X1 XEF216-512-TQ128

Commit message: xcore: WIP PCB
Signed-off-by: malo <pavol.malosek@gmail.com>
Parts:
- removed C23, C24, C25, C26, C27, C28: 100n, 0603, rcl:C-EUC0402K
- removed JP1, JP2: (no value), 25pinhead:PINHD-1X3
- added C31, C32, C33, C34, C35, C36, C37, C38: 100n, 0402, rcl:C-EUC0402K
- C10, C11, C12, C13, C14, C15, C16, C17, C18, C19, C20, C21, C22: value 100n, 0603 -> 100n, 0402
- XTAG: device 25pinhead:PINHD-2X10/90 -> 25pinhead:PINHD-2X10
Connections:
- net +1V0: now also C22.2
- net +3V3: now also C31.2, C32.2, C33.2, C34.2, C35.2, C36.2, C37.2, C38.2; no longer C22.2, C23.2, C24.2, C25.2, C26.2, C27.2, C28.2
- net GND: now also C31.1, C32.1, C33.1, C34.1, C35.1, C36.1, C37.1, C38.1; no longer C23.1, C24.1, C25.1, C26.1, C27.1, C28.1
Other:
- moved on the sheet: C10, C11, C12, C13, C14, C15, C16, C17, C18, C19, C20, C21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

Commit message: xcore: updated with liwe 40 8x8 device
Signed-off-by: malo <pavol.malosek@gmail.com>
Parts:
- removed PWR: (no value), 25cmsquare:LIWE_12_PIN_PWR8X8_COMPAT
- added J0: LIWE_40_PIN, 25cmsquare:LIWE_40_PIN
Connections:
- net +1V0: now also J0_PWR.VCC6; no longer PWR.2
- net +2V5: now also J0_PWR.VCC7; no longer PWR.1
- net +3V3: now also J0_PWR.VCC8; no longer PWR.4
- net +5V: now also J0_PWR.VCC9; no longer PWR.6
- net GND: now also J0_PWR.GND6, J0_PWR.GND7, J0_PWR.GND8, J0_PWR.GND9; no longer PWR.3, PWR.8
- net IO1: now also J0_IO.CLK0; no longer PWR.5
- net POR: now also J0_IO.IO0; no longer PWR.7
- net SCL: now also J0_IO.I2C0_SCL; no longer PWR.11
- net SDA: now also J0_IO.I2C0_SDA; no longer PWR.12
- net USB_DN: now also J0_IO.USB_DN; no longer PWR.9
- net USB_DP: now also J0_IO.USB_DP; no longer PWR.10
Other:
- moved on the sheet: CLK, R4, R5, X1_TILE_0_IO

Commit message: xcore: WIP PCB
Signed-off-by: malo <pavol.malosek@gmail.com>
Changed lines of the file:
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@@
 <part name="C38" library="rcl" deviceset="C-EU" device="C0402K" value="100n, 0402"/>
 <part name="J0" library="25cmsquare" deviceset="LIWE_40_PIN" device=""/>
+<part name="FRAME2" library="frames" deviceset="A4L-LOC" device=""/>
 </parts>
 <sheets>
@@
 <plain>
 <text x="300.99" y="12.7" size="3.556" layer="94">16.11.09.A</text>
-<text x="213.36" y="7.62" size="2.54" layer="94">This work is licensed under a Creative
+<text x="187.96" y="7.62" size="2.54" layer="94">This work is licensed under a Creative
 Commons Attribution-ShareAlike 4.0
 International License.
@@
 </nets>
 </sheet>
+<sheet>
+<plain>
+<text x="173.99" y="12.7" size="3.556" layer="94">16.11.09.A</text>
+<text x="60.96" y="7.62" size="2.54" layer="94" font="vector">This work is licensed under a Creative
+Commons Attribution-ShareAlike 4.0
+International License.
+http://creativecommons.org/licenses/by-sa/4.0/</text>
+<text x="215.9" y="20.32" size="2.54" layer="94">http://25cmsquare.io</text>
+</plain>
+<instances>
+<instance part="FRAME2" gate="G$1" x="0" y="0"/>
+</instances>
+<busses>
+</busses>
+<nets>
+</nets>
+</sheet>

Commit message: xcore: WIP PCB
Signed-off-by: malo <pavol.malosek@gmail.com>
Parts:
- removed CLK: (no value), 25pinhead:PINHD-1X2
- added C2, C4: 100n, 0603, rcl:C-EUC0603
- added JP1, JP2: (no value), 25pinhead:PINHD-1X3
- added R10, R11, R12, R13, R14, R15, R16, R17, R18, R19, R20, R21, R22, R23, R24, R25, R26, R27, R28: (no value), rcl:R-EU_R0603
- added R9: 1K, 0603, rcl:R-EU_R0603
- added U2, U3: FIN1002, 25cmsquare:FIN1002
- TDO: device 25pinhead:PINHD-1X3 -> 25pinhead:PINHD-2X2
Connections:
- net X_DN0 renamed XL0_IN_0
- net X_DN1 renamed XL0_IN_1
- net X_UP0 renamed XL0_OUT_0
- net X_UP1 renamed XL0_OUT_1
- removed net CLK: CLK.2, X1_SYSTEM.CLK
- removed net SCL: J0_IO.I2C0_SCL
- removed net SDA: J0_IO.I2C0_SDA
- removed net TDO_IN: J_TO_SLAVE.3, TDO.1
- removed net TDO_OUT: J_TO_MASTER.3, TDO.2
- new net CLK0: J0_IO.CLK0, JP1.3, J_TO_MASTER.13, J_TO_SLAVE.13, U2.RIN+
- new net CLK1: J0_IO.CLK1, JP1.1, J_TO_MASTER.15, J_TO_SLAVE.15, U2.RIN-
- new net CLK2: J0_IO.CLK2, JP2.3, J_TO_MASTER.10, J_TO_SLAVE.10, U3.RIN+
- new net CLK3: J0_IO.CLK3, JP2.1, J_TO_MASTER.12, J_TO_SLAVE.12, U3.RIN-
- new net CLK_A: JP1.2, U2.ROUT, X1_SYSTEM.CLK
- new net CLK_B: JP2.2, R27.1, R28.1, U3.ROUT
- new net N$1: R10.2, X1_TILE_1_IO.X1D03
- new net N$2: R11.2, X1_TILE_1_IO.X1D04
- new net N$3: R12.2, X1_TILE_1_IO.X1D05
- new net N$4: R13.2, X1_TILE_1_IO.X1D06
- new net N$5: R14.2, X1_TILE_1_IO.X1D07
- new net N$6: R20.2
- new net N$7: R19.2
- new net RX0: J0_IO.UART0_RX, R15.1
- new net RX1: J0_IO.UART1_RX, R17.1
- new net SCL0: J0_IO.I2C0_SCL, R19.1
- new net SCL1: J0_IO.I2C1_SCL, R21.1
- new net SDA0: J0_IO.I2C0_SDA, R20.1
- new net SDA1: J0_IO.I2C1_SDA, R22.1
- new net TCK_: R25.2, XTAG.9
- new net TDO_CHAIN: J_TO_MASTER.1, J_TO_SLAVE.1, TDO.3
- new net TDO_XTAG: TDO.2, TDO.4, XTAG.13
- new net TMS_: R24.2, XTAG.7
- new net TX0: J0_IO.UART0_TX, R16.1
- new net TX1: J0_IO.UART1_TX, R18.1
- new net XSYS_RST_N_: R26.2, XTAG.15
- net +3V3: now also C2.2, C4.2, R9.1, U2.VCC, U3.VCC
- net GND: now also C2.1, C4.1, U2.GND, U3.GND
- net IO1: now also J0_IO.IO1, R23.1; no longer CLK.1, J0_IO.CLK0
- net TCK: now also R25.1; no longer XTAG.9
- net TDI: now also J_TO_MASTER.3; no longer J_TO_MASTER.1, J_TO_SLAVE.1
- net TDO: now also J_TO_SLAVE.3, TDO.1; no longer TDO.3, XTAG.13
- net TMS: now also R24.1; no longer XTAG.7
- net X0D00: now also J_TO_MASTER.61; no longer J_TO_SLAVE.61
- net X0D01: now also J_TO_MASTER.58, R9.2; no longer J_TO_SLAVE.58
- net X0D02: now also J_TO_MASTER.70; no longer J_TO_SLAVE.70
- net X0D03: now also J_TO_MASTER.72; no longer J_TO_SLAVE.72
- net X0D04: now also J_TO_MASTER.63; no longer J_TO_SLAVE.63
- net X0D05: now also J_TO_MASTER.66; no longer J_TO_SLAVE.66
- net X0D06: now also J_TO_MASTER.67; no longer J_TO_SLAVE.67
- net X0D07: now also J_TO_MASTER.69; no longer J_TO_SLAVE.69
- net X0D08: now also J_TO_MASTER.73, R21.2; no longer J_TO_SLAVE.73
- net X0D09: now also J_TO_MASTER.75, R22.2; no longer J_TO_SLAVE.75
- net X0D10: now also J_TO_MASTER.60; no longer J_TO_SLAVE.60
- net X0D11: now also J_TO_MASTER.64, R28.2; no longer J_TO_SLAVE.64
- net X0D12: now also J_TO_SLAVE.63; no longer J_TO_MASTER.63
- net X0D13: now also J_TO_SLAVE.61; no longer J_TO_MASTER.61
- net X0D14: now also J_TO_SLAVE.69; no longer J_TO_MASTER.69
- net X0D15: now also J_TO_SLAVE.67; no longer J_TO_MASTER.67
- net X0D16: now also J_TO_SLAVE.57; no longer J_TO_MASTER.57
- net X0D17: now also J_TO_SLAVE.55; no longer J_TO_MASTER.55
- net X0D18: now also J_TO_SLAVE.54; no longer J_TO_MASTER.54
- net X0D19: now also J_TO_SLAVE.52; no longer J_TO_MASTER.52
- net X0D20: now also J_TO_SLAVE.66; no longer J_TO_MASTER.66
- net X0D21: now also J_TO_SLAVE.64; no longer J_TO_MASTER.64
- net X0D22: now also J_TO_SLAVE.60, R15.2; no longer J_TO_MASTER.60
- net X0D23: now also J_TO_SLAVE.58, R16.2; no longer J_TO_MASTER.58
- net X0D24: now also J_TO_SLAVE.36, R18.2; no longer J_TO_MASTER.36
- net X0D25: now also J_TO_SLAVE.34, R17.2; no longer J_TO_MASTER.34
- net X0D26: now also J_TO_SLAVE.30; no longer J_TO_MASTER.30
- net X0D27: now also J_TO_SLAVE.28; no longer J_TO_MASTER.28
- net X0D28: now also J_TO_SLAVE.25, R23.2; no longer J_TO_MASTER.25
- net X0D29: now also J_TO_SLAVE.22; no longer J_TO_MASTER.22
- net X0D30: now also J_TO_SLAVE.21; no longer J_TO_MASTER.21
- net X0D31: now also J_TO_SLAVE.19; no longer J_TO_MASTER.19
- net X0D32: now also J_TO_SLAVE.27; no longer J_TO_MASTER.27
- net X0D33: now also J_TO_SLAVE.24; no longer J_TO_MASTER.24
- net X0D34: now also J_TO_SLAVE.33; no longer J_TO_MASTER.33
- net X0D35: now also J_TO_SLAVE.31; no longer J_TO_MASTER.31
- net X0D36: now also J_TO_MASTER.39; no longer J_TO_SLAVE.39
- net X0D37: now also J_TO_MASTER.40; no longer J_TO_SLAVE.40
- net X0D38: now also J_TO_MASTER.42; no longer J_TO_SLAVE.42
- net X0D39: now also J_TO_MASTER.43; no longer J_TO_SLAVE.43
- net X1D00: now also J_TO_SLAVE.39, R27.2; no longer J_TO_MASTER.39
- net X1D01: now also J_TO_SLAVE.37; no longer J_TO_MASTER.37
- net X1D02: now also J_TO_SLAVE.51; no longer J_TO_MASTER.51
- net X1D03: now also J_TO_SLAVE.49, R10.1; no longer J_TO_MASTER.49, X1_TILE_1_IO.X1D03
- net X1D04: now also J_TO_SLAVE.48, R11.1; no longer J_TO_MASTER.48, X1_TILE_1_IO.X1D04
- net X1D05: now also J_TO_SLAVE.46, R12.1; no longer J_TO_MASTER.46, X1_TILE_1_IO.X1D05
- net X1D06: now also J_TO_SLAVE.45, R13.1; no longer J_TO_MASTER.45, X1_TILE_1_IO.X1D06
- net X1D07: now also J_TO_SLAVE.43, R14.1; no longer J_TO_MASTER.43, X1_TILE_1_IO.X1D07
- net X1D08: now also J_TO_SLAVE.42; no longer J_TO_MASTER.42
- net X1D09: now also J_TO_SLAVE.40; no longer J_TO_MASTER.40
- net X1D10: now also J_TO_MASTER.36; no longer J_TO_SLAVE.36
- net X1D11: now also J_TO_MASTER.37; no longer J_TO_SLAVE.37
- net X1D14: now also J_TO_SLAVE.75; no longer J_TO_MASTER.75
- net X1D15: now also J_TO_SLAVE.73; no longer J_TO_MASTER.73
- net X1D16: now also J_TO_MASTER.52; no longer J_TO_SLAVE.52
- net X1D17: now also J_TO_MASTER.54; no longer J_TO_SLAVE.54
- net X1D18: now also J_TO_MASTER.55; no longer J_TO_SLAVE.55
- net X1D19: now also J_TO_MASTER.57; no longer J_TO_SLAVE.57
- net X1D20: now also J_TO_SLAVE.72; no longer J_TO_MASTER.72
- net X1D21: now also J_TO_SLAVE.70; no longer J_TO_MASTER.70
- net X1D26: now also J_TO_MASTER.24; no longer J_TO_SLAVE.24
- net X1D27: now also J_TO_MASTER.25; no longer J_TO_SLAVE.25
- net X1D28: now also J_TO_MASTER.27; no longer J_TO_SLAVE.27
- net X1D29: now also J_TO_MASTER.28; no longer J_TO_SLAVE.28
- net X1D30: now also J_TO_MASTER.30; no longer J_TO_SLAVE.30
- net X1D31: now also J_TO_MASTER.31; no longer J_TO_SLAVE.31
- net X1D32: now also J_TO_MASTER.33; no longer J_TO_SLAVE.33
- net X1D33: now also J_TO_MASTER.34; no longer J_TO_SLAVE.34
- net X1D35: now also J_TO_MASTER.45; no longer J_TO_SLAVE.45
- net X1D36: now also J_TO_MASTER.46; no longer J_TO_SLAVE.46
- net X1D37: now also J_TO_MASTER.48; no longer J_TO_SLAVE.48
- net X1D38: now also J_TO_MASTER.49; no longer J_TO_SLAVE.49
- net X1D39: now also J_TO_MASTER.51; no longer J_TO_SLAVE.51
- net X1D40: now also J_TO_MASTER.18; no longer J_TO_SLAVE.18
- net X1D41: now also J_TO_MASTER.19; no longer J_TO_SLAVE.19
- net X1D42: now also J_TO_MASTER.21; no longer J_TO_SLAVE.21
- net X1D43: now also J_TO_MASTER.22; no longer J_TO_SLAVE.22
- net XSYS_RST_N: now also R26.1; no longer XTAG.15
Other:
- note added: "Place R10 and R14 close to the device."
- note added: "TBS"
- note added: "TDI"
- note added: "TDO"
- note added: "TDO_CHAIN"
- note added: "TDO_XTAG"
- note added: "TO_MASTER"
- note added: "TO_SLAVE"
- note added: "XMOS"
- note added: "XTAG"
- moved on the sheet: J0_IO, J_TO_MASTER, J_TO_SLAVE, R1, R2, R3, R4, R5, R6, R7, TPID, U1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

Commit message: xcore: WIP PCB
Signed-off-by: malo <pavol.malosek@gmail.com>
Parts:
- added R29: (no value), rcl:R-EU_R0603
Connections:
- net USB_DN renamed USB_N
- net USB_DP renamed USB_P
- removed net N$6: R20.2
- removed net N$7: R19.2
- new net IO2: J0_IO.IO2, R29.1
- net X0D14: now also R15.2
- net X0D15: now also R17.2
- net X0D20: now also R29.2
- net X0D22: now also R20.2; no longer R15.2
- net X0D23: now also R19.2; no longer R16.2
- net X0D24: no longer R18.2
- net X0D25: no longer R17.2
- net X0D26: now also R16.2
- net X0D27: now also R18.2
Other:
- note removed: "TBS"
Changed lines of the file:
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@@
 <part name="GND14" library="supply1" deviceset="GND" device=""/>
 <part name="GND15" library="supply1" deviceset="GND" device=""/>
+<part name="R29" library="rcl" deviceset="R-EU_" device="R0603"/>
 </parts>
 <sheets>
@@
 <text x="73.66" y="66.04" size="1.778" layer="94">Place R4 and R5 close to the device.</text>
 <text x="208.28" y="180.34" size="1.778" layer="94">Place R10 and R14 close to the device.</text>
-<circle x="116.84" y="167.64" radius="8.128" width="0.1524" layer="94"/>
-<text x="114.3" y="170.18" size="2.54" layer="94">TBS</text>
 </plain>
 <instances>
@@
 <instance part="GND14" gate="1" x="228.6" y="101.6"/>
 <instance part="GND15" gate="1" x="302.26" y="81.28"/>
+<instance part="R29" gate="G$1" x="104.14" y="139.7" smashed="yes">
+<attribute name="NAME" x="105.41" y="143.2814" size="1.778" layer="95" rot="R180"/>
+<attribute name="VALUE" x="107.95" y="137.922" size="1.778" layer="96" rot="R180"/>
+</instance>
 </instances>
 <busses>
@@
 </segment>
 </net>
-<net name="USB_DP" class="0">
+<net name="USB_P" class="0">
 <segment>
 <label x="38.1" y="195.58" size="1.778" layer="95" rot="R180" xref="yes"/>
@@
 </segment>
 </net>
-<net name="USB_DN" class="0">
+<net name="USB_N" class="0">
 <segment>
 <label x="81.28" y="195.58" size="1.778" layer="95" xref="yes"/>
@@
 </segment>
 <segment>
-<pinref part="R15" gate="G$1" pin="2"/>
-<wire x1="53.34" y1="167.64" x2="63.5" y2="167.64" width="0.1524" layer="91"/>
-<label x="63.5" y="167.64" size="1.778" layer="95" xref="yes"/>
+<pinref part="R20" gate="G$1" pin="2"/>
+<wire x1="109.22" y1="162.56" x2="111.76" y2="162.56" width="0.1524" layer="91"/>
+<label x="111.76" y="162.56" size="1.778" layer="95" xref="yes"/>
 </segment>
 </net>
@@
 </segment>
 <segment>
-<pinref part="R16" gate="G$1" pin="2"/>
-<wire x1="60.96" y1="162.56" x2="63.5" y2="162.56" width="0.1524" layer="91"/>
-<label x="63.5" y="162.56" size="1.778" layer="95" xref="yes"/>
+<pinref part="R19" gate="G$1" pin="2"/>
+<wire x1="101.6" y1="167.64" x2="111.76" y2="167.64" width="0.1524" layer="91"/>
+<label x="111.76" y="167.64" size="1.778" layer="95" xref="yes"/>
 </segment>
 </net>
@@
 <pinref part="J_TO_SLAVE" gate="G$1" pin="36"/>
 </segment>
-<segment>
-<pinref part="R18" gate="G$1" pin="2"/>
-<wire x1="60.96" y1="152.4" x2="63.5" y2="152.4" width="0.1524" layer="91"/>
-<label x="63.5" y="152.4" size="1.778" layer="95" xref="yes"/>
-</segment>
 </net>
 <net name="X0D25" class="0">
@@
 <label x="340.36" y="139.7" size="1.778" layer="95" rot="MR0" xref="yes"/>
 <pinref part="J_TO_SLAVE" gate="G$1" pin="34"/>
-</segment>
-<segment>
-<pinref part="R17" gate="G$1" pin="2"/>
-<wire x1="53.34" y1="157.48" x2="63.5" y2="157.48" width="0.1524" layer="91"/>
-<label x="63.5" y="157.48" size="1.778" layer="95" xref="yes"/>
 </segment>
 </net>
@@
 <pinref part="J_TO_SLAVE" gate="G$1" pin="69"/>
 </segment>
+<segment>
+<pinref part="R15" gate="G$1" pin="2"/>
+<wire x1="53.34" y1="167.64" x2="63.5" y2="167.64" width="0.1524" layer="91"/>
+<label x="63.5" y="167.64" size="1.778" layer="95" xref="yes"/>
+</segment>
 </net>
 <net name="X0D15" class="0">
@@
 <label x="340.36" y="83.82" size="1.778" layer="95" rot="R180" xref="yes"/>
 </segment>
+<segment>
+<pinref part="R17" gate="G$1" pin="2"/>
+<wire x1="53.34" y1="157.48" x2="63.5" y2="157.48" width="0.1524" layer="91"/>
+<label x="63.5" y="157.48" size="1.778" layer="95" xref="yes"/>
+</segment>
 </net>
 <net name="X0D16" class="0">
@@
 <wire x1="358.14" y1="88.9" x2="363.22" y2="88.9" width="0.1524" layer="91"/>
 </segment>
+<segment>
+<pinref part="R29" gate="G$1" pin="2"/>
+<wire x1="109.22" y1="139.7" x2="111.76" y2="139.7" width="0.1524" layer="91"/>
+<label x="111.76" y="139.7" size="1.778" layer="95" xref="yes"/>
+</segment>
 </net>
 <net name="X0D21" class="0">
@@
 <pinref part="J_TO_SLAVE" gate="G$1" pin="30"/>
 </segment>
+<segment>
+<pinref part="R16" gate="G$1" pin="2"/>
+<wire x1="60.96" y1="162.56" x2="63.5" y2="162.56" width="0.1524" layer="91"/>
+<label x="63.5" y="162.56" size="1.778" layer="95" xref="yes"/>
+</segment>
 </net>
 <net name="X0D27" class="0">
@@
 <label x="340.36" y="149.86" size="1.778" layer="95" rot="MR0" xref="yes"/>
 <pinref part="J_TO_SLAVE" gate="G$1" pin="28"/>
+</segment>
+<segment>
+<pinref part="R18" gate="G$1" pin="2"/>
+<wire x1="60.96" y1="152.4" x2="63.5" y2="152.4" width="0.1524" layer="91"/>
+<label x="63.5" y="152.4" size="1.778" layer="95" xref="yes"/>
 </segment>
 </net>
@@
 </segment>
 </net>
-<net name="N$6" class="0">
-<segment>
-<pinref part="R20" gate="G$1" pin="2"/>
-<wire x1="109.22" y1="162.56" x2="111.76" y2="162.56" width="0.1524" layer="91"/>
-<label x="111.76" y="162.56" size="1.778" layer="95" xref="yes"/>
-</segment>
-</net>
-<net name="N$7" class="0">
-<segment>
-<pinref part="R19" gate="G$1" pin="2"/>
-<wire x1="101.6" y1="167.64" x2="111.76" y2="167.64" width="0.1524" layer="91"/>
-<label x="111.76" y="167.64" size="1.778" layer="95" xref="yes"/>
-</segment>
-</net>
 <net name="TMS_" class="0">
 <segment>
@@
 </segment>
 </net>
+<net name="IO2" class="0">
+<segment>
+<pinref part="J0" gate="_IO" pin="IO2"/>
+<wire x1="78.74" y1="190.5" x2="81.28" y2="190.5" width="0.1524" layer="91"/>
+<label x="81.28" y="190.5" size="1.778" layer="95" xref="yes"/>
+</segment>
+<segment>
+<pinref part="R29" gate="G$1" pin="1"/>
+<wire x1="99.06" y1="139.7" x2="88.9" y2="139.7" width="0.1524" layer="91"/>
+<label x="88.9" y="139.7" size="1.778" layer="95" rot="R180" xref="yes"/>
+</segment>
+</net>

Commit message: xcore: WIP PCB
Signed-off-by: malo <pavol.malosek@gmail.com>
Parts:
- J_TO_MASTER: device 25pinhead:PINHD-3X25/90 -> 25pinhead:PINHD-3X25/90/M
Changed lines of the file:
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@@
 <grid distance="0.1" unitdist="inch" unit="inch" style="lines" multiple="1" display="no" altdistance="0.01" altunitdist="inch" altunit="inch"/>
 <layers>
-<layer number="1" name="Top" color="4" fill="1" visible="no" active="no"/>
-<layer number="2" name="Route2" color="1" fill="3" visible="no" active="no"/>
-<layer number="3" name="Route3" color="4" fill="3" visible="no" active="no"/>
-<layer number="14" name="Route14" color="1" fill="6" visible="no" active="no"/>
-<layer number="15" name="Route15" color="4" fill="6" visible="no" active="no"/>
-<layer number="16" name="Bottom" color="1" fill="1" visible="no" active="no"/>
-<layer number="17" name="Pads" color="2" fill="1" visible="no" active="no"/>
-<layer number="18" name="Vias" color="2" fill="1" visible="no" active="no"/>
-<layer number="19" name="Unrouted" color="6" fill="1" visible="no" active="no"/>
-<layer number="20" name="Dimension" color="15" fill="1" visible="no" active="no"/>
-<layer number="21" name="tPlace" color="7" fill="1" visible="no" active="no"/>
-<layer number="22" name="bPlace" color="7" fill="1" visible="no" active="no"/>
-<layer number="23" name="tOrigins" color="15" fill="1" visible="no" active="no"/>
-<layer number="24" name="bOrigins" color="15" fill="1" visible="no" active="no"/>
-<layer number="25" name="tNames" color="7" fill="1" visible="no" active="no"/>
-<layer number="26" name="bNames" color="7" fill="1" visible="no" active="no"/>
-<layer number="27" name="tValues" color="7" fill="1" visible="no" active="no"/>
-<layer number="28" name="bValues" color="7" fill="1" visible="no" active="no"/>
+<layer number="1" name="Top" color="4" fill="1" visible="yes" active="no"/>
+<layer number="2" name="Route2" color="1" fill="3" visible="yes" active="no"/>
+<layer number="3" name="Route3" color="4" fill="3" visible="yes" active="no"/>
+<layer number="14" name="Route14" color="1" fill="6" visible="yes" active="no"/>
+<layer number="15" name="Route15" color="4" fill="6" visible="yes" active="no"/>
+<layer number="16" name="Bottom" color="1" fill="1" visible="yes" active="no"/>
+<layer number="17" name="Pads" color="2" fill="1" visible="yes" active="no"/>
+<layer number="18" name="Vias" color="2" fill="1" visible="yes" active="no"/>
+<layer number="19" name="Unrouted" color="6" fill="1" visible="yes" active="no"/>
+<layer number="20" name="Dimension" color="15" fill="1" visible="yes" active="no"/>
+<layer number="21" name="tPlace" color="7" fill="1" visible="yes" active="no"/>
+<layer number="22" name="bPlace" color="7" fill="1" visible="yes" active="no"/>
+<layer number="23" name="tOrigins" color="15" fill="1" visible="yes" active="no"/>
+<layer number="24" name="bOrigins" color="15" fill="1" visible="yes" active="no"/>
+<layer number="25" name="tNames" color="7" fill="1" visible="yes" active="no"/>
+<layer number="26" name="bNames" color="7" fill="1" visible="yes" active="no"/>
+<layer number="27" name="tValues" color="7" fill="1" visible="yes" active="no"/>
+<layer number="28" name="bValues" color="7" fill="1" visible="yes" active="no"/>
 <layer number="29" name="tStop" color="7" fill="3" visible="no" active="no"/>
 <layer number="30" name="bStop" color="7" fill="6" visible="no" active="no"/>
@@
 <layer number="35" name="tGlue" color="7" fill="4" visible="no" active="no"/>
 <layer number="36" name="bGlue" color="7" fill="5" visible="no" active="no"/>
-<layer number="37" name="tTest" color="7" fill="1" visible="no" active="no"/>
-<layer number="38" name="bTest" color="7" fill="1" visible="no" active="no"/>
+<layer number="37" name="tTest" color="7" fill="1" visible="yes" active="no"/>
+<layer number="38" name="bTest" color="7" fill="1" visible="yes" active="no"/>
 <layer number="39" name="tKeepout" color="4" fill="11" visible="no" active="no"/>
 <layer number="40" name="bKeepout" color="1" fill="11" visible="no" active="no"/>
@@
 <layer number="44" name="Drills" color="7" fill="1" visible="no" active="no"/>
 <layer number="45" name="Holes" color="7" fill="1" visible="no" active="no"/>
-<layer number="46" name="Milling" color="3" fill="1" visible="no" active="no"/>
-<layer number="47" name="Measures" color="7" fill="1" visible="no" active="no"/>
-<layer number="48" name="Document" color="7" fill="1" visible="no" active="no"/>
-<layer number="49" name="Reference" color="7" fill="1" visible="no" active="no"/>
-<layer number="50" name="dxf" color="7" fill="1" visible="no" active="no"/>
-<layer number="51" name="tDocu" color="7" fill="1" visible="no" active="no"/>
-<layer number="52" name="bDocu" color="7" fill="1" visible="no" active="no"/>
-<layer number="53" name="tGND_GNDA" color="7" fill="9" visible="no" active="no"/>
-<layer number="54" name="bGND_GNDA" color="1" fill="9" visible="no" active="no"/>
-<layer number="56" name="wert" color="7" fill="1" visible="no" active="no"/>
-<layer number="57" name="tCAD" color="7" fill="1" visible="no" active="no"/>
-<layer number="59" name="Invisible" color="7" fill="1" visible="no" active="no"/>
-<layer number="61" name="stand" color="7" fill="1" visible="no" active="no"/>
+<layer number="46" name="Milling" color="3" fill="1" visible="yes" active="no"/>
+<layer number="47" name="Measures" color="7" fill="1" visible="yes" active="no"/>
+<layer number="48" name="Document" color="7" fill="1" visible="yes" active="no"/>
+<layer number="49" name="Reference" color="7" fill="1" visible="yes" active="no"/>
+<layer number="50" name="dxf" color="7" fill="1" visible="yes" active="no"/>
+<layer number="51" name="tDocu" color="7" fill="1" visible="yes" active="no"/>
+<layer number="52" name="bDocu" color="7" fill="1" visible="yes" active="no"/>
+<layer number="53" name="tGND_GNDA" color="7" fill="9" visible="yes" active="no"/>
+<layer number="54" name="bGND_GNDA" color="1" fill="9" visible="yes" active="no"/>
+<layer number="56" name="wert" color="7" fill="1" visible="yes" active="no"/>
+<layer number="57" name="tCAD" color="7" fill="1" visible="yes" active="no"/>
+<layer number="59" name="Invisible" color="7" fill="1" visible="yes" active="no"/>
+<layer number="61" name="stand" color="7" fill="1" visible="yes" active="no"/>
 <layer number="90" name="Modules" color="5" fill="1" visible="yes" active="yes"/>
 <layer number="91" name="Nets" color="2" fill="1" visible="yes" active="yes"/>
@@
 <part name="GND12" library="supply1" deviceset="GND" device=""/>
 <part name="+2V3" library="25cmsquare" deviceset="+2V5" device=""/>
-<part name="J_TO_MASTER" library="25pinhead" deviceset="PINHD-3X25" device="/90" value="TSW-125-08-G-T-RA"/>
+<part name="J_TO_MASTER" library="25pinhead" deviceset="PINHD-3X25" device="/90/M" value="TSW-125-08-G-T-RA"/>
 <part name="C37" library="rcl" deviceset="C-EU" device="C0402K" value="100n, 0402"/>
 <part name="J_TO_SLAVE" library="25pinhead" deviceset="PINHD-3X25" device="/90" value="TSW-125-08-G-T-RA"/>

Commit message: xcore: WIP PCB
Signed-off-by: malo <pavol.malosek@gmail.com>
Parts:
- added 1V0, 2V5, 3V3, 5V0, CLK, CLK1, CLK2, POR, RST_N: TPTP14R, testpad:TPTP14R
- added GND, GND17: TEST-22-MULTICOMP, 25cmsquare:TEST-22-MULTICOMP
Connections:
- net +1V0: now also 1V0.TP
- net +2V5: now also 2V5.TP
- net +3V3: now also 3V3.TP
- net +5V: now also 5V0.TP
- net CLK_A: now also CLK.TP
- net GND: now also GND.1, GND17.1
- net POR: now also POR.TP
- net RST_N: now also RST_N.TP
- net X0D11: now also CLK2.TP
- net X1D00: now also CLK1.TP
