File: xcore/xcore_A.sch (EAGLE design)
At the start: 77 parts, among them J0 LIWE_40_PIN, U1 NC7WZ07, U2 FIN1002, U3 FIN1002, X1 XEF216-512-TQ128

Commit message: xcore: PCB finished
Signed-off-by: malo <pavol.malosek@gmail.com>
Parts:
- renumbered CLK1 to X1D00, CLK2 to X0D11
Changed lines of the file:
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@@
 <part name="RST_N" library="testpad" deviceset="TP" device="TP14R"/>
 <part name="CLK" library="testpad" deviceset="TP" device="TP14R"/>
-<part name="CLK1" library="testpad" deviceset="TP" device="TP14R"/>
-<part name="CLK2" library="testpad" deviceset="TP" device="TP14R"/>
+<part name="X1D00" library="testpad" deviceset="TP" device="TP14R"/>
+<part name="X0D11" library="testpad" deviceset="TP" device="TP14R"/>
 </parts>
 <sheets>
@@
 <instance part="RST_N" gate="G$1" x="121.92" y="40.64"/>
 <instance part="CLK" gate="G$1" x="149.86" y="45.72"/>
-<instance part="CLK1" gate="G$1" x="228.6" y="76.2"/>
-<instance part="CLK2" gate="G$1" x="228.6" y="66.04" rot="R180"/>
+<instance part="X1D00" gate="G$1" x="228.6" y="76.2"/>
+<instance part="X0D11" gate="G$1" x="228.6" y="66.04" rot="R180"/>
 </instances>
 <busses>
@@
 <wire x1="226.06" y1="68.58" x2="228.6" y2="68.58" width="0.1524" layer="91"/>
 <label x="231.14" y="68.58" size="1.778" layer="95" xref="yes"/>
-<pinref part="CLK2" gate="G$1" pin="TP"/>
+<pinref part="X0D11" gate="G$1" pin="TP"/>
 <wire x1="228.6" y1="68.58" x2="231.14" y2="68.58" width="0.1524" layer="91"/>
 <junction x="228.6" y="68.58"/>
@@
 <wire x1="226.06" y1="73.66" x2="228.6" y2="73.66" width="0.1524" layer="91"/>
 <label x="231.14" y="73.66" size="1.778" layer="95" xref="yes"/>
-<pinref part="CLK1" gate="G$1" pin="TP"/>
+<pinref part="X1D00" gate="G$1" pin="TP"/>
 <wire x1="228.6" y1="73.66" x2="231.14" y2="73.66" width="0.1524" layer="91"/>
 <junction x="228.6" y="73.66"/>
