File: xcore/xcore_A.brd (EAGLE design)
At the start: 80 x 80 mm, 40 parts, among them J0 LIWE_40_PIN, U1 NC7WZ07, X1 XEF216-512-TQ128

Commit message: xcore: WIP PCB
Signed-off-by: malo <pavol.malosek@gmail.com>
Connections:
- net SCL: now also J0.116; no longer J0.105
- net SDA: now also J0.115; no longer J0.106
- net USB_DN: now also J0.111; no longer J0.119
- net USB_DP: now also J0.112; no longer J0.120
Routing:
- net +1V0: track 81.0 -> 112.9 mm
- net +3V3: track 130.9 -> 129.1 mm
- added copper zone on layer 15, net +3V3
Changed lines of the file:
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@@
 <setting verticaltext="up"/>
 </settings>
-<grid distance="25" unitdist="mil" unit="mil" style="lines" multiple="1" display="yes" altdistance="0.025" altunitdist="inch" altunit="inch"/>
+<grid distance="1" unitdist="mil" unit="mil" style="lines" multiple="1" display="yes" altdistance="0.025" altunitdist="inch" altunit="inch"/>
 <layers>
 <layer number="1" name="Top" color="4" fill="1" visible="yes" active="yes"/>
@@
 <layer number="42" name="bRestrict" color="1" fill="10" visible="yes" active="yes"/>
 <layer number="43" name="vRestrict" color="2" fill="10" visible="yes" active="yes"/>
-<layer number="44" name="Drills" color="7" fill="1" visible="no" active="yes"/>
+<layer number="44" name="Drills" color="7" fill="1" visible="yes" active="yes"/>
 <layer number="45" name="Holes" color="7" fill="1" visible="yes" active="yes"/>
 <layer number="46" name="Milling" color="3" fill="1" visible="yes" active="yes"/>
@@
 <board>
 <plain>
-<text x="11.43" y="1.27" size="1.27" layer="21" font="vector" ratio="15" rot="R90" align="center-left">DP</text>
+<text x="24.765" y="6.985" size="1.27" layer="21" font="vector" ratio="15" rot="R90" align="center-left">DP</text>
 <text x="8.636" y="12.065" size="1.27" layer="21" font="vector" ratio="15" align="center-left">003|002</text>
 <text x="8.636" y="14.605" size="1.27" layer="21" font="vector" ratio="15" align="center-left">007|006</text>
@@
 <text x="59.436" y="67.945" size="1.27" layer="21" font="vector" ratio="15" align="center-left">TMS|TCK</text>
 <text x="59.817" y="70.485" size="1.27" layer="21" font="vector" ratio="15" align="center-left">TDI|TDO_OUT</text>
-<text x="11.43" y="5.08" size="1.27" layer="21" font="vector" ratio="15" rot="R90" align="center-left">DN</text>
+<text x="24.765" y="9.525" size="1.27" layer="21" font="vector" ratio="15" rot="R90" align="center-left">DN</text>
 <text x="27.305" y="7.62" size="1.27" layer="21" font="vector" ratio="15" rot="R90" align="center-left">POR</text>
 <text x="37.465" y="6.985" size="1.27" layer="21" font="vector" ratio="15" rot="R90" align="center-left">CLK</text>
@@
 <wire x1="43.0022" y1="45.847" x2="44.2722" y2="47.117" width="0.4064" layer="15"/>
 <wire x1="44.2722" y1="47.117" x2="47.0916" y2="47.117" width="0.4064" layer="15"/>
-<wire x1="47.0916" y1="32.893" x2="33.2232" y2="32.893" width="0.4064" layer="15"/>
+<wire x1="45.212" y1="32.9184" x2="33.2232" y2="32.893" width="0.4064" layer="15"/>
 <wire x1="45.0088" y1="43.4594" x2="45.0088" y2="44.577" width="0.4064" layer="15"/>
 <wire x1="45.0088" y1="44.577" x2="45.212" y2="44.577" width="0.4064" layer="15"/>
@@
 <wire x1="34.29" y1="43.2816" x2="35.1028" y2="43.2816" width="0.1524" layer="1"/>
 <contactref element="J0" pad="17"/>
+<polygon width="0.1524" layer="15">
+<vertex x="34.671" y="35.4838"/>
+<vertex x="34.671" y="45.466"/>
+<vertex x="36.068" y="45.466"/>
+<vertex x="37.7444" y="45.466"/>
+<vertex x="38.7604" y="44.45"/>
+<vertex x="39.0144" y="44.196"/>
+<vertex x="43.5356" y="44.196"/>
+<vertex x="43.6372" y="44.196"/>
+<vertex x="44.958" y="45.5168"/>
+<vertex x="45.4406" y="45.5168"/>
+<vertex x="45.4406" y="44.958"/>
+<vertex x="45.4406" y="34.544"/>
+<vertex x="34.671" y="34.544"/>
+<vertex x="34.671" y="35.4584"/>
+</polygon>
 <wire x1="51.6308" y1="62.5876" x2="55.9308" y2="61.507" width="0" layer="19" extent="1-1"/>
 <wire x1="49.5046" y1="60.9736" x2="51.6308" y2="62.5876" width="0" layer="19" extent="1-1"/>
@@
 <wire x1="42.672" y1="45.939" x2="43.0022" y2="45.847" width="0" layer="19" extent="15-16"/>
 <wire x1="43.01" y1="47.5" x2="44.2722" y2="47.117" width="0" layer="19" extent="1-15"/>
-<wire x1="47.0916" y1="32.893" x2="47.51" y2="34.6" width="0" layer="19" extent="1-15"/>
+<wire x1="45.212" y1="32.9184" x2="47.51" y2="34.6" width="0" layer="19" extent="1-15"/>
 <wire x1="32.51" y1="41" x2="32.51" y2="39" width="0" layer="19" extent="1-1"/>
-<wire x1="47.5742" y1="18.6182" x2="47.0916" y2="32.893" width="0" layer="19" extent="15-15"/>
+<wire x1="47.5742" y1="18.6182" x2="45.212" y2="32.9184" width="0" layer="19" extent="15-15"/>
 <wire x1="45.085" y1="5.07" x2="47.5742" y2="18.6182" width="0" layer="19" extent="1-15"/>
 </signal>
@@
 <wire x1="33.909" y1="46.228" x2="33.909" y2="42.1894" width="1.016" layer="15"/>
 <wire x1="33.909" y1="42.1894" x2="33.909" y2="40.0304" width="1.016" layer="15"/>
-<wire x1="33.909" y1="40.0304" x2="33.909" y2="36.7284" width="1.016" layer="15"/>
+<wire x1="33.909" y1="40.0304" x2="33.909" y2="36.1696" width="1.016" layer="15"/>
 <wire x1="33.909" y1="46.228" x2="34.61" y2="46.228" width="1.016" layer="15"/>
 <wire x1="34.61" y1="46.228" x2="37.0078" y2="46.228" width="1.016" layer="15"/>
@@
 <wire x1="35.01" y1="33.7732" x2="35.0012" y2="33.782" width="0.1524" layer="1"/>
 <wire x1="34.198" y1="37.5158" x2="34.198" y2="37.0174" width="0.1524" layer="16"/>
-<wire x1="34.198" y1="37.0174" x2="33.909" y2="36.7284" width="0.1524" layer="16"/>
-<via x="33.909" y="36.7284" extent="1-16" drill="0.3048"/>
+<wire x1="34.198" y1="37.0174" x2="33.909" y2="36.1696" width="0.1524" layer="16"/>
+<via x="33.909" y="36.1696" extent="1-16" drill="0.3048"/>
 <wire x1="32.51" y1="37" x2="33.6374" y2="37" width="0.1524" layer="1"/>
-<wire x1="33.6374" y1="37" x2="33.909" y2="36.7284" width="0.1524" layer="1"/>
+<wire x1="33.6374" y1="37" x2="33.909" y2="36.1696" width="0.1524" layer="1"/>
 <wire x1="34.452" y1="40.767" x2="34.452" y2="40.3194" width="0.1524" layer="16"/>
 <via x="33.909" y="40.0304" extent="1-16" drill="0.3048"/>
@@
 <wire x1="33.8984" y1="42.2" x2="33.909" y2="42.1894" width="0.1524" layer="1"/>
 <contactref element="J0" pad="13"/>
+<wire x1="50.165" y1="5.07" x2="50.165" y2="29.8196" width="1.6764" layer="15"/>
+<wire x1="50.165" y1="29.8196" x2="46.2026" y2="33.782" width="1.6764" layer="15"/>
 <wire x1="44.61" y1="47.5" x2="45.5054" y2="51.7254" width="0" layer="19" extent="1-1"/>
-<wire x1="50.165" y1="5.07" x2="44.61" y2="32.5" width="0" layer="19" extent="1-1"/>
 </signal>
 <signal name="+5V">
@@
 <wire x1="39.01" y1="32.5" x2="39.01" y2="18.817" width="0.1524" layer="1"/>
 <wire x1="39.01" y1="18.817" x2="29.85" y2="9.657" width="0.1524" layer="1"/>
-<contactref element="J0" pad="120"/>
-<wire x1="14.605" y1="2.53" x2="29.85" y2="9.657" width="0" layer="19" extent="1-1"/>
+<contactref element="J0" pad="112"/>
+<wire x1="24.765" y1="2.53" x2="29.85" y2="9.657" width="0" layer="19" extent="1-1"/>
 </signal>
 <signal name="USB_DN">
@@
 <wire x1="39.41" y1="32.5" x2="39.41" y2="17.185" width="0.1524" layer="1"/>
 <wire x1="39.41" y1="17.185" x2="32.512" y2="10.287" width="0.1524" layer="1"/>
-<contactref element="J0" pad="119"/>
-<wire x1="14.605" y1="5.07" x2="32.512" y2="10.287" width="0" layer="19" extent="1-1"/>
+<contactref element="J0" pad="111"/>
+<wire x1="24.765" y1="5.07" x2="32.512" y2="10.287" width="0" layer="19" extent="1-1"/>
 </signal>
 <signal name="X0D00">
@@
 </signal>
 <signal name="SCL">
-<contactref element="J0" pad="105"/>
+<contactref element="J0" pad="116"/>
 </signal>
 <signal name="SDA">
-<contactref element="J0" pad="106"/>
+<contactref element="J0" pad="115"/>
 </signal>
 </signals>

Commit message: xcore: WIP PCB
Signed-off-by: malo <pavol.malosek@gmail.com>
Parts:
- removed CLK: (no value), 25pinhead:1X02
- added C2, C4: 100n, 0603, rcl:C0603
- added JP1, JP2: (no value), 25pinhead:1X03
- added R10, R11, R12, R13, R14, R15, R16, R17, R18, R19, R20, R21, R22, R23, R24, R25, R26, R27, R28: (no value), rcl:R0603
- added R9: 1K, 0603, rcl:R0603
- added U2, U3: FIN1002, 25cmsquare:SOT95P280X140-5N
- TDO: device 25pinhead:1X03 -> 25pinhead:2X02
- moved J_TO_MASTER 74.9 mm to (2.54, 40.0), flipped to the bottom
- moved J_TO_SLAVE 74.9 mm to (77.5, 40.0), flipped to the top
- moved TDO 1.92 mm to (41.0, 65.0), turned to 0 degrees
Connections:
- net X_DN0 renamed XL0_IN_0
- net X_DN1 renamed XL0_IN_1
- net X_UP0 renamed XL0_OUT_0
- net X_UP1 renamed XL0_OUT_1
- removed net CLK: CLK.2, X1.125
- removed net SCL: J0.116
- removed net SDA: J0.115
- removed net TDO_IN: J_TO_SLAVE.3, TDO.1
- removed net TDO_OUT: J_TO_MASTER.3, TDO.2
- new net CLK0: J0.101, JP1.3, J_TO_MASTER.13, J_TO_SLAVE.13, U2.3
- new net CLK1: J0.102, JP1.1, J_TO_MASTER.15, J_TO_SLAVE.15, U2.4
- new net CLK2: J0.103, JP2.3, J_TO_MASTER.10, J_TO_SLAVE.10, U3.3
- new net CLK3: J0.104, JP2.1, J_TO_MASTER.12, J_TO_SLAVE.12, U3.4
- new net CLK_A: JP1.2, U2.5, X1.125
- new net CLK_B: JP2.2, R27.1, R28.1, U3.5
- new net N$1: R10.2, X1.74
- new net N$2: R11.2, X1.75
- new net N$3: R12.2, X1.76
- new net N$4: R13.2, X1.77
- new net N$5: R14.2, X1.79
- new net N$6: R20.2
- new net N$7: R19.2
- new net RX0: J0.120, R15.1
- new net RX1: J0.118, R17.1
- new net SCL0: J0.116, R19.1
- new net SCL1: J0.114, R21.1
- new net SDA0: J0.115, R20.1
- new net SDA1: J0.113, R22.1
- new net TCK_: R25.2, XTAG.9
- new net TDO_CHAIN: J_TO_MASTER.1, J_TO_SLAVE.1, TDO.3
- new net TDO_XTAG: TDO.2, TDO.4, XTAG.13
- new net TMS_: R24.2, XTAG.7
- new net TX0: J0.119, R16.1
- new net TX1: J0.117, R18.1
- new net XSYS_RST_N_: R26.2, XTAG.15
- net +3V3: now also C2.2, C4.2, R9.1, U2.1, U3.1
- net GND: now also C2.1, C4.1, U2.2, U3.2
- net IO1: now also J0.110, R23.1; no longer CLK.1, J0.101
- net TCK: now also R25.1; no longer XTAG.9
- net TDI: now also J_TO_MASTER.3; no longer J_TO_MASTER.1, J_TO_SLAVE.1
- net TDO: now also J_TO_SLAVE.3, TDO.1; no longer TDO.3, XTAG.13
- net TMS: now also R24.1; no longer XTAG.7
- net X0D00: now also J_TO_MASTER.61; no longer J_TO_SLAVE.61
- net X0D01: now also J_TO_MASTER.58, R9.2; no longer J_TO_SLAVE.58
- net X0D02: now also J_TO_MASTER.70; no longer J_TO_SLAVE.70
- net X0D03: now also J_TO_MASTER.72; no longer J_TO_SLAVE.72
- net X0D04: now also J_TO_MASTER.63; no longer J_TO_SLAVE.63
- net X0D05: now also J_TO_MASTER.66; no longer J_TO_SLAVE.66
- net X0D06: now also J_TO_MASTER.67; no longer J_TO_SLAVE.67
- net X0D07: now also J_TO_MASTER.69; no longer J_TO_SLAVE.69
- net X0D08: now also J_TO_MASTER.73, R21.2; no longer J_TO_SLAVE.73
- net X0D09: now also J_TO_MASTER.75, R22.2; no longer J_TO_SLAVE.75
- net X0D10: now also J_TO_MASTER.60; no longer J_TO_SLAVE.60
- net X0D11: now also J_TO_MASTER.64, R28.2; no longer J_TO_SLAVE.64
- net X0D12: now also J_TO_SLAVE.63; no longer J_TO_MASTER.63
- net X0D13: now also J_TO_SLAVE.61; no longer J_TO_MASTER.61
- net X0D14: now also J_TO_SLAVE.69; no longer J_TO_MASTER.69
- net X0D15: now also J_TO_SLAVE.67; no longer J_TO_MASTER.67
- net X0D16: now also J_TO_SLAVE.57; no longer J_TO_MASTER.57
- net X0D17: now also J_TO_SLAVE.55; no longer J_TO_MASTER.55
- net X0D18: now also J_TO_SLAVE.54; no longer J_TO_MASTER.54
- net X0D19: now also J_TO_SLAVE.52; no longer J_TO_MASTER.52
- net X0D20: now also J_TO_SLAVE.66; no longer J_TO_MASTER.66
- net X0D21: now also J_TO_SLAVE.64; no longer J_TO_MASTER.64
- net X0D22: now also J_TO_SLAVE.60, R15.2; no longer J_TO_MASTER.60
- net X0D23: now also J_TO_SLAVE.58, R16.2; no longer J_TO_MASTER.58
- net X0D24: now also J_TO_SLAVE.36, R18.2; no longer J_TO_MASTER.36
- net X0D25: now also J_TO_SLAVE.34, R17.2; no longer J_TO_MASTER.34
- net X0D26: now also J_TO_SLAVE.30; no longer J_TO_MASTER.30
- net X0D27: now also J_TO_SLAVE.28; no longer J_TO_MASTER.28
- net X0D28: now also J_TO_SLAVE.25, R23.2; no longer J_TO_MASTER.25
- net X0D29: now also J_TO_SLAVE.22; no longer J_TO_MASTER.22
- net X0D30: now also J_TO_SLAVE.21; no longer J_TO_MASTER.21
- net X0D31: now also J_TO_SLAVE.19; no longer J_TO_MASTER.19
- net X0D32: now also J_TO_SLAVE.27; no longer J_TO_MASTER.27
- net X0D33: now also J_TO_SLAVE.24; no longer J_TO_MASTER.24
- net X0D34: now also J_TO_SLAVE.33; no longer J_TO_MASTER.33
- net X0D35: now also J_TO_SLAVE.31; no longer J_TO_MASTER.31
- net X0D36: now also J_TO_MASTER.39; no longer J_TO_SLAVE.39
- net X0D37: now also J_TO_MASTER.40; no longer J_TO_SLAVE.40
- net X0D38: now also J_TO_MASTER.42; no longer J_TO_SLAVE.42
- net X0D39: now also J_TO_MASTER.43; no longer J_TO_SLAVE.43
- net X1D00: now also J_TO_SLAVE.39, R27.2; no longer J_TO_MASTER.39
- net X1D01: now also J_TO_SLAVE.37; no longer J_TO_MASTER.37
- net X1D02: now also J_TO_SLAVE.51; no longer J_TO_MASTER.51
- net X1D03: now also J_TO_SLAVE.49, R10.1; no longer J_TO_MASTER.49, X1.74
- net X1D04: now also J_TO_SLAVE.48, R11.1; no longer J_TO_MASTER.48, X1.75
- net X1D05: now also J_TO_SLAVE.46, R12.1; no longer J_TO_MASTER.46, X1.76
- net X1D06: now also J_TO_SLAVE.45, R13.1; no longer J_TO_MASTER.45, X1.77
- net X1D07: now also J_TO_SLAVE.43, R14.1; no longer J_TO_MASTER.43, X1.79
- net X1D08: now also J_TO_SLAVE.42; no longer J_TO_MASTER.42
- net X1D09: now also J_TO_SLAVE.40; no longer J_TO_MASTER.40
- net X1D10: now also J_TO_MASTER.36; no longer J_TO_SLAVE.36
- net X1D11: now also J_TO_MASTER.37; no longer J_TO_SLAVE.37
- net X1D14: now also J_TO_SLAVE.75; no longer J_TO_MASTER.75
- net X1D15: now also J_TO_SLAVE.73; no longer J_TO_MASTER.73
- net X1D16: now also J_TO_MASTER.52; no longer J_TO_SLAVE.52
- net X1D17: now also J_TO_MASTER.54; no longer J_TO_SLAVE.54
- net X1D18: now also J_TO_MASTER.55; no longer J_TO_SLAVE.55
- net X1D19: now also J_TO_MASTER.57; no longer J_TO_SLAVE.57
- net X1D20: now also J_TO_SLAVE.72; no longer J_TO_MASTER.72
- net X1D21: now also J_TO_SLAVE.70; no longer J_TO_MASTER.70
- net X1D26: now also J_TO_MASTER.24; no longer J_TO_SLAVE.24
- net X1D27: now also J_TO_MASTER.25; no longer J_TO_SLAVE.25
- net X1D28: now also J_TO_MASTER.27; no longer J_TO_SLAVE.27
- net X1D29: now also J_TO_MASTER.28; no longer J_TO_SLAVE.28
- net X1D30: now also J_TO_MASTER.30; no longer J_TO_SLAVE.30
- net X1D31: now also J_TO_MASTER.31; no longer J_TO_SLAVE.31
- net X1D32: now also J_TO_MASTER.33; no longer J_TO_SLAVE.33
- net X1D33: now also J_TO_MASTER.34; no longer J_TO_SLAVE.34
- net X1D35: now also J_TO_MASTER.45; no longer J_TO_SLAVE.45
- net X1D36: now also J_TO_MASTER.46; no longer J_TO_SLAVE.46
- net X1D37: now also J_TO_MASTER.48; no longer J_TO_SLAVE.48
- net X1D38: now also J_TO_MASTER.49; no longer J_TO_SLAVE.49
- net X1D39: now also J_TO_MASTER.51; no longer J_TO_SLAVE.51
- net X1D40: now also J_TO_MASTER.18; no longer J_TO_SLAVE.18
- net X1D41: now also J_TO_MASTER.19; no longer J_TO_SLAVE.19
- net X1D42: now also J_TO_MASTER.21; no longer J_TO_SLAVE.21
- net X1D43: now also J_TO_MASTER.22; no longer J_TO_SLAVE.22
- net XSYS_RST_N: now also R26.1; no longer XTAG.15
Routing:
- net TDI: track 96.9 -> 36.3 mm
- net CLK: track 53.5 -> 0.00 mm, vias 1 -> 0
- net TDO_OUT: track 38.7 -> 0.00 mm
- net TDO_IN: track 38.1 -> 0.00 mm
- net CLK_A: track 0.00 -> 34.9 mm, vias 0 -> 1
- net X1D04: track 33.2 -> 0.00 mm
- net X1D06: track 32.5 -> 0.00 mm
- net X1D03: track 28.0 -> 0.00 mm
- net X1D05: track 27.3 -> 0.00 mm
- net X1D07: track 26.7 -> 0.00 mm
- net TDO: track 37.7 -> 19.7 mm
- net XSYS_RST_N: track 80.9 -> 72.6 mm
- net TMS: track 96.0 -> 92.4 mm
- net TCK: track 108.9 -> 106.9 mm
- net IO1: track 1.91 -> 0.00 mm
