File: xcore/xcore_A.brd (EAGLE design)
At the start: 80 x 80 mm, 65 parts, among them J0 LIWE_40_PIN, U1 NC7WZ07, U2 FIN1002, U3 FIN1002, X1 XEF216-512-TQ128

Commit message: xcore: WIP PCB
Signed-off-by: malo <pavol.malosek@gmail.com>
Parts:
- moved R28 39.6 mm to (30.2, 31.0), turned to 45 degrees
- moved R27 32.3 mm to (53.4, 39.8), turned to 180 degrees
- moved C2 28.6 mm to (44.6, 59.7), turned to 90 degrees
- moved R26 23.6 mm to (46.4, 71.4)
- moved R24 21.9 mm to (36.1, 69.1)
- moved U3 20.8 mm to (41.5, 59.7), turned to 270 degrees
- moved R25 20.4 mm to (38.7, 69.1)
- moved JP2 15.4 mm to (34.4, 59.4), turned to 180 degrees
- moved C4 9.92 mm to (26.3, 58.9), turned to 90 degrees
- moved JP1 9.56 mm to (17.1, 59.4)
- moved TDO 4.42 mm to (42.5, 69.1)
- moved U2 3.73 mm to (23.3, 59.0), turned to 270 degrees
- moved U1 3.13 mm to (51.4, 59.7)
- moved R2 3.02 mm to (47.3, 59.7), turned to 90 degrees
- moved R1 2.93 mm to (54.6, 59.7), turned to 90 degrees
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Routing:
- net CLK3: track 0.00 -> 124.8 mm, vias 0 -> 1
- net CLK1: track 0.00 -> 122.1 mm, vias 0 -> 1
- net CLK0: track 0.00 -> 116.0 mm, vias 0 -> 1
- net CLK2: track 0.00 -> 113.6 mm, vias 0 -> 1
- net CLK_B: track 0.00 -> 95.3 mm, vias 0 -> 7
- net TDO_CHAIN: track 0.00 -> 67.2 mm
- net TDO: track 19.7 -> 71.2 mm, vias 1 -> 2
- net RST_N: track 13.2 -> 40.8 mm, vias 1 -> 4
- net TDI: track 36.3 -> 63.7 mm
- net XSYS_RST_N: track 72.6 -> 93.4 mm, vias 1 -> 3
- net XL0_IN_1: track 45.3 -> 53.1 mm, vias 1 -> 2
- net TDO_XTAG: track 0.00 -> 7.13 mm
- net XL0_IN_0: track 42.9 -> 49.0 mm, vias 1 -> 2
- net TMS_: track 0.00 -> 5.08 mm, vias 0 -> 1
- net TCK_: track 0.00 -> 5.03 mm, vias 0 -> 1
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Other:
- board text added: "TDI|TDO_CHAIN"
- board text added: "TDO_CHAIN|TDO"
- board text removed: "TDI|TDO_OUT"
- board text removed: "TDO_IN|TDI"

Commit message: xcore: WIP PCB
Signed-off-by: malo <pavol.malosek@gmail.com>
Parts:
- moved R9 15.5 mm to (17.0, 23.5), turned to 270 degrees
- moved R13 3.56 mm to (56.5, 36.9)
- moved R11 3.56 mm to (56.5, 34.8)
- moved R12 3.48 mm to (53.4, 35.9)
- moved R14 3.48 mm to (53.4, 37.9)
- moved R10 3.48 mm to (53.4, 33.8)
- moved R27 0.36 mm to (53.4, 40.2)
Routing:
- net X1D04: track 0.00 -> 22.2 mm
- net X1D06: track 0.00 -> 22.0 mm
- net X1D03: track 0.00 -> 19.7 mm
- net X1D05: track 0.00 -> 19.5 mm
- net X1D07: track 0.00 -> 19.3 mm
- net N$2: track 0.00 -> 9.34 mm
- net N$4: track 0.00 -> 8.83 mm
- net N$1: track 0.00 -> 6.56 mm
- net N$3: track 0.00 -> 6.05 mm
- net N$5: track 0.00 -> 5.70 mm
- net CLK1: track 122.1 -> 123.5 mm
- net CLK0: track 116.0 -> 117.3 mm

Commit message: xcore: WIP PCB
Signed-off-by: malo <pavol.malosek@gmail.com>
Parts:
- added R29: (no value), rcl:R0603
- moved R21 14.2 mm to (31.6, 14.7)
- moved R23 12.9 mm to (35.7, 14.7)
- moved R22 8.97 mm to (33.7, 14.7)
- moved R15 4.40 mm to (19.4, 14.7)
- moved R16 4.40 mm to (21.5, 14.7)
- moved R17 4.40 mm to (23.5, 14.7)
- moved R18 2.88 mm to (25.5, 14.7)
- moved R19 2.88 mm to (27.6, 14.7)
- moved R20 2.88 mm to (29.6, 14.7)
Connections:
- net USB_DN renamed USB_N
- net USB_DP renamed USB_P
- removed net N$6: R20.2
- removed net N$7: R19.2
- new net IO2: J0.107, R29.1
- net X0D14: now also R15.2
- net X0D15: now also R17.2
- net X0D20: now also R29.2
- net X0D22: now also R20.2; no longer R15.2
- net X0D23: now also R19.2; no longer R16.2
- net X0D24: no longer R18.2
- net X0D25: no longer R17.2
- net X0D26: now also R16.2
- net X0D27: now also R18.2
Routing:
- net X0D26: track 33.0 -> 81.3 mm, vias 0 -> 2
- net X0D27: track 27.8 -> 75.8 mm, vias 0 -> 2
- net X0D28: track 26.5 -> 64.4 mm, vias 0 -> 2
- net X0D23: track 29.8 -> 63.1 mm, vias 0 -> 2
- net X0D14: track 42.9 -> 75.9 mm, vias 0 -> 2
- net X0D22: track 36.9 -> 66.4 mm, vias 0 -> 1
- net X0D15: track 36.3 -> 65.4 mm, vias 0 -> 1
- net POR: track 54.6 -> 78.2 mm
- net CLK3: track 124.8 -> 146.1 mm
- net IO1: track 0.00 -> 18.7 mm, vias 0 -> 2
- net SCL1: track 0.00 -> 18.5 mm
- net CLK2: track 113.6 -> 132.0 mm
- net CLK1: track 123.5 -> 141.2 mm
- net IO2: track 0.00 -> 16.5 mm, vias 0 -> 2
- net SCL0: track 0.00 -> 16.3 mm
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Other:
- board text added: "009|008"

Commit message: xcore: WIP PCB
Signed-off-by: malo <pavol.malosek@gmail.com>
Routing:
- net USB_N: track 39.2 -> 42.1 mm
- net X0D15: track 65.4 -> 67.5 mm, vias 1 -> 2
- net X0D22: track 66.4 -> 64.3 mm, vias 1 -> 2
- net X0D20: track 55.8 -> 57.6 mm, vias 1 -> 2
- net X0D27: track 75.8 -> 74.3 mm
- net X1D14: track 47.3 -> 48.5 mm
- net X1D15: track 40.5 -> 41.6 mm
- net X1D20: track 45.1 -> 46.0 mm
- net X0D23: track 63.1 -> 62.2 mm
- net X1D21: track 38.6 -> 39.3 mm
- net X0D26: track 81.3 -> 80.6 mm
- net X0D14: track 75.9 -> 75.3 mm

Commit message: xcore: WIP PCB
Signed-off-by: malo <pavol.malosek@gmail.com>
Parts:
- moved R1 1.70 mm to (56.3, 59.7)
- moved C31 0.25 mm to (42.4, 45.3)
- turned R8 to 90 degrees
Routing:
- net +3V3: track 131.8 -> 52.0 mm, vias 10 -> 16
- net +2V5: track 0.00 -> 71.5 mm, vias 0 -> 3
- net +5V: track 0.00 -> 25.8 mm, vias 0 -> 3
- net +1V0: track 111.6 -> 118.0 mm, vias 14 -> 15
- net XSYS_RST_N: track 93.4 -> 96.6 mm
- net CLK_B: track 94.9 -> 96.7 mm
- net PLL_AVDD: track 4.82 -> 6.44 mm
- net XL0_OUT_0: track 45.9 -> 47.0 mm
- net CLK2: track 132.0 -> 132.7 mm
- added copper zone on layer 1, net GND
Other:
- board text removed: "DN"
- board text removed: "DP"

Commit message: xcore: WIP PCB
Signed-off-by: malo <pavol.malosek@gmail.com>
Parts:
- J_TO_MASTER: device 25pinhead:3X25/90 -> 25pinhead:3X25/90/M
- moved J_TO_SLAVE 30.9 mm to (72.4, 70.5)
- moved J_TO_MASTER 30.8 mm to (7.62, 70.4), flipped to the top, turned to 90 degrees
- moved R9 0.25 mm to (17.2, 23.5)
Routing:
- net +3V3: track 52.0 -> 49.4 mm
- net GND: track 0.00 -> 1.56 mm, vias 11 -> 20
- net RST_N: track 40.8 -> 41.5 mm
Other:
- board text added: ".IO2"
- board text added: "C..1|0"
- board text added: "C..3|CLK2"
- board text added: "CL1.CL0"
- board text added: "CL3.CL2"
- board text added: "CLK0|C..1"
- board text added: "CLK2|C..3"
- board text added: "IO1.POR"
- board text added: "RX0.TX0"
- board text added: "RX1.TX1"
- board text added: "SC0.SD0"
- board text added: "SC1.SD1"
- board text added: "USP.USN"
- board text removed: "CLK"
- board text removed: "POR"

Commit message: xcore: WIP PCB
Signed-off-by: malo <pavol.malosek@gmail.com>
Parts:
- added 1V0, 2V5, 3V3, 5V0, CLK, CLK1, CLK2, POR, RST_N: TPTP14R, testpad:TP14R
- added GND, GND17: TEST-22-MULTICOMP, 25cmsquare:TEST_1MM
- moved R28 2.51 mm to (28.4, 29.3)
Connections:
- net +1V0: now also 1V0.TP
- net +2V5: now also 2V5.TP
- net +3V3: now also 3V3.TP
- net +5V: now also 5V0.TP
- net CLK_A: now also CLK.TP
- net GND: now also GND.1, GND17.1
- net POR: now also POR.TP
- net RST_N: now also RST_N.TP
- net X0D11: now also CLK2.TP
- net X1D00: now also CLK1.TP
Routing:
- net +2V5: track 71.5 -> 76.3 mm
- net RST_N: track 41.5 -> 46.1 mm
- net X0D11: track 35.5 -> 38.2 mm
- net CLK_B: track 96.7 -> 94.2 mm
- net +5V: track 25.8 -> 28.3 mm
- net +1V0: track 118.0 -> 119.9 mm, vias 15 -> 16
- net POR: track 78.2 -> 80.1 mm
- net +3V3: track 49.4 -> 50.7 mm, vias 16 -> 17
- net CLK_A: track 31.6 -> 32.8 mm
- net X1D00: track 32.5 -> 33.3 mm
Other:
- board text added: "16.11.09.A"
- board text added: "25"

Commit message: xcore: PCB finished
Signed-off-by: malo <pavol.malosek@gmail.com>
Parts:
- moved R11 1.02 mm to (57.5, 34.8)
- moved R13 1.02 mm to (57.5, 36.9)
- moved R7 0.36 mm to (40.6, 28.9)
- moved R6 0.36 mm to (37.8, 28.9)
- moved GND 0.28 mm to (70.5, 3.81)
- renumbered CLK1 to X1D00, CLK2 to X0D11
Routing:
- net RST_N: track 46.1 -> 44.4 mm
- net N$4: track 8.83 -> 9.84 mm
- net N$2: track 9.34 -> 10.4 mm
- net X1D06: track 22.0 -> 21.0 mm
- net X1D04: track 22.2 -> 21.2 mm
- net TMS: track 89.5 -> 88.8 mm
- net CLK0: track 129.7 -> 129.0 mm
- net XSYS_RST_N: track 96.6 -> 97.1 mm
- net GND: track 1.56 -> 1.79 mm, vias 20 -> 59
Other:
- board text added: "GND"
- board text added: "XEF216-512-TQ128"
