File: xcore/xcore_A.brd (EAGLE design)
At the start: 80 x 80 mm, 77 parts, among them J0 LIWE_40_PIN, U1 NC7WZ07, U2 FIN1002, U3 FIN1002, X0D11 TPTP14R, X1 XEF216-512-TQ128, X1D00 TPTP14R

Commit message: xcore: PCB final tweaks
Signed-off-by: malo <pavol.malosek@gmail.com>
Parts:
- moved J_TO_MASTER 0.05 mm to (7.62, 70.5)
Routing:
- net GND: vias 59 -> 60
