File: xclock/xclock_B.sch (EAGLE design)
At the start: 41 parts, among them J1 PINHD-3X7/90, U1 5P49V5923, U2 SI7021, U3 FIN1001, U4 FIN1001, U5 FIN1001, X1 9C-24.000MEEJ-T

Commit message: xclock: WIP B variant
Signed-off-by: malo <pavol.malosek@gmail.com>
Parts:
- removed J1: PINHD-3X7/90, 25pinhead:PINHD-3X7/90
- added J2: TSW-108-08-G-T-RA, 25pinhead:PINHD-3X8/90
- added R13: (no value), rcl:R-EU_R0603
Connections:
- new net CLKIN: J2.1, U1.CLKIN
- new net CLKINB: J2.4, U1.CLKINB
- new net CLKSEL: J2.3, U1.CLKSEL
- new net SD/OE: J2.6, R13.1, U1.SD/OE
- net GND: now also J2.11, J2.14, J2.17, J2.2, J2.20, J2.23, J2.5, J2.8, R13.2; no longer J1.1, J1.11, J1.14, J1.17, J1.2, J1.20, J1.3, J1.5, J1.8, U1.SD/OE
- net OUT0: now also J2.7, J2.9; no longer J1.4, J1.6
- net OUT0_A: now also J2.10; no longer J1.7
- net OUT0_B: now also J2.12; no longer J1.9
- net OUT1: now also J2.13, J2.15; no longer J1.10, J1.12
- net OUT1_A: now also J2.16; no longer J1.13
- net OUT1_B: now also J2.18; no longer J1.15
- net OUT2: now also J2.19, J2.21; no longer J1.16, J1.18
- net OUT2_A: now also J2.22; no longer J1.19
- net OUT2_B: now also J2.24; no longer J1.21

Commit message: xclock: WIP B variant
Parts:
- removed J2: TSW-108-08-G-T-RA, 25pinhead:PINHD-3X8/90
- removed JP1, JP2: (no value), 25pinhead:PINHD-1X3
- added C14, C15: 0.1u, rcl:C-EUC0603
- added J1: (no value), 25pinhead:PINHD-3X8/90
- added R14, R15: (no value), rcl:R-EU_R0603
Connections:
- net N$6 renamed OUT0_
- net N$8 renamed OUT1_
- net N$9 renamed OUT2_
- net OUT0_A_ renamed OUT0_P_
- net OUT0_B_ renamed OUT0_N_
- net OUT1_A_ renamed OUT1_P_
- net OUT1_B_ renamed OUT1_N_
- net OUT2_A_ renamed OUT2_P_
- net OUT2_B_ renamed OUT2_N_
- removed net N$1: JP2.2, U$1_IO.CLK2
- removed net N$2: JP1.2, U$1_IO.CLK0
- removed net OUT0_A: J2.10, JP1.1, R3.1
- removed net OUT0_B: J2.12, R4.1, U$1_IO.CLK1
- removed net OUT1_A: J2.16, JP2.1, R9.1
- removed net OUT1_B: J2.18, R10.1, U$1_IO.CLK3
- removed net OUT2_A: J2.22, R11.1
- removed net OUT2_B: J2.24, R12.1
- new net OUT0_N: J1.24, R4.1, U$1_IO.CLK1
- new net OUT0_P: J1.22, R15.2, R3.1, U$1_IO.CLK0
- new net OUT1_N: J1.3, R10.1, U$1_IO.CLK3
- new net OUT1_P: J1.1, R14.1, R9.1, U$1_IO.CLK2
- new net OUT2_N: J1.12, R12.1
- new net OUT2_P: J1.10, R11.1
- net +3V3: no longer R1.2, R2.2
- net CLKIN: now also J1.16; no longer J2.1
- net CLKINB: now also J1.15; no longer J2.4
- net CLKSEL: now also J1.13; no longer J2.3
- net GND: now also C14.1, C15.1, J1.11, J1.14, J1.17, J1.2, J1.20, J1.23, J1.5, J1.8; no longer J2.11, J2.14, J2.17, J2.2, J2.20, J2.23, J2.5, J2.8
- net OUT0: now also J1.19, J1.21, R15.1; no longer J2.7, J2.9, JP1.3
- net OUT1: now also J1.4, J1.6, R14.2; no longer J2.13, J2.15, JP2.3
- net OUT2: now also J1.7, J1.9; no longer J2.19, J2.21
- net SD/OE: now also J1.18; no longer J2.6
- net VDDA: now also C14.2, C15.2
- net VDDD: now also R1.2, R2.2

Commit message: xclock: B variant finished PCB
Signed-off-by: malo <pavol.malosek@gmail.com>
Parts:
- added GND14, VDDA, VDDD: TEST-22-MULTICOMP, 25cmsquare:TEST-22-MULTICOMP
- added SCL, SDA: (no value), 25pinhead:PINHD-1X1
Connections:
- net GND: now also GND14.1
- net SCL: now also SCL.1
- net SDA: now also SDA.1
- net VDDA: now also VDDA.1
- net VDDD: now also VDDD.1
Changed lines of the file:
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@@
 <part name="C15" library="rcl" deviceset="C-EU" device="C0603" value="0.1u"/>
 <part name="J1" library="25pinhead" deviceset="PINHD-3X8" device="/90"/>
+<part name="SCL" library="25pinhead" deviceset="PINHD-1X1" device=""/>
+<part name="SDA" library="25pinhead" deviceset="PINHD-1X1" device=""/>
+<part name="GND14" library="25cmsquare" deviceset="TEST-22-MULTICOMP" device=""/>
+<part name="GND18" library="supply1" deviceset="GND" device=""/>
+<part name="VDDD" library="25cmsquare" deviceset="TEST-22-MULTICOMP" device=""/>
+<part name="VDDA" library="25cmsquare" deviceset="TEST-22-MULTICOMP" device=""/>
 </parts>
 <sheets>
@@
 <instance part="C15" gate="G$1" x="165.1" y="78.74" rot="R180"/>
 <instance part="J1" gate="G$1" x="332.74" y="226.06"/>
+<instance part="SCL" gate="G$1" x="27.94" y="246.38" rot="R90"/>
+<instance part="SDA" gate="G$1" x="83.82" y="246.38" rot="R90"/>
+<instance part="GND14" gate="G$1" x="40.64" y="71.12" rot="MR90"/>
+<instance part="GND18" gate="1" x="40.64" y="68.58" rot="MR0"/>
+<instance part="VDDD" gate="G$1" x="68.58" y="91.44" rot="MR90"/>
+<instance part="VDDA" gate="G$1" x="160.02" y="91.44" rot="MR90"/>
 </instances>
 <busses>
@@
 <segment>
 <pinref part="U$1" gate="_IO" pin="I2C1_SDA"/>
-<wire x1="76.2" y1="236.22" x2="81.28" y2="236.22" width="0.1524" layer="91"/>
-<label x="81.28" y="236.22" size="1.778" layer="95" xref="yes"/>
+<wire x1="76.2" y1="236.22" x2="83.82" y2="236.22" width="0.1524" layer="91"/>
+<label x="88.9" y="236.22" size="1.778" layer="95" xref="yes"/>
+<pinref part="SDA" gate="G$1" pin="1"/>
+<wire x1="83.82" y1="236.22" x2="88.9" y2="236.22" width="0.1524" layer="91"/>
+<wire x1="83.82" y1="243.84" x2="83.82" y2="236.22" width="0.1524" layer="91"/>
+<junction x="83.82" y="236.22"/>
 </segment>
 </net>
@@
 </segment>
 <segment>
-<wire x1="38.1" y1="236.22" x2="33.02" y2="236.22" width="0.1524" layer="91"/>
-<label x="33.02" y="236.22" size="1.778" layer="95" rot="R180" xref="yes"/>
+<wire x1="38.1" y1="236.22" x2="27.94" y2="236.22" width="0.1524" layer="91"/>
+<label x="22.86" y="236.22" size="1.778" layer="95" rot="R180" xref="yes"/>
 <pinref part="U$1" gate="_IO" pin="I2C1_SCL"/>
+<pinref part="SCL" gate="G$1" pin="1"/>
+<wire x1="27.94" y1="236.22" x2="22.86" y2="236.22" width="0.1524" layer="91"/>
+<wire x1="27.94" y1="243.84" x2="27.94" y2="236.22" width="0.1524" layer="91"/>
+<junction x="27.94" y="236.22"/>
 </segment>
 <segment>
@@
 <pinref part="GND6" gate="1" pin="GND"/>
 </segment>
+<segment>
+<pinref part="GND14" gate="G$1" pin="1"/>
+<pinref part="GND18" gate="1" pin="GND"/>
+</segment>
 </net>
 <net name="XOUT" class="0">
@@
 <wire x1="144.78" y1="86.36" x2="154.94" y2="86.36" width="0.1524" layer="91"/>
 <pinref part="C15" gate="G$1" pin="2"/>
-<wire x1="154.94" y1="86.36" x2="165.1" y2="86.36" width="0.1524" layer="91"/>
+<wire x1="154.94" y1="86.36" x2="160.02" y2="86.36" width="0.1524" layer="91"/>
+<wire x1="160.02" y1="86.36" x2="165.1" y2="86.36" width="0.1524" layer="91"/>
 <wire x1="165.1" y1="86.36" x2="165.1" y2="83.82" width="0.1524" layer="91"/>
 <pinref part="C14" gate="G$1" pin="2"/>
 <wire x1="154.94" y1="83.82" x2="154.94" y2="86.36" width="0.1524" layer="91"/>
 <junction x="154.94" y="86.36"/>
+<pinref part="VDDA" gate="G$1" pin="1"/>
+<wire x1="160.02" y1="91.44" x2="160.02" y2="86.36" width="0.1524" layer="91"/>
+<junction x="160.02" y="86.36"/>
 </segment>
 </net>
@@
 <wire x1="60.96" y1="83.82" x2="60.96" y2="86.36" width="0.1524" layer="91"/>
 <pinref part="R8" gate="G$1" pin="2"/>
-<wire x1="60.96" y1="86.36" x2="73.66" y2="86.36" width="0.1524" layer="91"/>
+<wire x1="60.96" y1="86.36" x2="68.58" y2="86.36" width="0.1524" layer="91"/>
 <pinref part="C7" gate="G$1" pin="2"/>
+<wire x1="68.58" y1="86.36" x2="73.66" y2="86.36" width="0.1524" layer="91"/>
 <wire x1="73.66" y1="86.36" x2="86.36" y2="86.36" width="0.1524" layer="91"/>
 <wire x1="86.36" y1="86.36" x2="99.06" y2="86.36" width="0.1524" layer="91"/>
@@
 <wire x1="58.42" y1="86.36" x2="60.96" y2="86.36" width="0.1524" layer="91"/>
 <junction x="60.96" y="86.36"/>
-</segment>
-<segment>
+<pinref part="VDDD" gate="G$1" pin="1"/>
+<wire x1="68.58" y1="91.44" x2="68.58" y2="86.36" width="0.1524" layer="91"/>
+<junction x="68.58" y="86.36"/>
+</segment>
+<segment>

Commit message: xclock: final tweaks
Signed-off-by: malo <pavol.malosek@gmail.com>
Other:
- note removed: "This work is licensed under a Creative Commons Attribution-ShareAlike 4.0 International License. http://creativecommons.org/licenses/by-sa/4.0/"
- note removed: "http://25cmsquare.io"
Changed lines of the file:
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@@
 3  x xtal, 25MHz, 800-2968-1-ND
 3  x xtal, 25MHz, 887-1283-1-ND</text>
-<text x="86.36" y="5.08" size="2.54" layer="94">This work is licensed under a Creative
-Commons Attribution-ShareAlike 4.0
-International License.
-http://creativecommons.org/licenses/by-sa/4.0/</text>
-<text x="342.9" y="20.32" size="2.54" layer="94">http://25cmsquare.io</text>
 </plain>
 <instances>

Commit message: xclock: update with recent library changes + xtal cap values updated to 15p
Signed-off-by: malo <pavol.malosek@gmail.com>
Parts:
- C1, C2: value (none) -> 15p
- R10, R11, R12, R3, R4, R9: value 33 -> 0
Other:
- moved on the sheet: U$1_IO, U$1_PWR
Changed lines of the file:
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@@
 <part name="GND1" library="supply1" deviceset="GND" device=""/>
 <part name="X1" library="25cmsquare" deviceset="TXC_9C" device="" value="9C-24.000MEEJ-T"/>
-<part name="C1" library="rcl" deviceset="C-EU" device="C0603"/>
-<part name="C2" library="rcl" deviceset="C-EU" device="C0603"/>
+<part name="C1" library="rcl" deviceset="C-EU" device="C0603" value="15p"/>
+<part name="C2" library="rcl" deviceset="C-EU" device="C0603" value="15p"/>
 <part name="GND2" library="supply1" deviceset="GND" device=""/>
 <part name="GND3" library="supply1" deviceset="GND" device=""/>
@@
 <part name="GND16" library="supply1" deviceset="GND" device=""/>
 <part name="GND17" library="supply1" deviceset="GND" device=""/>
-<part name="R3" library="rcl" deviceset="R-EU_" device="R0603" value="33"/>
-<part name="R4" library="rcl" deviceset="R-EU_" device="R0603" value="33"/>
-<part name="R9" library="rcl" deviceset="R-EU_" device="R0603" value="33"/>
-<part name="R10" library="rcl" deviceset="R-EU_" device="R0603" value="33"/>
-<part name="R11" library="rcl" deviceset="R-EU_" device="R0603" value="33"/>
-<part name="R12" library="rcl" deviceset="R-EU_" device="R0603" value="33"/>
+<part name="R3" library="rcl" deviceset="R-EU_" device="R0603" value="0"/>
+<part name="R4" library="rcl" deviceset="R-EU_" device="R0603" value="0"/>
+<part name="R9" library="rcl" deviceset="R-EU_" device="R0603" value="0"/>
+<part name="R10" library="rcl" deviceset="R-EU_" device="R0603" value="0"/>
+<part name="R11" library="rcl" deviceset="R-EU_" device="R0603" value="0"/>
+<part name="R12" library="rcl" deviceset="R-EU_" device="R0603" value="0"/>
 <part name="R13" library="rcl" deviceset="R-EU_" device="R0603"/>
 <part name="GND6" library="supply1" deviceset="GND" device=""/>
@@
 <instance part="CLK1" gate="G$1" x="248.92" y="147.32"/>
 <instance part="CLK2" gate="G$1" x="248.92" y="137.16"/>
-<instance part="GND21" gate="1" x="30.48" y="165.1" rot="MR90"/>
-<instance part="+3V7" gate="G$1" x="68.58" y="165.1" smashed="yes" rot="R270">
-<attribute name="VALUE" x="68.58" y="165.1" size="1.778" layer="96"/>
+<instance part="GND21" gate="1" x="25.4" y="167.64" rot="MR90"/>
+<instance part="+3V7" gate="G$1" x="68.58" y="167.64" smashed="yes" rot="R270">
+<attribute name="VALUE" x="68.58" y="167.64" size="1.778" layer="96"/>
 </instance>
 <instance part="+3V1" gate="G$1" x="33.02" y="93.98"/>
@@
 <segment>
 <pinref part="U$1" gate="_IO" pin="I2C1_SDA"/>
-<wire x1="76.2" y1="236.22" x2="83.82" y2="236.22" width="0.1524" layer="91"/>
+<wire x1="71.12" y1="236.22" x2="83.82" y2="236.22" width="0.1524" layer="91"/>
 <label x="88.9" y="236.22" size="1.778" layer="95" xref="yes"/>
 <pinref part="SDA" gate="G$1" pin="1"/>
@@
 </segment>
 <segment>
-<wire x1="38.1" y1="236.22" x2="27.94" y2="236.22" width="0.1524" layer="91"/>
+<wire x1="33.02" y1="236.22" x2="27.94" y2="236.22" width="0.1524" layer="91"/>
 <label x="22.86" y="236.22" size="1.778" layer="95" rot="R180" xref="yes"/>
 <pinref part="U$1" gate="_IO" pin="I2C1_SCL"/>
@@
 <pinref part="GND21" gate="1" pin="GND"/>
 <pinref part="U$1" gate="_PWR" pin="GND8"/>
-<wire x1="35.56" y1="165.1" x2="33.02" y2="165.1" width="0.1524" layer="91"/>
+<wire x1="30.48" y1="167.64" x2="27.94" y2="167.64" width="0.1524" layer="91"/>
 </segment>
 <segment>
@@
 <segment>
 <pinref part="+3V7" gate="G$1" pin="+3V3"/>
-<wire x1="63.5" y1="165.1" x2="66.04" y2="165.1" width="0.1524" layer="91"/>
+<wire x1="58.42" y1="167.64" x2="66.04" y2="167.64" width="0.1524" layer="91"/>
 <pinref part="U$1" gate="_PWR" pin="VCC8"/>
 </segment>
@@
 <label x="116.84" y="223.52" size="1.778" layer="95" xref="yes"/>
 <pinref part="U$1" gate="_IO" pin="CLK2"/>
-<wire x1="76.2" y1="223.52" x2="99.06" y2="223.52" width="0.1524" layer="91"/>
+<wire x1="71.12" y1="223.52" x2="99.06" y2="223.52" width="0.1524" layer="91"/>
 <pinref part="R14" gate="G$1" pin="1"/>
 <wire x1="99.06" y1="223.52" x2="116.84" y2="223.52" width="0.1524" layer="91"/>
@@
 <label x="101.6" y="220.98" size="1.778" layer="95" xref="yes"/>
 <pinref part="U$1" gate="_IO" pin="CLK0"/>
-<wire x1="76.2" y1="220.98" x2="99.06" y2="220.98" width="0.1524" layer="91"/>
+<wire x1="71.12" y1="220.98" x2="99.06" y2="220.98" width="0.1524" layer="91"/>
 <pinref part="R15" gate="G$1" pin="2"/>
 <wire x1="99.06" y1="220.98" x2="101.6" y2="220.98" width="0.1524" layer="91"/>
@@
 <segment>
 <pinref part="U$1" gate="_IO" pin="CLK1"/>
-<wire x1="38.1" y1="220.98" x2="22.86" y2="220.98" width="0.1524" layer="91"/>
+<wire x1="33.02" y1="220.98" x2="22.86" y2="220.98" width="0.1524" layer="91"/>
 <label x="22.86" y="220.98" size="1.778" layer="95" rot="R180" xref="yes"/>
 </segment>
@@
 <segment>
 <pinref part="U$1" gate="_IO" pin="CLK3"/>
-<wire x1="38.1" y1="223.52" x2="35.56" y2="223.52" width="0.1524" layer="91"/>
+<wire x1="33.02" y1="223.52" x2="35.56" y2="223.52" width="0.1524" layer="91"/>
 <label x="35.56" y="223.52" size="1.778" layer="95" rot="R180" xref="yes"/>
 </segment>
