File: xdac/xdac_A.sch (EAGLE design)
At the start: 76 parts, among them J1 LIWE_40_PIN, J12 FC68131, J3 PINHD-3X9/90, J34 FC68131, J4 PINHD-3X5/90, J56 FC68131, J78 FC68131, U1 STA311B, U2 CS4384, U3 FIN1002

Commit message: xdac: VIP
Signed-off-by: malo <pavol.malosek@gmail.com>
Parts:
- removed CKOUT, MUTEC_1, MUTEC_234: TPB1,27, testpad:TPB1,27
- removed J4: PINHD-3X5/90, 25pinhead:PINHD-3X5/90
- removed R1: 220R, rcl:R-EU_R0603
- removed R2, R3, R4, R5, R6: 470R, rcl:R-EU_R0603
- removed U1: STA311B, 25cmsquare:STA311B
- C11, C12, C13, C14, C17, C18, C23, C24: device 25cmsquare:C-POL_D -> 25cmsquare:C-POL_C
- C15, C16, C19, C2, C20, C21, C22, C25, C26, C8, C9: device rcl:C-EUC0603K -> rcl:C-EUC0603
- J2: value (none) -> PINHD-3X5/90; device 25pinhead:PINHD-3X8/90 -> 25pinhead:PINHD-3X5/90
- J3: value PINHD-3X9/90 -> PINHD-3X5/90; device 25pinhead:PINHD-3X9/90 -> 25pinhead:PINHD-3X5/90
Connections:
- net CS_AOUT1 renamed AOUT1
- net CS_AOUT2 renamed AOUT2
- net CS_AOUT3 renamed AOUT3
- net CS_AOUT4 renamed AOUT4
- net CS_AOUT5 renamed AOUT5
- net CS_AOUT6 renamed AOUT6
- net CS_AOUT7 renamed AOUT7
- net CS_AOUT8 renamed AOUT8
- net N$13 renamed AUOT1_
- net N$14 renamed AOUT2_
- net N$23 renamed FILT+
- net N$25 renamed AOUT4_
- net N$26 renamed VQ
- net N$29 renamed AOUT3_
- net N$32 renamed AOUT6_
- net N$35 renamed AOUT5_
- net N$38 renamed AOUT8_
- net N$41 renamed AOUT7_
- removed net CS_DSD1: J2.10, U2_MAIN.DSD1
- removed net CS_DSD2: J2.12, U2_MAIN.DSD2
- removed net CS_DSD3: J2.13, U2_MAIN.DSD3
- removed net CS_DSD4: J2.15, U2_MAIN.DSD4
- removed net CS_DSD5: J2.16, U2_MAIN.DSD5
- removed net CS_DSD6: J2.18, U2_MAIN.DSD6
- removed net CS_DSD7: J2.19, U2_MAIN.DSD7
- removed net CS_DSD8: J2.21, U2_MAIN.DSD8
- removed net CS_DSD_CLK: J2.22, U2_MAIN.DSD_SCLK
- removed net CS_LRCLK: J2.3, R2.2, U2_MAIN.LRCLK
- removed net CS_RST_N: J2.24, U2_MAIN.RST_N
- removed net CS_SCLK: J2.1, R1.2, U2_MAIN.SCLK
- removed net CS_SDIN1: J2.4, R3.2, U2_MAIN.SDIN1
- removed net CS_SDIN2: J2.6, R4.2, U2_MAIN.SDIN2
- removed net CS_SDIN3: J2.7, R5.2, U2_MAIN.SDIN3
- removed net CS_SDIN4: J2.9, R6.2, U2_MAIN.SDIN4
- removed net N$1: R1.1, U1_MAIN.BICKO
- removed net N$10: CKOUT.TP, U1_MAIN.CKOUT
- removed net N$2: R2.1, U1_MAIN.LRCKO
- removed net N$3: R3.1, U1_MAIN.SDO_12
- removed net N$31: J4.15
- removed net N$4: R4.1, U1_MAIN.SDO_34
- removed net N$43: J3.27
- removed net N$5: R5.1, U1_MAIN.SDO_56
- removed net N$6: R6.1, U1_MAIN.SDO_78
- removed net N$8: MUTEC_1.TP, U2_MAIN.MUTEC_1
- removed net N$9: MUTEC_234.TP, U2_MAIN.MUTEC_234
- removed net STA_1A: J3.1, U1_MAIN.OUT_1A
- removed net STA_1B: J3.3, U1_MAIN.OUT_1B
- removed net STA_2A: J3.4, U1_MAIN.OUT_2A
- removed net STA_2B: J3.6, U1_MAIN.OUT_2B
- removed net STA_3A: J3.7, U1_MAIN.OUT_3A
- removed net STA_3B: J3.9, U1_MAIN.OUT_3B
- removed net STA_4A: J3.10, U1_MAIN.OUT_4A
- removed net STA_4B: J3.12, U1_MAIN.OUT_4B
- removed net STA_5A: J3.13, U1_MAIN.OUT_5A
- removed net STA_5B: J3.15, U1_MAIN.OUT_5B
- removed net STA_6A: J3.16, U1_MAIN.OUT_6A
- removed net STA_6B: J3.18, U1_MAIN.OUT_6B
- removed net STA_7A: J3.19, U1_MAIN.OUT_7A
- removed net STA_7B: J3.21, U1_MAIN.OUT_7B
- removed net STA_8A: J3.22, U1_MAIN.OUT_8A
- removed net STA_8B: J3.24, U1_MAIN.OUT_8B
- removed net STA_BICKI: J4.1, U1_MAIN.BICKI/DSD_1
- removed net STA_EAPD: J3.25, U1_MAIN.EAPD
- removed net STA_LRCKI: J4.3, U1_MAIN.LRCKI/DSD_2
- removed net STA_MVO: J4.10, U1_MAIN.MVO/DSD_CLK
- removed net STA_PWDN: J4.13, U1_MAIN.PWDN
- removed net STA_RST_N: J4.12, U1_MAIN.RESET_N
- removed net STA_SDI12: J4.4, U1_MAIN.SDI_12/DSD_3
- removed net STA_SDI34: J4.6, U1_MAIN.SDI_34/DSD_4
- removed net STA_SDI56: J4.7, U1_MAIN.SDI_56/DSD_5
- removed net STA_SDI78: J4.9, U1_MAIN.SDI_78/DSD_6
- new net DSD1: J2.3, U2_MAIN.DSD1
- new net DSD2: J2.1, U2_MAIN.DSD2
- new net DSD3: J2.6, U2_MAIN.DSD3
- new net DSD4: J2.4, U2_MAIN.DSD4
- new net DSD5: J2.9, U2_MAIN.DSD5
- new net DSD6: J2.7, U2_MAIN.DSD6
- new net DSD7: J2.12, U2_MAIN.DSD7
- new net DSD8: J2.10, U2_MAIN.DSD8
- new net DSD_CLK: J2.15, U2_MAIN.DSD_SCLK
- new net LRCLK: J3.3, U2_MAIN.LRCLK
- new net MUTEC_1: J2.13, U2_MAIN.MUTEC_1
- new net MUTEC_234: J3.15, U2_MAIN.MUTEC_234
- new net RST_N: J3.12, U2_MAIN.RST_N
- new net SCLK: J3.1, U2_MAIN.SCLK
- new net SDIN1: J3.4, U2_MAIN.SDIN1
- new net SDIN2: J3.6, U2_MAIN.SDIN2
- new net SDIN3: J3.7, U2_MAIN.SDIN3
- new net SDIN4: J3.9, U2_MAIN.SDIN4
- net +3V3: no longer U1_POWER.VDD
- net 3V3A: no longer U1_POWER.VDDA
- net GND: no longer J2.17, J2.20, J2.23, J3.17, J3.20, J3.23, J3.26, J4.11, J4.14, J4.2, J4.5, J4.8, U1_MAIN.RESERVED, U1_MAIN.SA, U1_POWER.GND, U1_POWER.GNDA, U1_POWER.PAD
- net MCLK: no longer U1_MAIN.XTI
- net SCL: no longer U1_MAIN.SCL
- net SDA: no longer U1_MAIN.SDA
Other:
- moved on the sheet: C1, C10, C2, C3, C4, C5, C6, C7, C8, C9, U2_MAIN, U2_POWER

Commit message: xdac: WIP
Signed-off-by: malo <pavol.malosek@gmail.com>
Parts:
- added JP1, JP3: (no value), 25pinhead:PINHD-1X2/90
- C10: value 47u, EEEFC1V470P -> 47u, EEEFC0J470R; device 25cmsquare:C-POL_E -> 25cmsquare:C-POL_C
- C4, C5: device rcl:C-EUC0603K -> rcl:C-EUC0603
Connections:
- net GND: now also JP1.1, JP3.1
- net MUTEC_1: now also JP3.2; no longer J2.13
- net MUTEC_234: now also JP1.2; no longer J3.15
Changed lines of the file:
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@@
 <?xml version="1.0" encoding="utf-8"?>
 <!DOCTYPE eagle SYSTEM "eagle.dtd">
-<eagle version="7.7.0">
+<eagle version="8.0.0">
 <drawing>
 <settings>
@@
 <part name="GND1" library="supply1" deviceset="GND" device=""/>
 <part name="C3" library="25cmsquare" deviceset="C-POL" device="_B" value="1u, EEEFC1V1R0AR"/>
-<part name="C4" library="rcl" deviceset="C-EU" device="C0603K" value="100n"/>
+<part name="C4" library="rcl" deviceset="C-EU" device="C0603" value="100n"/>
 <part name="GND2" library="supply1" deviceset="GND" device=""/>
 <part name="+2V1" library="25cmsquare" deviceset="+2V5" device=""/>
-<part name="C5" library="rcl" deviceset="C-EU" device="C0603K" value="100n"/>
+<part name="C5" library="rcl" deviceset="C-EU" device="C0603" value="100n"/>
 <part name="C6" library="rcl" deviceset="C-EU" device="C0603K" value="100n"/>
 <part name="GND3" library="supply1" deviceset="GND" device=""/>
@@
 <part name="C8" library="rcl" deviceset="C-EU" device="C0603" value="100n"/>
 <part name="GND5" library="supply1" deviceset="GND" device=""/>
-<part name="C10" library="25cmsquare" deviceset="C-POL" device="_E" value="47u, EEEFC1V470P"/>
+<part name="C10" library="25cmsquare" deviceset="C-POL" device="_C" value="47u, EEEFC0J470R"/>
 <part name="C9" library="rcl" deviceset="C-EU" device="C0603" value="100n"/>
 <part name="GND6" library="supply1" deviceset="GND" device=""/>
@@
 <part name="GND39" library="supply1" deviceset="GND" device=""/>
 <part name="J3" library="25pinhead" deviceset="PINHD-3X5" device="/90"/>
+<part name="JP1" library="25pinhead" deviceset="PINHD-1X2" device="/90"/>
+<part name="JP3" library="25pinhead" deviceset="PINHD-1X2" device="/90"/>
+<part name="GND40" library="supply1" deviceset="GND" device=""/>
+<part name="GND41" library="supply1" deviceset="GND" device=""/>
 </parts>
 <sheets>
@@
 <instance part="GND39" gate="1" x="193.04" y="208.28"/>
 <instance part="J3" gate="G$1" x="248.92" y="223.52"/>
+<instance part="JP1" gate="G$1" x="264.16" y="203.2" rot="R180"/>
+<instance part="JP3" gate="G$1" x="264.16" y="185.42" rot="R180"/>
+<instance part="GND40" gate="1" x="274.32" y="195.58"/>
+<instance part="GND41" gate="1" x="274.32" y="177.8"/>
 </instances>
 <busses>
@@
 <junction x="193.04" y="215.9"/>
 </segment>
+<segment>
+<pinref part="JP1" gate="G$1" pin="1"/>
+<wire x1="266.7" y1="200.66" x2="274.32" y2="200.66" width="0.1524" layer="91"/>
+<wire x1="274.32" y1="200.66" x2="274.32" y2="198.12" width="0.1524" layer="91"/>
+<pinref part="GND40" gate="1" pin="GND"/>
+</segment>
+<segment>
+<pinref part="JP3" gate="G$1" pin="1"/>
+<wire x1="266.7" y1="182.88" x2="274.32" y2="182.88" width="0.1524" layer="91"/>
+<wire x1="274.32" y1="182.88" x2="274.32" y2="180.34" width="0.1524" layer="91"/>
+<pinref part="GND41" gate="1" pin="GND"/>
+</segment>
 </net>
 <net name="+2V5" class="0">
@@
 </segment>
 <segment>
-<wire x1="195.58" y1="218.44" x2="190.5" y2="218.44" width="0.1524" layer="91"/>
-<label x="190.5" y="218.44" size="1.778" layer="95" rot="R180" xref="yes"/>
-<pinref part="J2" gate="G$1" pin="13"/>
+<wire x1="266.7" y1="185.42" x2="274.32" y2="185.42" width="0.1524" layer="91"/>
+<label x="274.32" y="185.42" size="1.778" layer="95" xref="yes"/>
+<pinref part="JP3" gate="G$1" pin="2"/>
 </segment>
 </net>
@@
 </segment>
 <segment>
-<wire x1="256.54" y1="218.44" x2="261.62" y2="218.44" width="0.1524" layer="91"/>
-<label x="261.62" y="218.44" size="1.778" layer="95" xref="yes"/>
-<pinref part="J3" gate="G$1" pin="15"/>
-</segment>
-</net>
+<wire x1="266.7" y1="203.2" x2="274.32" y2="203.2" width="0.1524" layer="91"/>
+<label x="274.32" y="203.2" size="1.778" layer="95" xref="yes"/>
+<pinref part="JP1" gate="G$1" pin="2"/>
+</segment>
+</net>

Commit message: xdac: VIP
Signed-off-by: malo <pavol.malosek@gmail.com>
Parts:
- added A1, A2, A3, A4, A5, A6, A7, A8, LRCLK, SCLK, SDIN1, SDIN2, SDIN3, SDIN4: (no value), 25pinhead:PINHD-1X1
- added U$1, U$2, U$3, U$4, U$5, U$6: TEST-22-MULTICOMP, 25cmsquare:TEST-22-MULTICOMP
- renumbered JP2 to MCLK
Connections:
- net CLK2 renamed CLK_P
- net CLK3 renamed CLK_N
- net AOUT1: now also A1.1
- net AOUT2: now also A2.1
- net AOUT3: now also A3.1
- net AOUT4: now also A4.1
- net AOUT5: now also A5.1
- net AOUT6: now also A6.1
- net AOUT7: now also A7.1
- net AOUT8: now also A8.1
- net GND: now also U$1.1, U$2.1, U$3.1, U$4.1, U$5.1, U$6.1
- net LRCLK: now also J3.10, LRCLK.1; no longer J3.3
- net RST_N: now also J3.3; no longer J3.12
- net SCLK: now also J3.7, SCLK.1; no longer J3.1
- net SDIN1: now also J3.9, SDIN1.1; no longer J3.4
- net SDIN2: now also SDIN2.1
- net SDIN3: now also J3.4, SDIN3.1; no longer J3.7
- net SDIN4: now also J3.1, SDIN4.1; no longer J3.9

Commit message: xdac: VIP
Signed-off-by: malo <pavol.malosek@gmail.com>
Parts:
- added +5V, 2V5, 3V3: TPTP14R, testpad:TPTP14R
Connections:
- net +2V5: now also 2V5.TP
- net +3V3: now also 3V3.TP
- net +5V: now also +5V.TP
Other:
- note added: "17.03.27.A"
Changed lines of the file:
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@@
 <?xml version="1.0" encoding="utf-8"?>
 <!DOCTYPE eagle SYSTEM "eagle.dtd">
-<eagle version="8.1.0">
+<eagle version="7.7.0">
 <drawing>
 <settings>
@@
 <part name="U$6" library="25cmsquare" deviceset="TEST-22-MULTICOMP" device=""/>
 <part name="GND47" library="supply1" deviceset="GND" device=""/>
+<part name="2V5" library="testpad" deviceset="TP" device="TP14R"/>
+<part name="+2V4" library="25cmsquare" deviceset="+2V5" device=""/>
+<part name="3V3" library="testpad" deviceset="TP" device="TP14R"/>
+<part name="+3V1" library="supply1" deviceset="+3V3" device=""/>
+<part name="P+1" library="supply1" deviceset="+5V" device=""/>
+<part name="+5V" library="testpad" deviceset="TP" device="TP14R"/>
 </parts>
 <sheets>
 <sheet>
 <plain>
+<text x="293.37" y="12.7" size="5.08" layer="94">17.03.27.A</text>
 </plain>
 <instances>
@@
 <instance part="U$6" gate="G$1" x="154.94" y="12.7"/>
 <instance part="GND47" gate="1" x="147.32" y="12.7" rot="R270"/>
+<instance part="2V5" gate="G$1" x="76.2" y="223.52" rot="R180"/>
+<instance part="+2V4" gate="G$1" x="76.2" y="226.06" smashed="yes">
+<attribute name="VALUE" x="73.66" y="223.52" size="1.778" layer="96" rot="R90"/>
+</instance>
+<instance part="3V3" gate="G$1" x="81.28" y="223.52" rot="R180"/>
+<instance part="+3V1" gate="G$1" x="81.28" y="228.6" smashed="yes">
+<attribute name="VALUE" x="81.28" y="228.6" size="1.778" layer="96" rot="R90"/>
+</instance>
+<instance part="P+1" gate="1" x="86.36" y="228.6" smashed="yes">
+<attribute name="VALUE" x="86.36" y="231.14" size="1.778" layer="96" rot="R90"/>
+</instance>
+<instance part="+5V" gate="G$1" x="86.36" y="223.52" rot="R180"/>
 </instances>
 <busses>
@@
 <wire x1="58.42" y1="236.22" x2="53.34" y2="236.22" width="0.1524" layer="91"/>
 </segment>
+<segment>
+<pinref part="2V5" gate="G$1" pin="TP"/>
+<pinref part="+2V4" gate="G$1" pin="+2V5"/>
+</segment>
 </net>
 <net name="+5V" class="0">
@@
 <junction x="17.78" y="109.22"/>
 </segment>
+<segment>
+<pinref part="P+1" gate="1" pin="+5V"/>
+<pinref part="+5V" gate="G$1" pin="TP"/>
+</segment>
 </net>
 <net name="+3V3" class="0">
@@
 <junction x="35.56" y="68.58"/>
 </segment>
-</net>
+<segment>
+<pinref part="3V3" gate="G$1" pin="TP"/>
+<pinref part="+3V1" gate="G$1" pin="+3V3"/>
+</segment>
+</net>

Commit message: xdac: finished PCB
Signed-off-by: malo <pavol.malosek@gmail.com>
Parts:
- added 1, 2, 3, 4, 5, 6, 7, 8: (no value), 25pinhead:PINHD-1X1
- added 3V3A, 5VA, GND___: TPTP14R, testpad:TPTP14R
Connections:
- net 3V3A: now also 3V3A.TP
- net 5VA: now also 5VA.TP
- net AOUT2_: now also 2.1
- net AOUT3_: now also 3.1
- net AOUT4_: now also 4.1
- net AOUT5_: now also 5.1
- net AOUT6_: now also 6.1
- net AOUT7_: now also 7.1
- net AOUT8_: now also 8.1
- net AUOT1_: now also 1.1
- net GND: now also GND___.TP
Other:
- moved on the sheet: A1, A2, A3, A4, A5, A6, A7, A8, C11, C12, C13, C14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
