File: xdac/xdac_A.sch (EAGLE design)
At the start: 101 parts, among them J1 LIWE_40_PIN, J12 FC68131, J2 PINHD-3X5/90, J3 PINHD-3X5/90, J34 FC68131, J56 FC68131, J78 FC68131, U2 CS4384, U3 FIN1002

Commit message: xmod: fixed capacitor type in output filter
Signed-off-by: malo <pavol.malosek@gmail.com>
Parts:
- C11, C12, C14, C17, C18, C23, C24: value 22u, EEEFC1V220P -> 22u, EEEFC1C220R
- C13: value 22u, EEEFC1V220P -> 22u,EEEFC1C220R
Changed lines of the file:
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@@
 <?xml version="1.0" encoding="utf-8"?>
 <!DOCTYPE eagle SYSTEM "eagle.dtd">
-<eagle version="8.1.0">
+<eagle version="7.7.0">
 <drawing>
 <settings>
@@
 <part name="GND9" library="supply1" deviceset="GND" device=""/>
 <part name="GND10" library="supply1" deviceset="GND" device=""/>
-<part name="C11" library="25cmsquare" deviceset="C-POL" device="_C" value="22u, EEEFC1V220P"/>
-<part name="C12" library="25cmsquare" deviceset="C-POL" device="_C" value="22u, EEEFC1V220P"/>
+<part name="C11" library="25cmsquare" deviceset="C-POL" device="_C" value="22u, EEEFC1C220R"/>
+<part name="C12" library="25cmsquare" deviceset="C-POL" device="_C" value="22u, EEEFC1C220R"/>
 <part name="C19" library="rcl" deviceset="C-EU" device="C0603" value="2n2"/>
 <part name="GND20" library="supply1" deviceset="GND" device=""/>
@@
 <part name="GND12" library="supply1" deviceset="GND" device=""/>
 <part name="GND13" library="supply1" deviceset="GND" device=""/>
-<part name="C13" library="25cmsquare" deviceset="C-POL" device="_C" value="22u, EEEFC1V220P"/>
-<part name="C14" library="25cmsquare" deviceset="C-POL" device="_C" value="22u, EEEFC1V220P"/>
+<part name="C13" library="25cmsquare" deviceset="C-POL" device="_C" value="22u,EEEFC1C220R"/>
+<part name="C14" library="25cmsquare" deviceset="C-POL" device="_C" value="22u, EEEFC1C220R"/>
 <part name="C15" library="rcl" deviceset="C-EU" device="C0603" value="2n2"/>
 <part name="GND14" library="supply1" deviceset="GND" device=""/>
@@
 <part name="GND17" library="supply1" deviceset="GND" device=""/>
 <part name="GND18" library="supply1" deviceset="GND" device=""/>
-<part name="C17" library="25cmsquare" deviceset="C-POL" device="_C" value="22u, EEEFC1V220P"/>
-<part name="C18" library="25cmsquare" deviceset="C-POL" device="_C" value="22u, EEEFC1V220P"/>
+<part name="C17" library="25cmsquare" deviceset="C-POL" device="_C" value="22u, EEEFC1C220R"/>
+<part name="C18" library="25cmsquare" deviceset="C-POL" device="_C" value="22u, EEEFC1C220R"/>
 <part name="C21" library="rcl" deviceset="C-EU" device="C0603" value="2n2"/>
 <part name="GND19" library="supply1" deviceset="GND" device=""/>
@@
 <part name="GND24" library="supply1" deviceset="GND" device=""/>
 <part name="GND25" library="supply1" deviceset="GND" device=""/>
-<part name="C23" library="25cmsquare" deviceset="C-POL" device="_C" value="22u, EEEFC1V220P"/>
-<part name="C24" library="25cmsquare" deviceset="C-POL" device="_C" value="22u, EEEFC1V220P"/>
+<part name="C23" library="25cmsquare" deviceset="C-POL" device="_C" value="22u, EEEFC1C220R"/>
+<part name="C24" library="25cmsquare" deviceset="C-POL" device="_C" value="22u, EEEFC1C220R"/>
 <part name="C25" library="rcl" deviceset="C-EU" device="C0603" value="2n2"/>
 <part name="GND26" library="supply1" deviceset="GND" device=""/>
