File: xdac/xdac_A.brd (EAGLE design)
At the start: 80 x 80 mm, 101 parts, among them J1 LIWE_40_PIN, J12 FC68131, J2 PINHD-3X5/90, J3 PINHD-3X5/90, J34 FC68131, J56 FC68131, J78 FC68131, U2 CS4384, U3 FIN1002

Commit message: xmod: fixed capacitor type in output filter
Signed-off-by: malo <pavol.malosek@gmail.com>
Parts:
- C11, C12, C14, C17, C18, C23, C24: value 22u, EEEFC1V220P -> 22u, EEEFC1C220R
- C13: value 22u, EEEFC1V220P -> 22u,EEEFC1C220R
Changed lines of the file:
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@@
 <?xml version="1.0" encoding="utf-8"?>
 <!DOCTYPE eagle SYSTEM "eagle.dtd">
-<eagle version="8.1.0">
+<eagle version="7.7.0">
 <drawing>
 <settings>
@@
 <attribute name="NAME" x="41.1988" y="22.2504" size="1.016" layer="25" font="vector" ratio="15" rot="SR0"/>
 </element>
-<element name="C11" library="25cmsquare" package="EEE-FC1C220R" value="22u, EEEFC1V220P" x="61.468" y="66.929" smashed="yes">
+<element name="C11" library="25cmsquare" package="EEE-FC1C220R" value="22u, EEEFC1C220R" x="61.468" y="66.929" smashed="yes">
 <attribute name="NAME" x="60.6298" y="69.8754" size="1.016" layer="25" font="vector" ratio="15" rot="SR0"/>
 </element>
-<element name="C12" library="25cmsquare" package="EEE-FC1C220R" value="22u, EEEFC1V220P" x="61.468" y="61.087" smashed="yes">
+<element name="C12" library="25cmsquare" package="EEE-FC1C220R" value="22u, EEEFC1C220R" x="61.468" y="61.087" smashed="yes">
 <attribute name="NAME" x="60.6044" y="57.1246" size="1.016" layer="25" font="vector" ratio="15" rot="SR0"/>
 </element>
-<element name="C13" library="25cmsquare" package="EEE-FC1C220R" value="22u, EEEFC1V220P" x="61.468" y="50.927" smashed="yes">
+<element name="C13" library="25cmsquare" package="EEE-FC1C220R" value="22u,EEEFC1C220R" x="61.468" y="50.927" smashed="yes">
 <attribute name="NAME" x="60.4774" y="53.8226" size="1.016" layer="25" font="vector" ratio="15" rot="SR0"/>
 </element>
-<element name="C14" library="25cmsquare" package="EEE-FC1C220R" value="22u, EEEFC1V220P" x="61.468" y="45.085" smashed="yes">
+<element name="C14" library="25cmsquare" package="EEE-FC1C220R" value="22u, EEEFC1C220R" x="61.468" y="45.085" smashed="yes">
 <attribute name="NAME" x="60.4774" y="41.1988" size="1.016" layer="25" font="vector" ratio="15" rot="SR0"/>
 </element>
@@
 <attribute name="NAME" x="68.4784" y="40.513" size="1.016" layer="25" font="vector" ratio="15"/>
 </element>
-<element name="C17" library="25cmsquare" package="EEE-FC1C220R" value="22u, EEEFC1V220P" x="61.468" y="34.925" smashed="yes">
+<element name="C17" library="25cmsquare" package="EEE-FC1C220R" value="22u, EEEFC1C220R" x="61.468" y="34.925" smashed="yes">
 <attribute name="NAME" x="60.3504" y="37.8206" size="1.016" layer="25" font="vector" ratio="15" rot="SR0"/>
 </element>
-<element name="C18" library="25cmsquare" package="EEE-FC1C220R" value="22u, EEEFC1V220P" x="61.468" y="29.083" smashed="yes">
+<element name="C18" library="25cmsquare" package="EEE-FC1C220R" value="22u, EEEFC1C220R" x="61.468" y="29.083" smashed="yes">
 <attribute name="NAME" x="60.6044" y="25.1206" size="1.016" layer="25" font="vector" ratio="15" rot="SR0"/>
 </element>
@@
 <attribute name="NAME" x="68.6054" y="24.511" size="1.016" layer="25" font="vector" ratio="15"/>
 </element>
-<element name="C23" library="25cmsquare" package="EEE-FC1C220R" value="22u, EEEFC1V220P" x="61.468" y="18.923" smashed="yes">
+<element name="C23" library="25cmsquare" package="EEE-FC1C220R" value="22u, EEEFC1C220R" x="61.468" y="18.923" smashed="yes">
 <attribute name="NAME" x="60.706" y="21.7678" size="1.016" layer="25" font="vector" ratio="15" rot="SR0"/>
 </element>
-<element name="C24" library="25cmsquare" package="EEE-FC1C220R" value="22u, EEEFC1V220P" x="61.468" y="13.081" smashed="yes">
+<element name="C24" library="25cmsquare" package="EEE-FC1C220R" value="22u, EEEFC1C220R" x="61.468" y="13.081" smashed="yes">
 <attribute name="NAME" x="60.6806" y="9.1948" size="1.016" layer="25" font="vector" ratio="15" rot="SR0"/>
 </element>
