File: xmod/xmod_A.brd (EAGLE design)
At the start: 80 x 80 mm, 32 parts, among them J1 LIWE_40_PIN, J4 PINHD-3X5/90, J5 PINHD-3X9/90, U1 STA311B, U3 FIN1002

Commit message: xmod: PCB finished
Signed-off-by: malo <pavol.malosek@gmail.com>
Parts:
- added BICKO, LRCLKO, RST_N, SDO12, SDO34, SDO56, SDO78: (no value), 25pinhead:1X01
- added CKOUT, MVO, PWDN: TPTP14R, testpad:TP14R
- added R10, R11, R8, R9: (no value), rcl:R0603
- added U$1, U$2, U$3, U$4: TEST-22-MULTICOMP, 25cmsquare:TEST_1MM
- moved C34 2.54 mm to (18.8, 27.3)
Connections:
- net +3V3: now also R11.2, R8.1, R9.2
- net BICKO: now also BICKO.1
- net CKOUT: now also CKOUT.TP
- net GND: now also R10.2, U$1.1, U$2.1, U$3.1, U$4.1; no longer J1.16, J1.20
- net LRCLKO: now also LRCLKO.1
- net MVO: now also MVO.TP, R10.1
- net PWDN: now also PWDN.TP, R11.1
- net RST_N: now also J4.1, RST_N.1
- net SCL: now also R9.1
- net SDA: now also R8.2
- net SDO12: now also SDO12.1
- net SDO34: now also SDO34.1
- net SDO56: now also SDO56.1
- net SDO78: now also SDO78.1
Routing:
- net RST_N: track 0.00 -> 32.8 mm, vias 0 -> 2
- net CKOUT: track 0.00 -> 8.33 mm
- net PWDN: track 35.8 -> 40.7 mm
- net +3V3: track 454.1 -> 458.6 mm, vias 2 -> 4
- net MVO: track 29.1 -> 31.8 mm
- net SCL: track 40.9 -> 42.0 mm
- net SDO12: track 20.2 -> 21.3 mm
- net BICKO: track 25.7 -> 26.7 mm
- net SDO34: track 26.1 -> 26.6 mm
- net LRCLKO: track 20.4 -> 20.9 mm
- net GND: vias 43 -> 52
Other:
- board text added: "25"
- board text added: "BICKI"
- board text added: "BICKO"
- board text added: "CL3.CL2"
- board text added: "EAPD"
- board text added: "GND"
- board text added: "LRCKI"
- board text added: "LRCLKO"
- board text added: "MVO"
- board text added: "OUT_1A"
- board text added: "OUT_1B"
- board text added: "OUT_2A"
- board text added: "OUT_2B"
- board text added: "OUT_3A"
- board text added: "OUT_3B"
- board text added: "OUT_4A"
- board text added: "OUT_4B"
- board text added: "OUT_5A"
- board text added: "OUT_5B"
- board text added: "OUT_6A"
- board text added: "OUT_6B"
- board text added: "OUT_7A"
- board text added: "OUT_7B"
- board text added: "OUT_8A"
- board text added: "OUT_8B"
- board text added: "PWDN"
- board text added: "RST_N"
- board text added: "SC1.SD1"
- board text added: "SDI12"
- board text added: "SDI34"
- board text added: "SDI56"
- board text added: "SDI78"
- board text added: "SDO12"
- board text added: "SDO34"
- board text added: "SDO56"
- board text added: "SDO78"
