File: xmod/xmod_A.sch (EAGLE design)
At the start: 32 parts, among them J1 LIWE_40_PIN, J4 PINHD-3X5/90, J5 PINHD-3X9/90, U1 STA311B, U3 FIN1002

Commit message: xmod: PCB finished
Signed-off-by: malo <pavol.malosek@gmail.com>
Parts:
- added BICKO, LRCLKO, RST_N, SDO12, SDO34, SDO56, SDO78: (no value), 25pinhead:PINHD-1X1
- added CKOUT, MVO, PWDN: TPTP14R, testpad:TPTP14R
- added R10, R11, R8, R9: (no value), rcl:R-EU_R0603
- added U$1, U$2, U$3, U$4: TEST-22-MULTICOMP, 25cmsquare:TEST-22-MULTICOMP
Connections:
- net +3V3: now also R11.2, R8.1, R9.2
- net BICKO: now also BICKO.1
- net CKOUT: now also CKOUT.TP
- net GND: now also R10.2, U$1.1, U$2.1, U$3.1, U$4.1; no longer J1_PWR.GND7, J1_PWR.GND9
- net LRCLKO: now also LRCLKO.1
- net MVO: now also MVO.TP, R10.1
- net PWDN: now also PWDN.TP, R11.1
- net RST_N: now also J4.1, RST_N.1
- net SCL: now also R9.1
- net SDA: now also R8.2
- net SDO12: now also SDO12.1
- net SDO34: now also SDO34.1
- net SDO56: now also SDO56.1
- net SDO78: now also SDO78.1
Other:
- note added: "17.03.28.A"
- moved on the sheet: J1_IO, SCL, SDA
