File: xcodec/xcodec_CS42526_A.sch (EAGLE design)
At the start: 6 parts, among them U1 CS42526, U3 FIN1002

Commit message: xcodec: WIP
Signed-off-by: malo <pavol.malosek@gmail.com>
Parts:
- added 3V3, 5V0, RMCK: TPTP14R, testpad:TPTP14R
- added C1, C11, C12, C2: 10u, 16V, EEEFC1C100R, 25cmsquare:C-POL_B
- added C10, C14, C17, C22, C23, C4, C6, C8: 100n, rcl:C-EUC0603K
- added C13, C16: 1u, 35V, EEEFC1V1R0R, 25cmsquare:C-POL_B
- added C15, C18, C25, C26, C27, C28, C29, C3, C30, C31, C32, C5, C7, C9: 10n, rcl:C-EUC0603K
- added C19: 0.022u, rcl:C-EUC0603K
- added C20: 1n, rcl:C-EUC0603K
- added C21: 100u, 6.3V, EEEFC0J101P, 25cmsquare:C-POL_D
- added C24: 4.7u, 35V,EEEFC1V4R7R, 25cmsquare:C-POL_B
- added C34, C35, C36, C37: 10u, rcl:C-EUC0603K
- added C38: 100n, 0603, rcl:C-EUC0603K
- added J1: PINHD-3X13/90, 25pinhead:PINHD-3X13/90
- added J2: PINHD-3X9/90, 25pinhead:PINHD-3X9/90
- added J3: PINHD-3X7/90, 25pinhead:PINHD-3X7/90
- added JP1: (no value), 25pinhead:PINHD-1X2
- added JP2: (no value), 25pinhead:PINHD-2X13
- added JP3: (no value), 25pinhead:PINHD-2X4
- added L1, L2: 600R@100MHz, 25cmsquare:L0603(1608)
- added LRCK, SCLK, SDIN1, SDIN2, SDIN3, SDOUT: (no value), 25pinhead:PINHD-1X1
- added R1: 1k2, rcl:R-EU_R0603
- added R10: 4k7, rcl:R-EU_R0603
- added R11: 120R, rcl:R-EU_R0603
- added R12, R13, R14, R2, R3, R4, R5, R6, R8, R9: (no value), rcl:R-EU_R0603
- added U2: FIN1002, 25cmsquare:FIN1002
- C33: device rcl:C-EUC0603 -> rcl:C-EUC0603K
Connections:
- new net +3V3_CODEC: C1.+, C10.1, C11.+, C13.+, C14.1, C15.1, C16.+, C17.1, C18.1, C3.1, C4.1, C9.1, L1.1, U1.VD_0, U1.VD_1, U1.VLC, U1.VLS
- new net +5V: 5V0.TP, L2.1, U$1_PWR.VCC9
- new net +5V_CODEC: C12.+, C2.+, C5.1, C6.1, C7.1, C8.1, L2.2, U1.VA, U1.VARX
- new net A1+: JP2.5, U1.AOUTA1+
- new net A1-: JP2.3, U1.AOUTA1-
- new net A2+: JP2.13, U1.AOUTA2+
- new net A2-: JP2.11, U1.AOUTA2-
- new net A3+: JP2.21, U1.AOUTA3+
- new net A3-: JP2.19, U1.AOUTA3-
- new net ADCIN1: U1.ADCIN1
- new net ADCIN2: U1.ADCIN2
- new net B1+: JP2.7, U1.AOUTB1+
- new net B1-: JP2.9, U1.AOUTB1-
- new net B2+: JP2.15, U1.AOUTB2+
- new net B2-: JP2.17, U1.AOUTB2-
- new net B3+: JP2.23, U1.AOUTB3+
- new net B3-: JP2.25, U1.AOUTB3-
- new net CX_LRCK: LRCK.1, U1.CX_LRCK
- new net CX_SCLK: SCLK.1, U1.CX_SCLK
- new net CX_SDIN1: SDIN1.1, U1.CX_SDIN1
- new net CX_SDIN2: SDIN2.1, U1.CX_SDIN2
- new net CX_SDIN3: SDIN3.1, U1.CX_SDIN3
- new net CX_SDOUT: SDOUT.1, U1.CX_SDOUT
- new net FILT+: C21.+, C22.1, U1.FILT+
- new net INL+: C37.2, JP3.1
- new net INL-: C36.2, JP3.3
- new net INR+: C35.2, JP3.5
- new net INR-: C34.2, JP3.7
- new net INT: U1.INT
- new net LPFLT: C20.1, R1.2, U1.LPFLT
- new net MUTEC: JP2.1, U1.MUTEC
- new net N$1: R12.1, U1.SAI_SDOUT
- new net N$16: C37.1, U1.AINL+
- new net N$17: C36.1, U1.AINL-
- new net N$18: C35.1, U1.AINR+
- new net N$19: C34.1, U1.AINR-
- new net N$2: R11.2, U2.ROUT
- new net N$3: C19.1, R1.1
- new net N$4: R13.1, U1.SAI_LRCK
- new net N$5: R14.1, U1.SAI_SCLK
- new net RMCK: RMCK.TP, U1.RMCK
- new net RP0: C25.2, U1.RXP0
- new net RP1: C26.2, U1.RXP1/GPO1
- new net RP2: C27.2, U1.RXP2/GPO2
- new net RP3: C28.2, U1.RXP3/GPO3
- new net RP4: C29.2, U1.RXP4/GPO4
- new net RP5: C30.2, U1.RXP5/GPO5
- new net RP6: C31.2, U1.RXP6/GPO6
- new net RP7: C32.2, U1.RXP7/GPO7
- new net RST_N: R10.1, U1.RST_N
- new net RXP0: C25.1
- new net RXP1: C26.1, R11.1
- new net RXP1_N: U2.RIN-
- new net RXP1_P: U2.RIN+
- new net RXP2: C27.1
- new net RXP3: C28.1
- new net RXP4: C29.1
- new net RXP5: C30.1
- new net RXP6: C31.1
- new net RXP7: C32.1
- new net SAI_LRCK: R13.2
- new net SAI_SCLK: R14.2
- new net SAI_SDOUT: R12.2
- new net SCL: JP1.1, R3.1, R4.1, R8.2, U1.SCL/CCLK
- new net SCL0: R3.2, U$1_IO.I2C0_SCL
- new net SCL1: R4.2, U$1_IO.I2C1_SCL
- new net SDA: JP1.2, R5.1, R6.1, R9.1, U1.SDA/CDOUT
- new net SDA0: R5.2, U$1_IO.I2C0_SDA
- new net SDA1: R6.2, U$1_IO.I2C1_SDA
- new net TP0: R2.2, U1.TXP
- new net TXP0: R2.1
- new net VQ: C23.1, C24.+, U1.VQ
- net +3V3: now also 3V3.TP, C38.2, L1.2, R10.2, R8.1, R9.2, U$1_PWR.VCC8, U2.VCC
- net GND: now also C1.-, C10.2, C11.-, C12.-, C13.-, C14.2, C15.2, C16.-, C17.2, C18.2, C19.2, C2.-, C20.2, C21.-, C22.2, C23.2, C24.-, C3.2, C38.1, C4.2, C5.2, C6.2, C7.2, C8.2, C9.2, U1.AD0/CS_N, U1.AD1/CDIN, U1.AGND_0, U1.AGND_1, U1.DGND_0, U1.DGND_1, U1.REFGND, U1.TEST, U2.GND
- net MCLK: now also U1.OMCK
Other:
- moved on the sheet: U$1_IO, U$1_PWR, U1

Commit message: xdac: WIP
Signed-off-by: malo <pavol.malosek@gmail.com>
Parts:
- removed SDOUT: (no value), 25pinhead:PINHD-1X1
Connections:
- removed net ADCIN1: U1.ADCIN1
- removed net ADCIN2: U1.ADCIN2
- removed net CX_SDOUT: SDOUT.1, U1.CX_SDOUT
Changed lines of the file:
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@@
 <setting verticaltext="up"/>
 </settings>
-<grid distance="100" unitdist="mil" unit="mil" style="lines" multiple="1" display="no" altdistance="0.01" altunitdist="inch" altunit="inch"/>
+<grid distance="0.1" unitdist="inch" unit="inch" style="lines" multiple="1" display="no" altdistance="0.01" altunitdist="inch" altunit="inch"/>
 <layers>
-<layer number="1" name="Top" color="4" fill="1" visible="yes" active="no"/>
-<layer number="16" name="Bottom" color="1" fill="1" visible="yes" active="no"/>
-<layer number="17" name="Pads" color="2" fill="1" visible="yes" active="no"/>
-<layer number="18" name="Vias" color="2" fill="1" visible="yes" active="no"/>
-<layer number="19" name="Unrouted" color="6" fill="1" visible="yes" active="no"/>
-<layer number="20" name="Dimension" color="15" fill="1" visible="yes" active="no"/>
-<layer number="21" name="tPlace" color="7" fill="1" visible="yes" active="no"/>
-<layer number="22" name="bPlace" color="7" fill="1" visible="yes" active="no"/>
-<layer number="23" name="tOrigins" color="15" fill="1" visible="yes" active="no"/>
-<layer number="24" name="bOrigins" color="15" fill="1" visible="yes" active="no"/>
-<layer number="25" name="tNames" color="7" fill="1" visible="yes" active="no"/>
-<layer number="26" name="bNames" color="7" fill="1" visible="yes" active="no"/>
-<layer number="27" name="tValues" color="7" fill="1" visible="yes" active="no"/>
-<layer number="28" name="bValues" color="7" fill="1" visible="yes" active="no"/>
+<layer number="1" name="Top" color="4" fill="1" visible="no" active="no"/>
+<layer number="16" name="Bottom" color="1" fill="1" visible="no" active="no"/>
+<layer number="17" name="Pads" color="2" fill="1" visible="no" active="no"/>
+<layer number="18" name="Vias" color="2" fill="1" visible="no" active="no"/>
+<layer number="19" name="Unrouted" color="6" fill="1" visible="no" active="no"/>
+<layer number="20" name="Dimension" color="15" fill="1" visible="no" active="no"/>
+<layer number="21" name="tPlace" color="7" fill="1" visible="no" active="no"/>
+<layer number="22" name="bPlace" color="7" fill="1" visible="no" active="no"/>
+<layer number="23" name="tOrigins" color="15" fill="1" visible="no" active="no"/>
+<layer number="24" name="bOrigins" color="15" fill="1" visible="no" active="no"/>
+<layer number="25" name="tNames" color="7" fill="1" visible="no" active="no"/>
+<layer number="26" name="bNames" color="7" fill="1" visible="no" active="no"/>
+<layer number="27" name="tValues" color="7" fill="1" visible="no" active="no"/>
+<layer number="28" name="bValues" color="7" fill="1" visible="no" active="no"/>
 <layer number="29" name="tStop" color="7" fill="3" visible="no" active="no"/>
 <layer number="30" name="bStop" color="7" fill="6" visible="no" active="no"/>
@@
 <layer number="35" name="tGlue" color="7" fill="4" visible="no" active="no"/>
 <layer number="36" name="bGlue" color="7" fill="5" visible="no" active="no"/>
-<layer number="37" name="tTest" color="7" fill="1" visible="yes" active="no"/>
-<layer number="38" name="bTest" color="7" fill="1" visible="yes" active="no"/>
+<layer number="37" name="tTest" color="7" fill="1" visible="no" active="no"/>
+<layer number="38" name="bTest" color="7" fill="1" visible="no" active="no"/>
 <layer number="39" name="tKeepout" color="4" fill="11" visible="no" active="no"/>
 <layer number="40" name="bKeepout" color="1" fill="11" visible="no" active="no"/>
@@
 <layer number="44" name="Drills" color="7" fill="1" visible="no" active="no"/>
 <layer number="45" name="Holes" color="7" fill="1" visible="no" active="no"/>
-<layer number="46" name="Milling" color="3" fill="1" visible="yes" active="no"/>
-<layer number="47" name="Measures" color="7" fill="1" visible="yes" active="no"/>
-<layer number="48" name="Document" color="7" fill="1" visible="yes" active="no"/>
-<layer number="49" name="Reference" color="7" fill="1" visible="yes" active="no"/>
-<layer number="50" name="dxf" color="7" fill="1" visible="yes" active="no"/>
-<layer number="51" name="tDocu" color="7" fill="1" visible="yes" active="no"/>
-<layer number="52" name="bDocu" color="7" fill="1" visible="yes" active="no"/>
-<layer number="53" name="tGND_GNDA" color="7" fill="9" visible="yes" active="no"/>
-<layer number="54" name="bGND_GNDA" color="1" fill="9" visible="yes" active="no"/>
-<layer number="56" name="wert" color="7" fill="1" visible="yes" active="no"/>
-<layer number="57" name="tCAD" color="7" fill="1" visible="yes" active="no"/>
-<layer number="59" name="Invisible" color="7" fill="1" visible="yes" active="no"/>
-<layer number="61" name="stand" color="7" fill="1" visible="yes" active="no"/>
+<layer number="46" name="Milling" color="3" fill="1" visible="no" active="no"/>
+<layer number="47" name="Measures" color="7" fill="1" visible="no" active="no"/>
+<layer number="48" name="Document" color="7" fill="1" visible="no" active="no"/>
+<layer number="49" name="Reference" color="7" fill="1" visible="no" active="no"/>
+<layer number="50" name="dxf" color="7" fill="1" visible="no" active="no"/>
+<layer number="51" name="tDocu" color="7" fill="1" visible="no" active="no"/>
+<layer number="52" name="bDocu" color="7" fill="1" visible="no" active="no"/>
+<layer number="53" name="tGND_GNDA" color="7" fill="9" visible="no" active="no"/>
+<layer number="54" name="bGND_GNDA" color="1" fill="9" visible="no" active="no"/>
+<layer number="56" name="wert" color="7" fill="1" visible="no" active="no"/>
+<layer number="57" name="tCAD" color="7" fill="1" visible="no" active="no"/>
+<layer number="59" name="Invisible" color="7" fill="1" visible="no" active="no"/>
+<layer number="61" name="stand" color="7" fill="1" visible="no" active="no"/>
 <layer number="90" name="Modules" color="5" fill="1" visible="yes" active="yes"/>
 <layer number="91" name="Nets" color="2" fill="1" visible="yes" active="yes"/>
@@
 <part name="LRCK" library="25pinhead" deviceset="PINHD-1X1" device=""/>
 <part name="SCLK" library="25pinhead" deviceset="PINHD-1X1" device=""/>
-<part name="SDOUT" library="25pinhead" deviceset="PINHD-1X1" device=""/>
 <part name="SDIN1" library="25pinhead" deviceset="PINHD-1X1" device=""/>
 <part name="SDIN2" library="25pinhead" deviceset="PINHD-1X1" device=""/>
@@
 <instance part="LRCK" gate="G$1" x="170.18" y="45.72" rot="R90"/>
 <instance part="SCLK" gate="G$1" x="177.8" y="45.72" rot="R90"/>
-<instance part="SDOUT" gate="G$1" x="185.42" y="45.72" rot="R90"/>
 <instance part="SDIN1" gate="G$1" x="193.04" y="45.72" rot="R90"/>
 <instance part="SDIN2" gate="G$1" x="200.66" y="45.72" rot="R90"/>
@@
 </segment>
 </net>
-<net name="CX_SDOUT" class="0">
-<segment>
-<pinref part="U1" gate="G$1" pin="CX_SDOUT"/>
-<wire x1="185.42" y1="109.22" x2="177.8" y2="109.22" width="0.1524" layer="91"/>
-<label x="177.8" y="109.22" size="1.778" layer="95" rot="R180" xref="yes"/>
-</segment>
-<segment>
-<pinref part="SDOUT" gate="G$1" pin="1"/>
-<wire x1="185.42" y1="43.18" x2="185.42" y2="35.56" width="0.1524" layer="91"/>
-<label x="185.42" y="35.56" size="1.778" layer="95" rot="R270" xref="yes"/>
-</segment>
-</net>
 <net name="CX_SDIN1" class="0">
 <segment>
@@
 </segment>
 </net>
-<net name="ADCIN1" class="0">
-<segment>
-<pinref part="U1" gate="G$1" pin="ADCIN1"/>
-<wire x1="185.42" y1="137.16" x2="177.8" y2="137.16" width="0.1524" layer="91"/>
-<label x="177.8" y="137.16" size="1.778" layer="95" rot="R180" xref="yes"/>
-</segment>
-</net>
-<net name="ADCIN2" class="0">
-<segment>
-<pinref part="U1" gate="G$1" pin="ADCIN2"/>
-<wire x1="185.42" y1="134.62" x2="160.02" y2="134.62" width="0.1524" layer="91"/>
-<label x="160.02" y="134.62" size="1.778" layer="95" rot="R180" xref="yes"/>
-</segment>
-</net>

Commit message: xcodec: WIP
Signed-off-by: malo <pavol.malosek@gmail.com>
Parts:
- J1: value PINHD-3X13/90 -> (none); device 25pinhead:PINHD-3X13/90 -> 25pinhead:PINHD-3X3/90
- RMCK: value TPTP14R -> (none); device testpad:TPTP14R -> 25pinhead:PINHD-1X1
Connections:
- removed net RXP7: C32.1
- new net IN_L+: J1.1, JP3.4
- new net IN_L-: J1.3, JP3.2
- new net IN_R+: J1.6, JP3.6
- new net IN_R-: J1.4, JP3.8
- new net N$6: J3.1
- new net _A1+: J3.4, JP2.6
- new net _A1-: J3.6, JP2.4
- new net _A2+: J3.10, JP2.14
- new net _A2-: J3.12, JP2.12
- new net _A3+: J3.16, JP2.22
- new net _A3-: J3.18, JP2.20
- new net _B1+: J3.7, JP2.8
- new net _B1-: J3.9, JP2.10
- new net _B2+: J3.13, JP2.16
- new net _B2-: J3.15, JP2.18
- new net _B3+: J3.19, JP2.24
- new net _B3-: J3.21, JP2.26
- new net _MUTEC: J3.3, JP2.2
- net CX_LRCK: now also J2.3
- net CX_SCLK: now also J2.1
- net CX_SDIN1: now also J2.6
- net CX_SDIN2: now also J2.4
- net CX_SDIN3: now also J2.9
- net GND: now also C32.1, J1.2, J1.5, J1.8, J2.11, J2.14, J2.17, J2.2, J2.20, J2.23, J2.26, J2.5, J2.8, J3.11, J3.14, J3.17, J3.2, J3.20, J3.5, J3.8, U$1_PWR.GND8, U$1_PWR.GND9
- net INL+: now also JP3.3; no longer JP3.1
- net INL-: now also JP3.1; no longer JP3.3
- net INT: now also J1.9
- net RMCK: now also RMCK.1; no longer RMCK.TP
- net RST_N: now also J1.7
- net RXP0: now also J2.13
- net RXP1: now also J2.18
- net RXP1_N: now also J2.21
- net RXP1_P: now also J2.19
- net RXP2: now also J2.16
- net RXP3: now also J2.22
- net RXP4: now also J2.24
- net RXP5: now also J2.25
- net RXP6: now also J2.27
- net SAI_LRCK: now also J2.12
- net SAI_SCLK: now also J2.7
- net SAI_SDOUT: now also J2.10
- net TXP0: now also J2.15
Other:
- moved on the sheet: J2, J3
