File: xcodec/xcodec_CS42526_A.brd (EAGLE design)
At the start: 80 x 80 mm, 80 parts, among them J2 PINHD-3X9/90, J3 PINHD-3X7/90, U1 CS42526, U2 FIN1002, U3 FIN1002

Commit message: xcodec: final DSP
Signed-off-by: malo <pavol.malosek@gmail.com>
Parts:
- moved C5 0.51 mm to (45.6, 48.5)
- moved C6 0.51 mm to (47.2, 48.5)
- moved C19 0.25 mm to (52.5, 46.5)
- moved C20 0.25 mm to (50.1, 47.4)
- moved GND_4 0.25 mm to (20.3, 11.4)
- moved R1 0.25 mm to (50.2, 45.6)
Routing:
- net GND: track 0.13 -> 0.19 mm, vias 90 -> 91
