File: xcodec/xcodec_CS42526_A.brd (EAGLE design)
At the start: 100 x 80 mm, 6 parts, among them U1 CS42526, U3 FIN1002

Commit message: xcodec: WIP
Signed-off-by: malo <pavol.malosek@gmail.com>
Parts:
- added 3V3, 5V0, RMCK: TPTP14R, testpad:TP14R
- added C1, C11, C12, C2: 10u, 16V, EEEFC1C100R, 25cmsquare:EEE-FC1V1R0AR
- added C10, C14, C17, C22, C23, C4, C6, C8: 100n, rcl:C0603K
- added C13, C16: 1u, 35V, EEEFC1V1R0R, 25cmsquare:EEE-FC1V1R0AR
- added C15, C18, C25, C26, C27, C28, C29, C3, C30, C31, C32, C5, C7, C9: 10n, rcl:C0603K
- added C19: 0.022u, rcl:C0603K
- added C20: 1n, rcl:C0603K
- added C21: 100u, 6.3V, EEEFC0J101P, 25cmsquare:EEE-FC1V220P
- added C24: 4.7u, 35V,EEEFC1V4R7R, 25cmsquare:EEE-FC1V1R0AR
- added C34, C35, C36, C37: 10u, rcl:C0603K
- added C38: 100n, 0603, rcl:C0603K
- added J1: PINHD-3X13/90, 25pinhead:3X13/90
- added J2: PINHD-3X9/90, 25pinhead:3X9/90
- added J3: PINHD-3X7/90, 25pinhead:3X07/90
- added JP1: (no value), 25pinhead:1X02
- added JP2: (no value), 25pinhead:2X13
- added JP3: (no value), 25pinhead:2X04
- added L1, L2: 600R@100MHz, 25cmsquare:L0603
- added LRCK, SCLK, SDIN1, SDIN2, SDIN3, SDOUT: (no value), 25pinhead:1X01
- added R1: 1k2, rcl:R0603
- added R10: 4k7, rcl:R0603
- added R11: 120R, rcl:R0603
- added R12, R13, R14, R2, R3, R4, R5, R6, R8, R9: (no value), rcl:R0603
- added U2: FIN1002, 25cmsquare:SOT95P280X140-5N
- C33: device rcl:C0603 -> rcl:C0603K
- moved C33 99.0 mm to (17.1, 47.9)
- moved R7 96.8 mm to (19.2, 40.6)
- moved U3 78.2 mm to (16.8, 45.0), turned to 270 degrees
- moved MCLK 71.6 mm to (12.1, 45.0), turned to 90 degrees
- turned U1 to 45 degrees
Connections:
- new net +3V3_CODEC: C1.1, C10.1, C11.1, C13.1, C14.1, C15.1, C16.1, C17.1, C18.1, C3.1, C4.1, C9.1, L1.1, U1.4, U1.51, U1.53, U1.6
- new net +5V: 5V0.TP, L2.1, U$1.19
- new net +5V_CODEC: C12.1, C2.1, C5.1, C6.1, C7.1, C8.1, L2.2, U1.24, U1.41
- new net A1+: JP2.5, U1.36
- new net A1-: JP2.3, U1.37
- new net A2+: JP2.13, U1.32
- new net A2-: JP2.11, U1.33
- new net A3+: JP2.21, U1.28
- new net A3-: JP2.19, U1.29
- new net ADCIN1: U1.58
- new net ADCIN2: U1.57
- new net B1+: JP2.7, U1.35
- new net B1-: JP2.9, U1.34
- new net B2+: JP2.15, U1.31
- new net B2-: JP2.17, U1.30
- new net B3+: JP2.23, U1.27
- new net B3-: JP2.25, U1.26
- new net CX_LRCK: LRCK.1, U1.3
- new net CX_SCLK: SCLK.1, U1.2
- new net CX_SDIN1: SDIN1.1, U1.1
- new net CX_SDIN2: SDIN2.1, U1.64
- new net CX_SDIN3: SDIN3.1, U1.63
- new net CX_SDOUT: SDOUT.1, U1.56
- new net FILT+: C21.1, C22.1, U1.18
- new net INL+: C37.2, JP3.1
- new net INL-: C36.2, JP3.3
- new net INR+: C35.2, JP3.5
- new net INR-: C34.2, JP3.7
- new net INT: U1.11
- new net LPFLT: C20.1, R1.2, U1.39
- new net MUTEC: JP2.1, U1.38
- new net N$1: R12.1, U1.54
- new net N$16: C37.1, U1.15
- new net N$17: C36.1, U1.16
- new net N$18: C35.1, U1.14
- new net N$19: C34.1, U1.13
- new net N$2: R11.2, U2.5
- new net N$3: C19.1, R1.1
- new net N$4: R13.1, U1.60
- new net N$5: R14.1, U1.61
- new net RMCK: RMCK.TP, U1.55
- new net RP0: C25.2, U1.49
- new net RP1: C26.2, U1.48
- new net RP2: C27.2, U1.47
- new net RP3: C28.2, U1.46
- new net RP4: C29.2, U1.45
- new net RP5: C30.2, U1.44
- new net RP6: C31.2, U1.43
- new net RP7: C32.2, U1.42
- new net RST_N: R10.1, U1.12
- new net RXP0: C25.1
- new net RXP1: C26.1, R11.1
- new net RXP1_N: U2.4
- new net RXP1_P: U2.3
- new net RXP2: C27.1
- new net RXP3: C28.1
- new net RXP4: C29.1
- new net RXP5: C30.1
- new net RXP6: C31.1
- new net RXP7: C32.1
- new net SAI_LRCK: R13.2
- new net SAI_SCLK: R14.2
- new net SAI_SDOUT: R12.2
- new net SCL: JP1.1, R3.1, R4.1, R8.2, U1.7
- new net SCL0: R3.2, U$1.116
- new net SCL1: R4.2, U$1.114
- new net SDA: JP1.2, R5.1, R6.1, R9.1, U1.8
- new net SDA0: R5.2, U$1.115
- new net SDA1: R6.2, U$1.113
- new net TP0: R2.2, U1.50
- new net TXP0: R2.1
- new net VQ: C23.1, C24.1, U1.17
- net +3V3: now also 3V3.TP, C38.2, L1.2, R10.2, R8.1, R9.2, U$1.17, U2.1
- net GND: now also C1.2, C10.2, C11.2, C12.2, C13.2, C14.2, C15.2, C16.2, C17.2, C18.2, C19.2, C2.2, C20.2, C21.2, C22.2, C23.2, C24.2, C3.2, C38.1, C4.2, C5.2, C6.2, C7.2, C8.2, C9.2, U1.10, U1.19, U1.25, U1.40, U1.5, U1.52, U1.62, U1.9, U2.2
- net MCLK: now also U1.59
Routing:
- net +5V_CODEC: track 0.00 -> 253.2 mm
- net +3V3_CODEC: track 0.00 -> 99.3 mm
- net RP7: track 0.00 -> 17.2 mm
- net RP6: track 0.00 -> 15.7 mm
- net RP5: track 0.00 -> 14.4 mm
- net RP4: track 0.00 -> 13.1 mm
- net RP3: track 0.00 -> 12.3 mm
- net RP0: track 0.00 -> 11.9 mm
- net RP2: track 0.00 -> 11.5 mm
- net RP1: track 0.00 -> 10.7 mm
- net B2+: track 0.00 -> 9.59 mm
- net B1-: track 0.00 -> 9.49 mm
- net A3-: track 0.00 -> 8.44 mm
- net B2-: track 0.00 -> 8.16 mm
- net B1+: track 0.00 -> 7.35 mm
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Other:
- board size 100 x 80 mm -> 80 x 80 mm

Commit message: xdac: WIP
Signed-off-by: malo <pavol.malosek@gmail.com>
Parts:
- removed SDOUT: (no value), 25pinhead:1X01
- moved SDIN3 169.5 mm to (30.9, 65.3)
- moved RMCK 9.07 mm to (34.3, 45.6)
- moved C2 6.38 mm to (55.7, 49.5)
- moved R10 5.26 mm to (32.8, 28.9)
- moved C1 4.55 mm to (25.2, 35.5)
- moved C13 4.55 mm to (25.2, 30.3)
- moved C4 3.65 mm to (30.1, 34.3), turned to 180 degrees
- moved R8 3.26 mm to (16.6, 62.8)
- moved C14 3.12 mm to (31.1, 31.7)
- moved JP1 2.30 mm to (18.0, 55.9)
- moved C3 1.87 mm to (31.2, 36.0), turned to 180 degrees
- moved C15 1.83 mm to (33.0, 33.1)
- moved R9 1.36 mm to (18.1, 51.5)
- moved R12 0.79 mm to (30.4, 47.6)
- moved R13 0.79 mm to (30.4, 45.5)
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Connections:
- removed net ADCIN1: U1.58
- removed net ADCIN2: U1.57
- removed net CX_SDOUT: SDOUT.1, U1.56
Routing:
- net +3V3_CODEC: track 99.3 -> 177.0 mm
- net CX_LRCK: track 4.95 -> 38.5 mm
- net CX_SCLK: track 3.49 -> 36.4 mm
- net CX_SDIN1: track 2.13 -> 34.5 mm
- net CX_SDIN3: track 0.00 -> 31.7 mm
- net CX_SDIN2: track 2.17 -> 31.2 mm
- net MCLK: track 0.00 -> 6.98 mm
- net N$1: track 0.00 -> 6.68 mm
- net N$19: track 0.00 -> 5.51 mm
- net N$18: track 0.00 -> 4.67 mm
- net N$16: track 0.00 -> 4.59 mm
- net N$4: track 0.00 -> 4.58 mm
- net SCL: track 0.00 -> 4.19 mm
- net N$17: track 0.00 -> 4.17 mm
- net SDA: track 0.00 -> 4.09 mm
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
Commit message: xcodec: WIP
Signed-off-by: malo <pavol.malosek@gmail.com>
Parts:
- J1: value PINHD-3X13/90 -> (none); device 25pinhead:3X13/90 -> 25pinhead:3X03/90
- RMCK: value TPTP14R -> (none); device testpad:TP14R -> 25pinhead:1X01
- moved J1 80.0 mm to (40.0, -0.03), turned to 180 degrees
- moved J3 57.5 mm to (81.3, 40.0), turned to 270 degrees
- moved J2 56.6 mm to (40.0, 80.0), turned to 0 degrees
- moved 5V0 12.2 mm to (7.66, 39.3)
- moved 3V3 11.8 mm to (10.4, 30.2)
- moved R10 10.7 mm to (30.3, 18.5), turned to 180 degrees
- moved C24 8.96 mm to (41.4, 27.2)
- moved C21 8.60 mm to (49.0, 25.4)
- moved C2 6.33 mm to (49.8, 51.9)
- moved R7 4.59 mm to (21.7, 44.5), turned to 270 degrees
- moved C11 4.55 mm to (35.2, 61.0), turned to 180 degrees
- moved C16 4.48 mm to (35.2, 55.7), turned to 0 degrees
- moved R9 4.15 mm to (14.5, 53.6), turned to 180 degrees
- moved R6 3.58 mm to (14.5, 55.7)
- moved C23 3.47 mm to (40.6, 31.1), turned to 180 degrees
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Connections:
- removed net RXP7: C32.1
- new net IN_L+: J1.1, JP3.4
- new net IN_L-: J1.3, JP3.2
- new net IN_R+: J1.6, JP3.6
- new net IN_R-: J1.4, JP3.8
- new net N$6: J3.1
- new net _A1+: J3.4, JP2.6
- new net _A1-: J3.6, JP2.4
- new net _A2+: J3.10, JP2.14
- new net _A2-: J3.12, JP2.12
- new net _A3+: J3.16, JP2.22
- new net _A3-: J3.18, JP2.20
- new net _B1+: J3.7, JP2.8
- new net _B1-: J3.9, JP2.10
- new net _B2+: J3.13, JP2.16
- new net _B2-: J3.15, JP2.18
- new net _B3+: J3.19, JP2.24
- new net _B3-: J3.21, JP2.26
- new net _MUTEC: J3.3, JP2.2
- net CX_LRCK: now also J2.3
- net CX_SCLK: now also J2.1
- net CX_SDIN1: now also J2.6
- net CX_SDIN2: now also J2.4
- net CX_SDIN3: now also J2.9
- net GND: now also C32.1, J1.2, J1.5, J1.8, J2.11, J2.14, J2.17, J2.2, J2.20, J2.23, J2.26, J2.5, J2.8, J3.11, J3.14, J3.17, J3.2, J3.20, J3.5, J3.8, U$1.18, U$1.20
- net INL+: now also JP3.3; no longer JP3.1
- net INL-: now also JP3.1; no longer JP3.3
- net INT: now also J1.9
- net RMCK: now also RMCK.1; no longer RMCK.TP
- net RST_N: now also J1.7
- net RXP0: now also J2.13
- net RXP1: now also J2.18
- net RXP1_N: now also J2.21
- net RXP1_P: now also J2.19
- net RXP2: now also J2.16
- net RXP3: now also J2.22
- net RXP4: now also J2.24
- net RXP5: now also J2.25
- net RXP6: now also J2.27
- net SAI_LRCK: now also J2.12
- net SAI_SCLK: now also J2.7
- net SAI_SDOUT: now also J2.10
- net TXP0: now also J2.15
Routing:
- net +3V3: track 0.00 -> 193.1 mm, vias 0 -> 3
- net SCL: track 4.19 -> 67.9 mm, vias 0 -> 4
- net SDA: track 4.09 -> 66.5 mm, vias 0 -> 4
- net SAI_LRCK: track 0.00 -> 38.3 mm
- net INT: track 0.00 -> 38.2 mm
- net SAI_SCLK: track 0.00 -> 34.7 mm
- net RST_N: track 0.00 -> 33.8 mm
- net +5V_CODEC: track 256.8 -> 288.8 mm
- net SAI_SDOUT: track 0.00 -> 30.7 mm
- net +3V3_CODEC: track 177.0 -> 147.8 mm, vias 0 -> 2
- net TXP0: track 0.00 -> 26.4 mm
- net RXP4: track 0.00 -> 21.3 mm
- net RXP6: track 0.00 -> 21.0 mm
- net RXP1: track 0.00 -> 20.9 mm
- net CX_LRCK: track 38.5 -> 58.3 mm
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- added copper zone on layer 1, net GND
- added copper zone on layer 16, net GND

Commit message: xcodec: manual merge from upstream.
Signed-off-by: malo <pavol.malosek@gmail.com>
Parts:
- added +3V3_CODEC, +5V_CODEC, GND_0, GND_1, GND_2, GND_3, GND_4: (no value), 25pinhead:1X01
- moved C5 1.61 mm to (45.6, 48.5)
- moved JP3 1.55 mm to (40.3, 19.1)
- moved C34 0.85 mm to (32.3, 25.9)
- moved C35 0.80 mm to (34.0, 25.9)
- moved C37 0.77 mm to (35.6, 25.9)
- moved C36 0.76 mm to (37.3, 25.9)
- moved C32 0.63 mm to (52.2, 57.7)
- moved R2 0.51 mm to (41.2, 51.9)
- moved C6 0.51 mm to (47.2, 48.5)
- moved C31 0.41 mm to (50.5, 57.7)
- moved C30 0.30 mm to (48.9, 57.7)
- moved C19 0.27 mm to (52.5, 46.5)
- moved C20 0.25 mm to (50.1, 47.4)
- moved C10 0.25 mm to (38.8, 50.6)
- moved C17 0.25 mm to (33.5, 50.6)
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Connections:
- net +3V3_CODEC: now also +3V3_CODEC.1
- net +5V_CODEC: now also +5V_CODEC.1
- net GND: now also GND_0.1, GND_1.1, GND_2.1, GND_3.1, GND_4.1
Routing:
- net +3V3_CODEC: track 147.8 -> 159.2 mm
- net SDA: track 66.5 -> 71.4 mm
- net +5V_CODEC: track 288.8 -> 292.1 mm
- net CX_SDIN1: track 51.2 -> 48.5 mm
- net SCL: track 67.9 -> 70.3 mm
- net CX_LRCK: track 58.3 -> 56.6 mm
- net IN_L-: track 14.3 -> 15.9 mm
- net RST_N: track 33.8 -> 32.2 mm
- net CX_SCLK: track 49.6 -> 48.1 mm
- net IN_R+: track 15.3 -> 16.7 mm
- net IN_R-: track 10.3 -> 11.7 mm
- net IN_L+: track 9.20 -> 10.6 mm
- net GND: track 1.52 -> 0.19 mm, vias 66 -> 91
- net SAI_SDOUT: track 30.7 -> 29.7 mm
- net N$19: track 8.77 -> 9.68 mm
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Other:
- board text added: "17.05.10.A"
- board text added: "25"
- board text added: "A1+"
- board text added: "A1-"
- board text added: "A2+"
- board text added: "A2-"
- board text added: "A3+"
- board text added: "A3-"
- board text added: "B1+"
- board text added: "B1-"
- board text added: "B2+"
- board text added: "B2-"
- board text added: "B3+"
- board text added: "B3-"
- board text added: "CX_LRC"
- board text added: "CX_SCK"
- board text added: "CX_SD1"
- board text added: "CX_SD2"
- board text added: "CX_SD3"
- board text added: "GND"
- board text added: "IL+"
- board text added: "IL-"
- board text added: "INT"
- board text added: "IR+"
- board text added: "IR-"
- board text added: "L+"
- board text added: "L-"
- board text added: "MTC"
- board text added: "MUTEC"
- board text added: "R+"
- board text added: "R-"
- board text added: "RST_N"
- board text added: "RXP0"
- board text added: "RXP1"
- board text added: "RXP1_N"
- board text added: "RXP1_P"
- board text added: "RXP2"
- board text added: "RXP3"
- board text added: "RXP4"
- board text added: "RXP5"
- board text added: "RXP6"
- board text added: "SCL"
- board text added: "SDA"
- board text added: "SI_LRC"
- board text added: "SI_OUT"
- board text added: "SI_SCK"
- board text added: "TXP0"
